File: hw_sch/autoharpie/display.kicad_sch (KiCad schematic)
At the start: 0 parts

Commit message: matrix, flattening
Parts:
- added C10, C11, C12, C13, C14, C16, C17, C19, C20: 0.1u, symbol Device:C
- added J5: Conn_01x04_Socket, Display:OLED-128O064D, symbol Connector:Conn_01x04_Socket
- added R11, R12, R13, R14, R15, R17, R18, R20, R21: 10k, symbol Device:R
- added SW1: RotaryEncoder_Switch, symbol Device:RotaryEncoder_Switch
- added SW2, SW75, SW76: RotaryEncoder, symbol Device:RotaryEncoder
Connections:
- new net +3.3V: J5.3 (Pin_3)
- new net +3V3: R11.1, R12.1, R13.1, R14.1, R15.1, R17.1, R18.1, R20.1, R21.1
- new net DISPLAY_I2C_SCL: J5.2 (Pin_2)
- new net DISPLAY_I2C_SDA: J5.1 (Pin_1)
- new net FRONT_ROT_A: C11.1, R12.2, SW1.A
- new net FRONT_ROT_A1: C13.1, R14.2, SW2.A
- new net FRONT_ROT_A2: C16.1, R17.2, SW76.A
- new net FRONT_ROT_A3: C19.1, R20.2, SW75.A
- new net FRONT_ROT_B: C12.1, R13.2, SW1.B
- new net FRONT_ROT_B1: C14.1, R15.2, SW2.B
- new net FRONT_ROT_B2: C17.1, R18.2, SW76.B
- new net FRONT_ROT_B3: C20.1, R21.2, SW75.B
- new net FRONT_ROT_SW: C10.1, R11.2, SW1.S1
- new net GND: C10.2, C11.2, C12.2, C13.2, C14.2, C16.2, C17.2, C19.2, C20.2, J5.4 (Pin_4), SW1.C, SW1.S2, SW2.C, SW75.C, SW76.C
