File: hw_sch/autoharpie/autoharpie.kicad_sch (KiCad schematic)
At the start: 0 parts

Commit message: isolated ground
Other:
- removed sheet Chord
- sheet Chord & Sequencer ports: added C0, C1, C10, C11, C2, C3, C4, C5, C6, C7, C8, C9, LED_DIN, R0, R1, R2, R3, R4; removed none
Changed lines of the file:
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@@
     )
   )
-  (sheet (at 31.75 15.24) (size 62.23 54.61) (fields_autoplaced)
+  (sheet (at 31.75 16.51) (size 62.23 58.42) (fields_autoplaced)
     (stroke (width 0.1524) (type solid))
     (fill (color 0 0 0 0.0000))
-    (property "Sheetname" "Controller" (at 31.75 14.5284 0)
+    (property "Sheetname" "Controller" (at 31.75 15.7984 0)
       (effects (font (size 1.27 1.27)) (justify left bottom))
     )
-    (property "Sheetfile" "controller.kicad_sch" (at 31.75 70.4346 0)
+    (property "Sheetfile" "controller.kicad_sch" (at 31.75 75.5146 0)
       (effects (font (size 1.27 1.27)) (justify left top))
     )
@@
     )
   )
-  (sheet (at 31.75 120.65) (size 62.23 22.86) (fields_autoplaced)
+  (sheet (at 31.75 135.89) (size 62.23 7.62) (fields_autoplaced)
     (stroke (width 0.1524) (type solid))
     (fill (color 0 0 0 0.0000))
-    (property "Sheetname" "USB Power" (at 31.75 119.9384 0)
+    (property "Sheetname" "USB Power" (at 31.75 135.1784 0)
       (effects (font (size 1.27 1.27)) (justify left bottom))
     )
@@
       (effects (font (size 1.27 1.27)) (justify left top))
     )
-    (pin "USB_D-" bidirectional (at 93.98 125.73 0)
+    (pin "USB_D-" bidirectional (at 93.98 140.97 0)
       (effects (font (size 1.27 1.27)) (justify right))
     )
-    (pin "USB_D+" bidirectional (at 93.98 123.19 0)
+    (pin "USB_D+" bidirectional (at 93.98 138.43 0)
       (effects (font (size 1.27 1.27)) (justify right))
     )
@@
     )
   )
-  (sheet (at 31.75 76.2) (size 62.23 38.1) (fields_autoplaced)
+  (sheet (at 31.75 81.28) (size 62.23 48.26) (fields_autoplaced)
     (stroke (width 0.1524) (type solid))
     (fill (color 0 0 0 0.0000))
-    (property "Sheetname" "Chord & Sequencer" (at 31.75 75.4884 0)
+    (property "Sheetname" "Chord & Sequencer" (at 31.75 80.5684 0)
       (effects (font (size 1.27 1.27)) (justify left bottom))
     )
-    (property "Sheetfile" "fpio_chord_seq.kicad_sch" (at 31.75 114.8846 0)
+    (property "Sheetfile" "fpio_chord_seq.kicad_sch" (at 31.75 130.1246 0)
       (effects (font (size 1.27 1.27)) (justify left top))
+    )
+    (pin "C7" input (at 93.98 114.3 0)
+      (effects (font (size 1.27 1.27)) (justify right))
+    )
+    (pin "C6" input (at 93.98 111.76 0)
+      (effects (font (size 1.27 1.27)) (justify right))
+    )
+    (pin "C2" input (at 93.98 101.6 0)
+      (effects (font (size 1.27 1.27)) (justify right))
+    )
+    (pin "C5" input (at 93.98 109.22 0)
+      (effects (font (size 1.27 1.27)) (justify right))
+    )
+    (pin "C3" input (at 93.98 104.14 0)
+      (effects (font (size 1.27 1.27)) (justify right))
+    )
+    (pin "C4" input (at 93.98 106.68 0)
+      (effects (font (size 1.27 1.27)) (justify right))
+    )
+    (pin "R0" output (at 93.98 83.82 0)
+      (effects (font (size 1.27 1.27)) (justify right))
+    )
+    (pin "C1" input (at 93.98 99.06 0)
+      (effects (font (size 1.27 1.27)) (justify right))
+    )
+    (pin "C0" input (at 93.98 96.52 0)
+      (effects (font (size 1.27 1.27)) (justify right))
+    )
+    (pin "R1" output (at 93.98 86.36 0)
+      (effects (font (size 1.27 1.27)) (justify right))
+    )
+    (pin "R2" output (at 93.98 88.9 0)
+      (effects (font (size 1.27 1.27)) (justify right))
+    )
+    (pin "R4" output (at 93.98 93.98 0)
+      (effects (font (size 1.27 1.27)) (justify right))
+    )
+    (pin "R3" output (at 93.98 91.44 0)
+      (effects (font (size 1.27 1.27)) (justify right))
+    )
+    (pin "LED_DIN" input (at 93.98 127 0)
+      (effects (font (size 1.27 1.27)) (justify right))
+    )
+    (pin "C8" input (at 93.98 116.84 0)
+      (effects (font (size 1.27 1.27)) (justify right))
+    )
+    (pin "C9" input (at 93.98 119.38 0)
+      (effects (font (size 1.27 1.27)) (justify right))
+    )
+    (pin "C10" input (at 93.98 121.92 0)
+      (effects (font (size 1.27 1.27)) (justify right))
+    )
+    (pin "C11" input (at 93.98 124.46 0)
+      (effects (font (size 1.27 1.27)) (justify right))
     )
     (instances
@@
       )
     )
-  )
-  (sheet (at 200.66 73.66) (size 73.66 33.02) (fields_autoplaced)
-    (stroke (width 0.1524) (type solid))
-    (fill (color 0 0 0 0.0000))
-    (property "Sheetname" "Chord" (at 200.66 72.9484 0)
-      (effects (font (size 1.27 1.27)) (justify left bottom))
-    )
-    (property "Sheetfile" "chord.kicad_sch" (at 200.66 107.2646 0)
-      (effects (font (size 1.27 1.27)) (justify left top))
-    )
-    (instances
-      (project "autoharpie"
-        (path "/f22a88c4-866b-40a0-9fc2-96344be0ec71" (page "5"))
-      )
-    )
