File: hw_sch/autoharpie/fpio_chord_seq.kicad_sch (KiCad schematic)
At the start: 144 parts, among them SW10 SW_Push_45deg, SW100 SW_Push_45deg, SW101 SW_Push_45deg, SW102 SW_Push_45deg, SW103 SW_Push_45deg, SW104 SW_Push_45deg, SW105 SW_Push_45deg, SW106 SW_Push_45deg, SW107 SW_Push_45deg, SW108 SW_Push_45deg, SW109 SW_Push_45deg, SW11 SW_Push_45deg, SW110 SW_Push_45deg, SW111 SW_Push_45deg, SW112 SW_Push_45deg, SW113 SW_Push_45deg, SW114 SW_Push_45deg, SW115 SW_Push_45deg, SW116 SW_Push_45deg, SW117 SW_Push_45deg, SW118 SW_Push_45deg, SW119 SW_Push_45deg, SW12 SW_Push_45deg, SW120 SW_Push_45deg, SW121 SW_Push_45deg, SW122 SW_Push_45deg, SW123 SW_Push_45deg, SW124 SW_Push_45deg, SW125 SW_Push_45deg, SW126 SW_Push_45deg, SW127 SW_Push_45deg, SW128 SW_Push_45deg, SW129 SW_Push_45deg, SW13 SW_Push_45deg, SW130 SW_Push_45deg, SW131 SW_Push_45deg, SW132 SW_Push_45deg, SW133 SW_Push_45deg, SW134 SW_Push_45deg, SW135 SW_Push_45deg, SW136 SW_Push_45deg, SW14 SW_Push_45deg, SW15 SW_Push_45deg, SW16 SW_Push_45deg, SW5 SW_Push_45deg, SW6 SW_Push_45deg, SW7 SW_Push_45deg, SW77 SW_Push_45deg, SW78 SW_Push_45deg, SW79 SW_Push_45deg, SW8 SW_Push_45deg, SW80 SW_Push_45deg, SW81 SW_Push_45deg, SW82 SW_Push_45deg, SW83 SW_Push_45deg, SW84 SW_Push_45deg, SW85 SW_Push_45deg, SW86 SW_Push_45deg, SW87 SW_Push_45deg, SW88 SW_Push_45deg, SW89 SW_Push_45deg, SW9 SW_Push_45deg, SW90 SW_Push_45deg, SW91 SW_Push_45deg, SW92 SW_Push_45deg, SW93 SW_Push_45deg, SW94 SW_Push_45deg, SW95 SW_Push_45deg, SW96 SW_Push_45deg, SW97 SW_Push_45deg, SW98 SW_Push_45deg, SW99 SW_Push_45deg

Commit message: keypad
Parts:
- D10: renamed from D77; footprint (none) -> Diode_THT:D_DO-35_SOD27_P7.62mm_Horizontal
- D11: renamed from D78; footprint (none) -> Diode_THT:D_DO-35_SOD27_P7.62mm_Horizontal
- D12: renamed from D79; footprint (none) -> Diode_THT:D_DO-35_SOD27_P7.62mm_Horizontal
- D13: renamed from D80; footprint (none) -> Diode_THT:D_DO-35_SOD27_P7.62mm_Horizontal
- D14: renamed from D81; footprint (none) -> Diode_THT:D_DO-35_SOD27_P7.62mm_Horizontal
- D15: renamed from D82; footprint (none) -> Diode_THT:D_DO-35_SOD27_P7.62mm_Horizontal
- D16: renamed from D83; footprint (none) -> Diode_THT:D_DO-35_SOD27_P7.62mm_Horizontal
- D17: renamed from D84; footprint (none) -> Diode_THT:D_DO-35_SOD27_P7.62mm_Horizontal
- D18: renamed from D85; footprint (none) -> Diode_THT:D_DO-35_SOD27_P7.62mm_Horizontal
- D19: renamed from D86; footprint (none) -> Diode_THT:D_DO-35_SOD27_P7.62mm_Horizontal
- D20: renamed from D87; footprint (none) -> Diode_THT:D_DO-35_SOD27_P7.62mm_Horizontal
- D21: renamed from D88; footprint (none) -> Diode_THT:D_DO-35_SOD27_P7.62mm_Horizontal
- D22: renamed from D89; footprint (none) -> Diode_THT:D_DO-35_SOD27_P7.62mm_Horizontal
- D23: renamed from D90; footprint (none) -> Diode_THT:D_DO-35_SOD27_P7.62mm_Horizontal
- D24: renamed from D91; footprint (none) -> Diode_THT:D_DO-35_SOD27_P7.62mm_Horizontal
- D25: renamed from D92; footprint (none) -> Diode_THT:D_DO-35_SOD27_P7.62mm_Horizontal
- D26: renamed from D93; footprint (none) -> Diode_THT:D_DO-35_SOD27_P7.62mm_Horizontal
- D27: renamed from D94; footprint (none) -> Diode_THT:D_DO-35_SOD27_P7.62mm_Horizontal
- D28: renamed from D95; footprint (none) -> Diode_THT:D_DO-35_SOD27_P7.62mm_Horizontal
- D29: renamed from D96; footprint (none) -> Diode_THT:D_DO-35_SOD27_P7.62mm_Horizontal
- D30: renamed from D97; footprint (none) -> Diode_THT:D_DO-35_SOD27_P7.62mm_Horizontal
- D31: renamed from D98; footprint (none) -> Diode_THT:D_DO-35_SOD27_P7.62mm_Horizontal
- D32: renamed from D99; footprint (none) -> Diode_THT:D_DO-35_SOD27_P7.62mm_Horizontal
- D33: renamed from D100; footprint (none) -> Diode_THT:D_DO-35_SOD27_P7.62mm_Horizontal
- D34: renamed from D101; footprint (none) -> Diode_THT:D_DO-35_SOD27_P7.62mm_Horizontal
- D35: renamed from D102; footprint (none) -> Diode_THT:D_DO-35_SOD27_P7.62mm_Horizontal
- D36: renamed from D103; footprint (none) -> Diode_THT:D_DO-35_SOD27_P7.62mm_Horizontal
- D37: renamed from D104; footprint (none) -> Diode_THT:D_DO-35_SOD27_P7.62mm_Horizontal
- D38: renamed from D105; footprint (none) -> Diode_THT:D_DO-35_SOD27_P7.62mm_Horizontal
- D39: renamed from D106; footprint (none) -> Diode_THT:D_DO-35_SOD27_P7.62mm_Horizontal
- D40: renamed from D107; footprint (none) -> Diode_THT:D_DO-35_SOD27_P7.62mm_Horizontal
- D41: renamed from D108; footprint (none) -> Diode_THT:D_DO-35_SOD27_P7.62mm_Horizontal
- D42: renamed from D109; footprint (none) -> Diode_THT:D_DO-35_SOD27_P7.62mm_Horizontal
- D43: renamed from D110; footprint (none) -> Diode_THT:D_DO-35_SOD27_P7.62mm_Horizontal
- D44: renamed from D111; footprint (none) -> Diode_THT:D_DO-35_SOD27_P7.62mm_Horizontal
- D45: renamed from D112; footprint (none) -> Diode_THT:D_DO-35_SOD27_P7.62mm_Horizontal
- D46: renamed from D113; footprint (none) -> Diode_THT:D_DO-35_SOD27_P7.62mm_Horizontal
- D47: renamed from D114; footprint (none) -> Diode_THT:D_DO-35_SOD27_P7.62mm_Horizontal
- D48: renamed from D115; footprint (none) -> Diode_THT:D_DO-35_SOD27_P7.62mm_Horizontal
- D49: renamed from D116; footprint (none) -> Diode_THT:D_DO-35_SOD27_P7.62mm_Horizontal
- D50: renamed from D117; footprint (none) -> Diode_THT:D_DO-35_SOD27_P7.62mm_Horizontal
- D51: renamed from D118; footprint (none) -> Diode_THT:D_DO-35_SOD27_P7.62mm_Horizontal
- D52: renamed from D119; footprint (none) -> Diode_THT:D_DO-35_SOD27_P7.62mm_Horizontal
- D53: renamed from D120; footprint (none) -> Diode_THT:D_DO-35_SOD27_P7.62mm_Horizontal
- D54: renamed from D121; footprint (none) -> Diode_THT:D_DO-35_SOD27_P7.62mm_Horizontal
- D55: renamed from D122; footprint (none) -> Diode_THT:D_DO-35_SOD27_P7.62mm_Horizontal
- D56: renamed from D123; footprint (none) -> Diode_THT:D_DO-35_SOD27_P7.62mm_Horizontal
- D57: renamed from D124; footprint (none) -> Diode_THT:D_DO-35_SOD27_P7.62mm_Horizontal
- D58: renamed from D125; footprint (none) -> Diode_THT:D_DO-35_SOD27_P7.62mm_Horizontal
- D59: renamed from D126; footprint (none) -> Diode_THT:D_DO-35_SOD27_P7.62mm_Horizontal
- D60: renamed from D127; footprint (none) -> Diode_THT:D_DO-35_SOD27_P7.62mm_Horizontal
- D61: renamed from D128; footprint (none) -> Diode_THT:D_DO-35_SOD27_P7.62mm_Horizontal
- D62: renamed from D129; footprint (none) -> Diode_THT:D_DO-35_SOD27_P7.62mm_Horizontal
- D63: renamed from D130; footprint (none) -> Diode_THT:D_DO-35_SOD27_P7.62mm_Horizontal
- D64: renamed from D131; footprint (none) -> Diode_THT:D_DO-35_SOD27_P7.62mm_Horizontal
- D65: renamed from D132; footprint (none) -> Diode_THT:D_DO-35_SOD27_P7.62mm_Horizontal
- D66: renamed from D133; footprint (none) -> Diode_THT:D_DO-35_SOD27_P7.62mm_Horizontal
- D67: renamed from D3; footprint (none) -> Diode_THT:D_DO-35_SOD27_P7.62mm_Horizontal
- D68: renamed from D4; footprint (none) -> Diode_THT:D_DO-35_SOD27_P7.62mm_Horizontal
- D69: renamed from D5; footprint (none) -> Diode_THT:D_DO-35_SOD27_P7.62mm_Horizontal
- D7: renamed from D74; footprint (none) -> Diode_THT:D_DO-35_SOD27_P7.62mm_Horizontal
- D70: renamed from D6; footprint (none) -> Diode_THT:D_DO-35_SOD27_P7.62mm_Horizontal
- D71: renamed from D7; footprint (none) -> Diode_THT:D_DO-35_SOD27_P7.62mm_Horizontal
- D72: renamed from D8; footprint (none) -> Diode_THT:D_DO-35_SOD27_P7.62mm_Horizontal
- D73: renamed from D9; footprint (none) -> Diode_THT:D_DO-35_SOD27_P7.62mm_Horizontal
- D74: renamed from D10; footprint (none) -> Diode_THT:D_DO-35_SOD27_P7.62mm_Horizontal
- D75: renamed from D11; footprint (none) -> Diode_THT:D_DO-35_SOD27_P7.62mm_Horizontal
- D76: renamed from D12; footprint (none) -> Diode_THT:D_DO-35_SOD27_P7.62mm_Horizontal
- D77: renamed from D13; footprint (none) -> Diode_THT:D_DO-35_SOD27_P7.62mm_Horizontal
- D78: renamed from D14; footprint (none) -> Diode_THT:D_DO-35_SOD27_P7.62mm_Horizontal
- D8: renamed from D75; footprint (none) -> Diode_THT:D_DO-35_SOD27_P7.62mm_Horizontal
- D9: renamed from D76; footprint (none) -> Diode_THT:D_DO-35_SOD27_P7.62mm_Horizontal
- SW10: renamed from SW83; footprint (none) -> Button_Switch_THT:SW_PUSH_6mm_H4.3mm
- SW11: renamed from SW84; footprint (none) -> Button_Switch_THT:SW_PUSH_6mm_H4.3mm
- SW12: renamed from SW85; footprint (none) -> Button_Switch_THT:SW_PUSH_6mm_H4.3mm
- SW13: renamed from SW86; footprint (none) -> Button_Switch_THT:SW_PUSH_6mm_H4.3mm
- SW14: renamed from SW87; footprint (none) -> Button_Switch_THT:SW_PUSH_6mm_H4.3mm
- SW15: renamed from SW88; footprint (none) -> Button_Switch_THT:SW_PUSH_6mm_H4.3mm
- SW16: renamed from SW89; footprint (none) -> Button_Switch_THT:SW_PUSH_6mm_H4.3mm
- SW17: renamed from SW90; footprint (none) -> Button_Switch_THT:SW_PUSH_6mm_H4.3mm
- SW18: renamed from SW91; footprint (none) -> Button_Switch_THT:SW_PUSH_6mm_H4.3mm
- SW19: renamed from SW92; footprint (none) -> Button_Switch_THT:SW_PUSH_6mm_H4.3mm
- SW20: renamed from SW93; footprint (none) -> Button_Switch_THT:SW_PUSH_6mm_H4.3mm
- SW21: renamed from SW94; footprint (none) -> Button_Switch_THT:SW_PUSH_6mm_H4.3mm
- SW22: renamed from SW95; footprint (none) -> Button_Switch_THT:SW_PUSH_6mm_H4.3mm
- SW23: renamed from SW96; footprint (none) -> Button_Switch_THT:SW_PUSH_6mm_H4.3mm
- SW24: renamed from SW97; footprint (none) -> Button_Switch_THT:SW_PUSH_6mm_H4.3mm
- SW25: renamed from SW98; footprint (none) -> Button_Switch_THT:SW_PUSH_6mm_H4.3mm
- SW26: renamed from SW99; footprint (none) -> Button_Switch_THT:SW_PUSH_6mm_H4.3mm
- SW27: renamed from SW100; footprint (none) -> Button_Switch_THT:SW_PUSH_6mm_H4.3mm
- SW28: renamed from SW101; footprint (none) -> Button_Switch_THT:SW_PUSH_6mm_H4.3mm
- SW29: renamed from SW102; footprint (none) -> Button_Switch_THT:SW_PUSH_6mm_H4.3mm
- SW30: renamed from SW103; footprint (none) -> Button_Switch_THT:SW_PUSH_6mm_H4.3mm
- SW31: renamed from SW104; footprint (none) -> Button_Switch_THT:SW_PUSH_6mm_H4.3mm
- SW32: renamed from SW105; footprint (none) -> Button_Switch_THT:SW_PUSH_6mm_H4.3mm
- SW33: renamed from SW106; footprint (none) -> Button_Switch_THT:SW_PUSH_6mm_H4.3mm
- SW34: renamed from SW107; footprint (none) -> Button_Switch_THT:SW_PUSH_6mm_H4.3mm
- SW35: renamed from SW108; footprint (none) -> Button_Switch_THT:SW_PUSH_6mm_H4.3mm
- SW36: renamed from SW109; footprint (none) -> Button_Switch_THT:SW_PUSH_6mm_H4.3mm
- SW37: renamed from SW110; footprint (none) -> Button_Switch_THT:SW_PUSH_6mm_H4.3mm
- SW38: renamed from SW111; footprint (none) -> Button_Switch_THT:SW_PUSH_6mm_H4.3mm
- SW39: renamed from SW112; footprint (none) -> Button_Switch_THT:SW_PUSH_6mm_H4.3mm
- SW4: renamed from SW77; footprint (none) -> Button_Switch_THT:SW_PUSH_6mm_H4.3mm
- SW40: renamed from SW113; footprint (none) -> Button_Switch_THT:SW_PUSH_6mm_H4.3mm
- SW41: renamed from SW114; footprint (none) -> Button_Switch_THT:SW_PUSH_6mm_H4.3mm
- SW42: renamed from SW115; footprint (none) -> Button_Switch_THT:SW_PUSH_6mm_H4.3mm
- SW43: renamed from SW116; footprint (none) -> Button_Switch_THT:SW_PUSH_6mm_H4.3mm
- SW44: renamed from SW117; footprint (none) -> Button_Switch_THT:SW_PUSH_6mm_H4.3mm
- SW45: renamed from SW118; footprint (none) -> Button_Switch_THT:SW_PUSH_6mm_H4.3mm
- SW46: renamed from SW119; footprint (none) -> Button_Switch_THT:SW_PUSH_6mm_H4.3mm
- SW47: renamed from SW120; footprint (none) -> Button_Switch_THT:SW_PUSH_6mm_H4.3mm
- SW48: renamed from SW121; footprint (none) -> Button_Switch_THT:SW_PUSH_6mm_H4.3mm
- SW49: renamed from SW122; footprint (none) -> Button_Switch_THT:SW_PUSH_6mm_H4.3mm
- SW5: renamed from SW78; footprint (none) -> Button_Switch_THT:SW_PUSH_6mm_H4.3mm
- SW50: renamed from SW123; footprint (none) -> Button_Switch_THT:SW_PUSH_6mm_H4.3mm
- SW51: renamed from SW124; footprint (none) -> Button_Switch_THT:SW_PUSH_6mm_H4.3mm
- SW52: renamed from SW125; footprint (none) -> Button_Switch_THT:SW_PUSH_6mm_H4.3mm
- SW53: renamed from SW126; footprint (none) -> Button_Switch_THT:SW_PUSH_6mm_H4.3mm
- SW54: renamed from SW127; footprint (none) -> Button_Switch_THT:SW_PUSH_6mm_H4.3mm
- SW55: renamed from SW128; footprint (none) -> Button_Switch_THT:SW_PUSH_6mm_H4.3mm
- SW56: renamed from SW129; footprint (none) -> Button_Switch_THT:SW_PUSH_6mm_H4.3mm
- SW57: renamed from SW130; footprint (none) -> Button_Switch_THT:SW_PUSH_6mm_H4.3mm
- SW58: renamed from SW131; footprint (none) -> Button_Switch_THT:SW_PUSH_6mm_H4.3mm
- SW59: renamed from SW132; footprint (none) -> Button_Switch_THT:SW_PUSH_6mm_H4.3mm
- SW6: renamed from SW79; footprint (none) -> Button_Switch_THT:SW_PUSH_6mm_H4.3mm
- SW60: renamed from SW133; footprint (none) -> Button_Switch_THT:SW_PUSH_6mm_H4.3mm
- SW61: renamed from SW134; footprint (none) -> Button_Switch_THT:SW_PUSH_6mm_H4.3mm
- SW62: renamed from SW135; footprint (none) -> Button_Switch_THT:SW_PUSH_6mm_H4.3mm
- SW63: renamed from SW136; footprint (none) -> Button_Switch_THT:SW_PUSH_6mm_H4.3mm
- SW64: renamed from SW5; footprint (none) -> Button_Switch_THT:SW_PUSH_6mm_H4.3mm
- SW65: renamed from SW6; footprint (none) -> Button_Switch_THT:SW_PUSH_6mm_H4.3mm
- SW66: renamed from SW7; footprint (none) -> Button_Switch_THT:SW_PUSH_6mm_H4.3mm
- SW67: renamed from SW8; footprint (none) -> Button_Switch_THT:SW_PUSH_6mm_H4.3mm
- SW68: renamed from SW9; footprint (none) -> Button_Switch_THT:SW_PUSH_6mm_H4.3mm
- SW69: renamed from SW10; footprint (none) -> Button_Switch_THT:SW_PUSH_6mm_H4.3mm
- SW7: renamed from SW80; footprint (none) -> Button_Switch_THT:SW_PUSH_6mm_H4.3mm
- SW70: renamed from SW11; footprint (none) -> Button_Switch_THT:SW_PUSH_6mm_H4.3mm
- SW71: renamed from SW12; footprint (none) -> Button_Switch_THT:SW_PUSH_6mm_H4.3mm
- SW72: renamed from SW13; footprint (none) -> Button_Switch_THT:SW_PUSH_6mm_H4.3mm
- SW73: renamed from SW14; footprint (none) -> Button_Switch_THT:SW_PUSH_6mm_H4.3mm
- SW74: renamed from SW15; footprint (none) -> Button_Switch_THT:SW_PUSH_6mm_H4.3mm
- SW75: renamed from SW16; footprint (none) -> Button_Switch_THT:SW_PUSH_6mm_H4.3mm
- SW8: renamed from SW81; footprint (none) -> Button_Switch_THT:SW_PUSH_6mm_H4.3mm
- SW9: renamed from SW82; footprint (none) -> Button_Switch_THT:SW_PUSH_6mm_H4.3mm
Other:
- removed sheet Sequencer Buttons

Commit message: rev 0.1 pcb
Parts:
- removed D10, D11, D12, D13, D14, D15, D16, D17, D18, D19, D20, D21, D22, D23, D24, D25, D26, D27, D28, D29, D30, D31, D32, D33, D34, D35, D36, D37, D38, D39, D40, D41, D42, D43, D44, D45, D46, D47, D48, D49, D50, D51, D52, D53, D54, D55, D56, D57, D58, D59, D60, D61, D62, D63, D64, D65, D66, D67, D68, D69, D7, D70, D71, D72, D73, D74, D75, D76, D77, D78, D8, D9: 1N4148, Diode_THT:D_DO-35_SOD27_P7.62mm_Horizontal, symbol Device:D
- removed SW10, SW11, SW12, SW13, SW14, SW15, SW16, SW17, SW18, SW19, SW20, SW21, SW22, SW23, SW24, SW25, SW26, SW27, SW28, SW29, SW30, SW31, SW32, SW33, SW34, SW35, SW36, SW37, SW38, SW39, SW4, SW40, SW41, SW42, SW43, SW44, SW45, SW46, SW47, SW48, SW49, SW5, SW50, SW51, SW52, SW53, SW54, SW55, SW56, SW57, SW58, SW59, SW6, SW60, SW61, SW62, SW63, SW64, SW65, SW66, SW67, SW68, SW69, SW7, SW70, SW71, SW72, SW73, SW74, SW75, SW8, SW9: SW_Push_45deg, Button_Switch_THT:SW_PUSH_6mm_H4.3mm, symbol Switch:SW_Push_45deg
- added SW10, SW11, SW12, SW13, SW14, SW15, SW16, SW17, SW18, SW19, SW2, SW20, SW21, SW22, SW23, SW24, SW25, SW26, SW27, SW28, SW29, SW3, SW30, SW31, SW32, SW33, SW34, SW35, SW36, SW37, SW38, SW39, SW4, SW40, SW41, SW42, SW43, SW44, SW45, SW46, SW47, SW48, SW49, SW5, SW50, SW51, SW52, SW53, SW54, SW55, SW56, SW57, SW58, SW59, SW6, SW60, SW61, SW7, SW8, SW9: SW_Push, Button_Switch_THT:SW_PUSH_6mm, symbol Switch:SW_Push
Connections:
- net C0: now also SW14.2, SW2.2, SW26.2, SW38.2, SW50.2
- net C1: now also SW15.2, SW27.2, SW3.2, SW39.2, SW51.2
- net C10: now also SW12.2, SW24.2, SW36.2, SW48.2, SW60.2
- net C11: now also SW13.2, SW25.2, SW37.2, SW49.2, SW61.2
- net C2: now also SW16.2, SW28.2, SW4.2, SW40.2, SW52.2
- net C3: now also SW17.2, SW29.2, SW41.2, SW5.2, SW53.2
- net C4: now also SW18.2, SW30.2, SW42.2, SW54.2, SW6.2
- net C5: now also SW19.2, SW31.2, SW43.2, SW55.2, SW7.2
- net C6: now also SW20.2, SW32.2, SW44.2, SW56.2, SW8.2
- net C7: now also SW21.2, SW33.2, SW45.2, SW57.2, SW9.2
- net C8: now also SW10.2, SW22.2, SW34.2, SW46.2, SW58.2
- net C9: now also SW11.2, SW23.2, SW35.2, SW47.2, SW59.2
- net R0: now also SW10.1, SW11.1, SW12.1, SW13.1, SW2.1, SW3.1, SW4.1, SW5.1, SW6.1, SW7.1, SW8.1, SW9.1
- net R1: now also SW14.1, SW15.1, SW16.1, SW17.1, SW18.1, SW19.1, SW20.1, SW21.1, SW22.1, SW23.1, SW24.1, SW25.1
- net R2: now also SW26.1, SW27.1, SW28.1, SW29.1, SW30.1, SW31.1, SW32.1, SW33.1, SW34.1, SW35.1, SW36.1, SW37.1
- net R3: now also SW38.1, SW39.1, SW40.1, SW41.1, SW42.1, SW43.1, SW44.1, SW45.1, SW46.1, SW47.1, SW48.1, SW49.1
- net R4: now also SW50.1, SW51.1, SW52.1, SW53.1, SW54.1, SW55.1, SW56.1, SW57.1, SW58.1, SW59.1, SW60.1, SW61.1
Other:
- removed sheet Chord LEDs
- removed sheet Sequencer LEDs
- added sheet LEDs (leds.kicad_sch)

Commit message: ic fix atept
Parts:
- renumbered SW9 to SW10, SW10 to SW11, SW11 to SW12, SW12 to SW13, SW13 to SW14, SW14 to SW15, SW15 to SW16, SW16 to SW17, SW17 to SW18, SW18 to SW19, SW19 to SW20, SW20 to SW21, SW21 to SW22, SW22 to SW23, SW23 to SW24, SW24 to SW25, SW25 to SW26, SW26 to SW27, SW27 to SW28, SW28 to SW29, SW2 to SW3, SW29 to SW30, SW30 to SW31, SW31 to SW32, SW32 to SW33, SW33 to SW34, SW34 to SW35, SW35 to SW36, SW36 to SW37, SW37 to SW38, SW38 to SW39, SW3 to SW4, SW39 to SW40, SW40 to SW41, SW41 to SW42, SW42 to SW43, SW43 to SW44, SW44 to SW45, SW45 to SW46, SW46 to SW47, SW47 to SW48, SW48 to SW49, SW4 to SW5, SW49 to SW50, SW50 to SW51, SW51 to SW52, SW52 to SW53, SW53 to SW54, SW54 to SW55, SW55 to SW56, SW56 to SW57, SW57 to SW58, SW58 to SW59, SW5 to SW6, SW59 to SW60, SW60 to SW61, SW61 to SW62, SW6 to SW7, SW7 to SW8, SW8 to SW9
