File: hw_sch/autoharpie/capsense_bus_switch.kicad_sch (KiCad schematic)
At the start: 16 parts, among them U11 FSA3157L6X, U12 FSA3157L6X, U13 FSA3157L6X, U14 FSA3157L6X, U15 FSA3157L6X, U16 FSA3157L6X, U17 FSA3157L6X, U5 FSA3157P6X

Commit message: DAC, touch sensors
Connections:
- net SW renamed SWITCH
Changed lines of the file:
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@@
+    (stroke (width 0) (type default))
+  )
+  (wire (pts (xy 139.7 50.8) (xy 147.32 50.8))
     (stroke (width 0) (type default))
   )
@@
   (label "A2" (at 93.98 64.77 180) (fields_autoplaced)
     (effects (font (size 1.27 1.27)) (justify right bottom))
+  )
+  (label "SW" (at 139.7 50.8 0) (fields_autoplaced)
+    (effects (font (size 1.27 1.27)) (justify left bottom))
   )
   (label "A2" (at 39.37 36.83 180) (fields_autoplaced)
@@
     (effects (font (size 1.27 1.27)) (justify left))
   )
+  (hierarchical_label "SWITCH" (shape input) (at 147.32 50.8 0) (fields_autoplaced)
+    (effects (font (size 1.27 1.27)) (justify left))
+  )
