File: hw_sch/autoharpie/key_sensor.kicad_sch (KiCad schematic)
At the start: 0 parts

Commit message: DAC, touch sensors
Other:
- sheet Key renamed Key 1
- added sheet Key 2 (key.kicad_sch)
- added sheet Key 3 (key.kicad_sch)
- added sheet Key 4 (key.kicad_sch)
- added sheet Key 5 (key.kicad_sch)
- added sheet Key 6 (key.kicad_sch)
- added sheet Key 7 (key.kicad_sch)
- added sheet Key 8 (key.kicad_sch)
- sheet Key 1 ports: added C0, RX0, RX1, RX2, RX3, RX4, RX5, RX6, RX7; removed none
