File: hw_sch/autoharpie/chordmod_led.kicad_sch (KiCad schematic)
At the start: 24 parts

Commit message: keypad
Parts:
- C15, C18, C21, C22, C23, C24, C25, C26, C27, C28, C29, C30: footprint (none) -> Capacitor_SMD:C_0402_1005Metric
