File: hw_sch/autoharpie/fpio_buttons.kicad_sch (KiCad schematic)
At the start: 27 parts, among them SW19 SW_Push, SW20 SW_Push, SW21 SW_Push

Commit message: keypad
Parts:
- removed C63 (x3): 0.1u, symbol Device:C
- removed R26 (x3): 10k, symbol Device:R
- removed SW19 (x3): SW_Push, symbol Switch:SW_Push
