File: hw_sch/autoharpie/sequencer_leds.kicad_sch (KiCad schematic)
At the start: 48 parts

Commit message: keypad
Parts:
- C40: renamed from C15; footprint (none) -> Capacitor_SMD:C_0402_1005Metric
- C41: renamed from C18; footprint (none) -> Capacitor_SMD:C_0402_1005Metric
- C42: renamed from C21; footprint (none) -> Capacitor_SMD:C_0402_1005Metric
- C43: renamed from C22; footprint (none) -> Capacitor_SMD:C_0402_1005Metric
- C44: renamed from C23; footprint (none) -> Capacitor_SMD:C_0402_1005Metric
- C45: renamed from C24; footprint (none) -> Capacitor_SMD:C_0402_1005Metric
- C46: renamed from C25; footprint (none) -> Capacitor_SMD:C_0402_1005Metric
- C47: renamed from C26; footprint (none) -> Capacitor_SMD:C_0402_1005Metric
- C48: renamed from C27; footprint (none) -> Capacitor_SMD:C_0402_1005Metric
- C49: renamed from C28; footprint (none) -> Capacitor_SMD:C_0402_1005Metric
- C50: renamed from C29; footprint (none) -> Capacitor_SMD:C_0402_1005Metric
- C51: renamed from C30; footprint (none) -> Capacitor_SMD:C_0402_1005Metric
- C52: renamed from C31; footprint (none) -> Capacitor_SMD:C_0402_1005Metric
- C53: renamed from C32; footprint (none) -> Capacitor_SMD:C_0402_1005Metric
- C54: renamed from C33; footprint (none) -> Capacitor_SMD:C_0402_1005Metric
- C55: renamed from C34; footprint (none) -> Capacitor_SMD:C_0402_1005Metric
- C56: renamed from C35; footprint (none) -> Capacitor_SMD:C_0402_1005Metric
- C57: renamed from C36; footprint (none) -> Capacitor_SMD:C_0402_1005Metric
- C58: renamed from C37; footprint (none) -> Capacitor_SMD:C_0402_1005Metric
- C59: renamed from C38; footprint (none) -> Capacitor_SMD:C_0402_1005Metric
- C60: renamed from C39; footprint (none) -> Capacitor_SMD:C_0402_1005Metric
- C61: renamed from C40; footprint (none) -> Capacitor_SMD:C_0402_1005Metric
- C62: renamed from C41; footprint (none) -> Capacitor_SMD:C_0402_1005Metric
- C63: renamed from C42; footprint (none) -> Capacitor_SMD:C_0402_1005Metric
- renumbered D154 to D100, D155 to D101, D156 to D102, D157 to D103, D134 to D80, D135 to D81, D136 to D82, D137 to D83, D138 to D84, D139 to D85, D140 to D86, D141 to D87, D142 to D88, D143 to D89, D144 to D90, D145 to D91, D146 to D92, D147 to D93, D148 to D94, D149 to D95, D150 to D96, D151 to D97, D152 to D98, D153 to D99
