File: hw_sch/autoharpie/rxpin_filter.kicad_sch (KiCad schematic)
At the start: 16 parts

Commit message: keypad
Parts:
- removed C45 (x8): 68p, symbol Device:C
- R30: footprint (none) -> Resistor_THT:R_Axial_DIN0204_L3.6mm_D1.6mm_P7.62mm_Horizontal
