File: hw_sch/autoharpie/usb_psu.kicad_sch (KiCad schematic)
At the start: 16 parts, among them J1 USB_C_Receptacle_USB2.0, U19 NCV8114ASN180T1G, U4 AP2112K-3.3, U7 RT6150B-33GQW

Commit message: keypad
Parts:
- added D1: PMEG2010AEH, Diode_SMD:D_SOD-123F, symbol Diode:PMEG2010AEH
- added J2: Conn_01x02_Pin, Connector_JST:JST_PH_B2B-PH-K_1x02_P2.00mm_Vertical, symbol Connector:Conn_01x02_Pin
- added R4, R9: 100k, Resistor_THT:R_Axial_DIN0204_L3.6mm_D1.6mm_P7.62mm_Horizontal, symbol Device:R
- added R7, R8: 10, Resistor_THT:R_Axial_DIN0204_L3.6mm_D1.6mm_P7.62mm_Horizontal, symbol Device:R
- C24: renamed from C55; footprint (none) -> Capacitor_SMD:C_0805_2012Metric
- C25: renamed from C54; footprint (none) -> Capacitor_SMD:C_0805_2012Metric
- C91: footprint (none) -> Capacitor_SMD:C_0402_1005Metric
- J1: footprint (none) -> Connector_USB:USB_C_Receptacle_GCT_USB4135-GF-A_6P_TopMnt_Horizontal
- L1: renamed from L3; footprint (none) -> Inductor_SMD:L_0805_2012Metric
- R10: renamed from R19; footprint (none) -> Resistor_THT:R_Axial_DIN0204_L3.6mm_D1.6mm_P7.62mm_Horizontal
- R11: renamed from R22; footprint (none) -> Resistor_THT:R_Axial_DIN0204_L3.6mm_D1.6mm_P7.62mm_Horizontal
- R5: renamed from R1; footprint (none) -> Resistor_THT:R_Axial_DIN0204_L3.6mm_D1.6mm_P7.62mm_Horizontal
- R6: renamed from R2; footprint (none) -> Resistor_THT:R_Axial_DIN0204_L3.6mm_D1.6mm_P7.62mm_Horizontal
- U4: renamed from U7; footprint 10-WFDFN-EP_RIT -> footprints:RT6150B-33GQW
- renumbered U4 to U3
Connections:
- net USB_D+: now also R8.2; no longer J1.A6 (D+), J1.B6 (D+)
- net USB_D-: now also R7.2; no longer J1.A7 (D-), J1.B7 (D-)
- net +BATT: now reaches C25.1, D2.1 (K), R10.2, U4.5 (VIN), U4.8 (VINA)
- net +BATT: now also C91.1, C91.1, U19.1 (IN), U3.1 (VIN), D1.1 (K), R4.1, R9.1
- net 1V8_ENABLE: no longer names the net of U19.3 (EN)
- net 1V8_ENABLE: now also R4.2
- net 3V3_AUDIO_ENABLE: no longer names the net of U3.3 (EN)
- net 3V3_AUDIO_ENABLE: now also R9.2
- removed net VBUS: C91.1, C91.1, D2.2 (A), J1.A4 (VBUS), J1.A9 (VBUS), J1.B4 (VBUS), J1.B9 (VBUS), U19.1 (IN), U3.1 (VIN)
- new net: J1.A7 (D-), J1.B7 (D-), R7.1
- new net: D1.2 (A), J1.A4 (VBUS), J1.A9 (VBUS), J1.B4 (VBUS), J1.B9 (VBUS)
- new net: J1.A6 (D+), J1.B6 (D+), R8.1
- new net: D2.2 (A), J2.1 (Pin_1)
- new net -BATT: J2.2 (Pin_2)
Other:
- moved on the sheet: C24, C25, L1, R10, R11, U4

Commit message: rev 0.1 pcb
Parts:
- removed C24, C25: 47u, Capacitor_SMD:C_0805_2012Metric, symbol Device:C
- removed C91 (x4): 1u, Capacitor_SMD:C_0402_1005Metric, symbol Device:C
- removed D1: PMEG2010AEH, Diode_SMD:D_SOD-123F, symbol Diode:PMEG2010AEH
- removed J1: USB_C_Receptacle_USB2.0, Connector_USB:USB_C_Receptacle_GCT_USB4135-GF-A_6P_TopMnt_Horizontal, symbol Connector:USB_C_Receptacle_USB2.0
- removed J2: Conn_01x02_Pin, Connector_JST:JST_PH_B2B-PH-K_1x02_P2.00mm_Vertical, symbol Connector:Conn_01x02_Pin
- removed L1: 2u2, Inductor_SMD:L_0805_2012Metric, symbol Device:L
- removed R10, R11, R4, R9: 100k, Resistor_THT:R_Axial_DIN0204_L3.6mm_D1.6mm_P7.62mm_Horizontal, symbol Device:R
- removed R5, R6: 5.1k, Resistor_THT:R_Axial_DIN0204_L3.6mm_D1.6mm_P7.62mm_Horizontal, symbol Device:R
- removed R7, R8: 10, Resistor_THT:R_Axial_DIN0204_L3.6mm_D1.6mm_P7.62mm_Horizontal, symbol Device:R
- removed U19: NCV8114ASN180T1G, Package_TO_SOT_SMD:TSOT-23-5, symbol Regulator_Linear:NCV8114ASN180T1G
- removed U3: AP2112K-3.3, Package_TO_SOT_SMD:SOT-23-5, symbol Regulator_Linear:AP2112K-3.3
- removed U4: RT6150B-33GQW, footprints:RT6150B-33GQW, symbol 2023-03-08_23-59-12:RT6150B-33GQW
- added C3, C4, C5, C6: 1u, Capacitor_SMD:C_0603_1608Metric, symbol Device:C
- added J1: Conn_01x02_Pin, Connector_JST:JST_PH_S2B-PH-K_1x02_P2.00mm_Horizontal, symbol Connector:Conn_01x02_Pin
- added U4: AP2112K-1.8, Package_TO_SOT_SMD:SOT-23-5, symbol Regulator_Linear:AP2112K-1.8
- added U8: NCP1117-5.0_TO252, Package_TO_SOT_SMD:TO-252-2, symbol Regulator_Linear:NCP1117-5.0_TO252
- renumbered D2 to D13
Connections:
- net +1V8: now also C4.1, U4.5 (VOUT)
- net +3V3: now also C3.1, U4.1 (VIN), U4.3 (EN)
- net +BATT: now also C6.1, U8.2 (VO); no longer D13.1 (K)
- net GND: now also C3.2, C4.2, C5.2, C6.2, J1.1 (Pin_1), U4.2 (GND), U8.1 (GND)
- net BATT_SENSE: now reaches D13.2 (A)
- net BATT_SENSE: now also J1.2 (Pin_2)
- new net: C5.1, D13.1 (K), U8.3 (VI)
