File: hw_sch/autoharpie/usb_psu.kicad_sch (KiCad schematic)
At the start: 8 parts, among them J1 Conn_01x02_Pin, U4 AP2112K-1.8, U8 NCP1117-5.0_TO252

Commit message: ic fix atept
Parts:
- renumbered C5 to C3, C6 to C4, C3 to C5, C4 to C6, U8 to U4, U4 to U5
Connections:
- net +BATT renamed +5V

Commit message: final final final 0.1 rev
Parts:
- removed C5, C6: 1u, Capacitor_SMD:C_0603_1608Metric, symbol Device:C
- removed U5: AP2112K-1.8, Package_TO_SOT_SMD:SOT-23-5, symbol Regulator_Linear:AP2112K-1.8
Changed lines of the file:
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@@
 (kicad_sch (version 20230121) (generator eeschema)
   (paper "A4")
-  (junction (at 31.75 127) (diameter 0) (color 0 0 0 0)
-  )
   (junction (at 99.06 101.6) (diameter 0) (color 0 0 0 0)
   )
-  (junction (at 27.94 127) (diameter 0) (color 0 0 0 0)
-  )
   (junction (at 40.64 101.6) (diameter 0) (color 0 0 0 0)
-  )
-  (junction (at 58.42 127) (diameter 0) (color 0 0 0 0)
   )
   (junction (at 73.66 101.6) (diameter 0) (color 0 0 0 0)
@@
     (stroke (width 0) (type default))
   )
-  (wire (pts (xy 31.75 128.27) (xy 31.75 127))
-    (stroke (width 0) (type default))
-  )
-  (wire (pts (xy 53.34 127) (xy 58.42 127))
-    (stroke (width 0) (type default))
-  )
-  (wire (pts (xy 27.94 129.54) (xy 38.1 129.54))
-    (stroke (width 0) (type default))
-  )
-  (wire (pts (xy 58.42 127) (xy 63.5 127))
-    (stroke (width 0) (type default))
-  )
   (wire (pts (xy 104.14 99.06) (xy 104.14 101.6))
-    (stroke (width 0) (type default))
-  )
-  (wire (pts (xy 27.94 127) (xy 27.94 129.54))
-    (stroke (width 0) (type default))
-  )
-  (wire (pts (xy 27.94 127) (xy 31.75 127))
-    (stroke (width 0) (type default))
-  )
-  (wire (pts (xy 31.75 127) (xy 38.1 127))
-    (stroke (width 0) (type default))
-  )
-  (wire (pts (xy 27.94 123.19) (xy 27.94 127))
-    (stroke (width 0) (type default))
-  )
-  (wire (pts (xy 58.42 128.27) (xy 58.42 127))
     (stroke (width 0) (type default))
   )
@@
     (property "Intersheetrefs" "${INTERSHEET_REFS}" (at 40.64 78.4953 90)
       (effects (font (size 1.27 1.27)) (justify left) hide)
-    )
-  )
-  (symbol (lib_id "power:GND") (at 45.72 137.16 0) (unit 1)
-    (in_bom yes) (on_board yes) (dnp no) (fields_autoplaced)
-    (property "Reference" "#PWR040" (at 45.72 143.51 0)
-      (effects (font (size 1.27 1.27)) hide)
-    )
-    (property "Value" "GND" (at 45.72 142.24 0)
-      (effects (font (size 1.27 1.27)))
-    )
-    (property "Footprint" "" (at 45.72 137.16 0)
-      (effects (font (size 1.27 1.27)) hide)
-    )
-    (property "Datasheet" "" (at 45.72 137.16 0)
-      (effects (font (size 1.27 1.27)) hide)
-    )
-    (pin "1")
-    (instances
-      (project "autoharpie"
-        (path "/f22a88c4-866b-40a0-9fc2-96344be0ec71/99b052d6-7969-4dd2-91c7-8bd18b784c30"
-          (reference "#PWR040") (unit 1)
-        )
-      )
     )
   )
@@
     )
   )
-  (symbol (lib_id "power:+3V3") (at 27.94 123.19 0) (unit 1)
-    (in_bom yes) (on_board yes) (dnp no) (fields_autoplaced)
-    (property "Reference" "#PWR036" (at 27.94 127 0)
-      (effects (font (size 1.27 1.27)) hide)
-    )
-    (property "Value" "+3V3" (at 27.94 119.38 0)
-      (effects (font (size 1.27 1.27)))
-    )
-    (property "Footprint" "" (at 27.94 123.19 0)
-      (effects (font (size 1.27 1.27)) hide)
-    )
-    (property "Datasheet" "" (at 27.94 123.19 0)
-      (effects (font (size 1.27 1.27)) hide)
-    )
-    (pin "1")
-    (instances
-      (project "autoharpie"
-        (path "/f22a88c4-866b-40a0-9fc2-96344be0ec71/99b052d6-7969-4dd2-91c7-8bd18b784c30"
-          (reference "#PWR036") (unit 1)
-        )
-      )
-    )
-  )
-  (symbol (lib_id "Regulator_Linear:AP2112K-1.8") (at 45.72 129.54 0) (unit 1)
-    (in_bom yes) (on_board yes) (dnp no) (fields_autoplaced)
-    (property "Reference" "U5" (at 45.72 120.65 0)
-      (effects (font (size 1.27 1.27)))
-    )
-    (property "Value" "AP2112K-1.8" (at 45.72 123.19 0)
-      (effects (font (size 1.27 1.27)))
-    )
-    (property "Footprint" "Package_TO_SOT_SMD:SOT-23-5" (at 45.72 121.285 0)
-      (effects (font (size 1.27 1.27)) hide)
-    )
-    (property "Datasheet" "https://www.diodes.com/assets/Datasheets/AP2112.pdf" (at 45.72 127 0)
-      (effects (font (size 1.27 1.27)) hide)
-    )
-    (pin "1")
-    (pin "2")
-    (pin "3")
-    (pin "4")
-    (pin "5")
-    (instances
-      (project "autoharpie"
-        (path "/f22a88c4-866b-40a0-9fc2-96344be0ec71/99b052d6-7969-4dd2-91c7-8bd18b784c30"
-          (reference "U5") (unit 1)
-        )
-      )
-    )
-  )
   (symbol (lib_id "Device:C") (at 73.66 105.41 0) (unit 1)
     (in_bom yes) (on_board yes) (dnp no) (fields_autoplaced)
@@
     )
   )
-  (symbol (lib_id "power:GND") (at 31.75 135.89 0) (unit 1)
-    (in_bom yes) (on_board yes) (dnp no) (fields_autoplaced)
-    (property "Reference" "#PWR038" (at 31.75 142.24 0)
-      (effects (font (size 1.27 1.27)) hide)
-    )
-    (property "Value" "GND" (at 31.75 140.97 0)
-      (effects (font (size 1.27 1.27)))
-    )
-    (property "Footprint" "" (at 31.75 135.89 0)
-      (effects (font (size 1.27 1.27)) hide)
-    )
-    (property "Datasheet" "" (at 31.75 135.89 0)
-      (effects (font (size 1.27 1.27)) hide)
-    )
-    (pin "1")
-    (instances
-      (project "autoharpie"
-        (path "/f22a88c4-866b-40a0-9fc2-96344be0ec71/99b052d6-7969-4dd2-91c7-8bd18b784c30"
-          (reference "#PWR038") (unit 1)
-        )
-      )
-    )
-  )
   (symbol (lib_id "power:GND") (at 73.66 109.22 0) (unit 1)
     (in_bom yes) (on_board yes) (dnp no) (fields_autoplaced)
@@
         (path "/f22a88c4-866b-40a0-9fc2-96344be0ec71/99b052d6-7969-4dd2-91c7-8bd18b784c30"
           (reference "#PWR033") (unit 1)
-        )
-      )
-    )
-  )
-  (symbol (lib_id "Device:C") (at 31.75 132.08 0) (unit 1)
-    (in_bom yes) (on_board yes) (dnp no) (fields_autoplaced)
-    (property "Reference" "C5" (at 35.56 131.445 0)
-      (effects (font (size 1.27 1.27)) (justify left))
-    )
-    (property "Value" "1u" (at 35.56 133.985 0)
-      (effects (font (size 1.27 1.27)) (justify left))
-    )
-    (property "Footprint" "Capacitor_SMD:C_0603_1608Metric" (at 32.7152 135.89 0)
-      (effects (font (size 1.27 1.27)) hide)
-    )
-    (property "Datasheet" "~" (at 31.75 132.08 0)
-      (effects (font (size 1.27 1.27)) hide)
-    )
-    (pin "1")
-    (pin "2")
-    (instances
-      (project "autoharpie"
-        (path "/f22a88c4-866b-40a0-9fc2-96344be0ec71/99b052d6-7969-4dd2-91c7-8bd18b784c30"
-          (reference "C5") (unit 1)
         )
       )
@@
     )
   )
-  (symbol (lib_id "power:GND") (at 58.42 135.89 0) (unit 1)
-    (in_bom yes) (on_board yes) (dnp no) (fields_autoplaced)
-    (property "Reference" "#PWR039" (at 58.42 142.24 0)
-      (effects (font (size 1.27 1.27)) hide)
-    )
-    (property "Value" "GND" (at 58.42 140.97 0)
-      (effects (font (size 1.27 1.27)))
-    )
-    (property "Footprint" "" (at 58.42 135.89 0)
-      (effects (font (size 1.27 1.27)) hide)
-    )
-    (property "Datasheet" "" (at 58.42 135.89 0)
-      (effects (font (size 1.27 1.27)) hide)
-    )
-    (pin "1")
-    (instances
-      (project "autoharpie"
-        (path "/f22a88c4-866b-40a0-9fc2-96344be0ec71/99b052d6-7969-4dd2-91c7-8bd18b784c30"
-          (reference "#PWR039") (unit 1)
-        )
-      )
-    )
-  )
-  (symbol (lib_id "Device:C") (at 58.42 132.08 0) (unit 1)
-    (in_bom yes) (on_board yes) (dnp no) (fields_autoplaced)
-    (property "Reference" "C6" (at 62.23 131.445 0)
-      (effects (font (size 1.27 1.27)) (justify left))
-    )
-    (property "Value" "1u" (at 62.23 133.985 0)
-      (effects (font (size 1.27 1.27)) (justify left))
-    )
-    (property "Footprint" "Capacitor_SMD:C_0603_1608Metric" (at 59.3852 135.89 0)
-      (effects (font (size 1.27 1.27)) hide)
-    )
-    (property "Datasheet" "~" (at 58.42 132.08 0)
-      (effects (font (size 1.27 1.27)) hide)
-    )
-    (pin "1")
-    (pin "2")
-    (instances
-      (project "autoharpie"
-        (path "/f22a88c4-866b-40a0-9fc2-96344be0ec71/99b052d6-7969-4dd2-91c7-8bd18b784c30"
-          (reference "C6") (unit 1)
-        )
-      )
-    )
-  )
   (symbol (lib_id "power:+5V") (at 104.14 99.06 0) (unit 1)
     (in_bom yes) (on_board yes) (dnp no) (fields_autoplaced)
@@
         )
       )
-    )
-  )
-  (symbol (lib_id "power:+1V8") (at 63.5 127 270) (unit 1)
-    (in_bom yes) (on_board yes) (dnp no) (fields_autoplaced)
-    (property "Reference" "#PWR037" (at 59.69 127 0)
-      (effects (font (size 1.27 1.27)) hide)
-    )
-    (property "Value" "+1V8" (at 67.31 127.635 90)
-      (effects (font (size 1.27 1.27)) (justify left))
-    )
-    (property "Footprint" "" (at 63.5 127 0)
-      (effects (font (size 1.27 1.27)) hide)
-    )
-    (property "Datasheet" "" (at 63.5 127 0)
-      (effects (font (size 1.27 1.27)) hide)
-    )
-    (pin "1")
-    (instances
-      (project "autoharpie"
-        (path "/f22a88c4-866b-40a0-9fc2-96344be0ec71/99b052d6-7969-4dd2-91c7-8bd18b784c30"
-          (reference "#PWR037") (unit 1)
-        )
-      )
