File: hw_sch/autoharpie/touchpad.kicad_sch (KiCad schematic)
At the start: 28 parts

Commit message: rev 0.1 pcb
Parts:
- removed TP1, TP10, TP11, TP12, TP13, TP14, TP15, TP16, TP17, TP18, TP19, TP2, TP20, TP21, TP22, TP23, TP24, TP25, TP26, TP27, TP28, TP3, TP4, TP5, TP6, TP7, TP8, TP9: TestPoint, TestPoint:TestPoint_Pad_D1.0mm, symbol Connector:TestPoint
- added CS1, CS10, CS100, CS101, CS102, CS103, CS104, CS105, CS106, CS107, CS108, CS109, CS11, CS110, CS111, CS112, CS113, CS114, CS115, CS116, CS117, CS118, CS119, CS12, CS120, CS121, CS122, CS123, CS124, CS125, CS126, CS127, CS128, CS129, CS13, CS130, CS131, CS132, CS133, CS134, CS135, CS136, CS137, CS138, CS139, CS14, CS140, CS141, CS142, CS143, CS144, CS145, CS146, CS147, CS148, CS149, CS15, CS150, CS16, CS17, CS18, CS19, CS2, CS20, CS21, CS22, CS23, CS24, CS25, CS26, CS27, CS28, CS29, CS3, CS30, CS31, CS32, CS33, CS34, CS35, CS36, CS37, CS38, CS39, CS4, CS40, CS41, CS42, CS43, CS44, CS45, CS46, CS47, CS48, CS49, CS5, CS50, CS51, CS52, CS53, CS54, CS55, CS56, CS57, CS58, CS59, CS6, CS60, CS61, CS62, CS63, CS64, CS65, CS66, CS67, CS68, CS69, CS7, CS70, CS71, CS72, CS73, CS74, CS75, CS76, CS77, CS78, CS79, CS8, CS80, CS81, CS82, CS83, CS84, CS85, CS86, CS87, CS88, CS89, CS9, CS90, CS91, CS92, CS93, CS94, CS95, CS96, CS97, CS98, CS99: ~, symbol captouch:Capacitive_Touch_Sensor
Connections:
- new net: CS123.3 (B), CS138.1 (T)
- new net: CS137.4 (R), CS138.2 (L)
- new net: CS138.4 (R), CS139.2 (L)
- new net: CS14.3 (B), CS29.1 (T)
- new net: CS28.4 (R), CS29.2 (L)
- new net: CS29.3 (B), CS44.1 (T)
- new net: CS29.4 (R), CS30.2 (L)
- new net: CS53.3 (B), CS68.1 (T)
- new net: CS67.4 (R), CS68.2 (L)
- new net: CS68.3 (B), CS83.1 (T)
- new net: CS68.4 (R), CS69.2 (L)
- new net: CS17.1 (T), CS2.3 (B)
- new net: CS16.4 (R), CS17.2 (L)
- new net: CS17.3 (B), CS32.1 (T)
- new net: CS17.4 (R), CS18.2 (L)
- new net: CS106.3 (B), CS121.1 (T)
- new net: CS121.3 (B), CS136.1 (T)
- new net: CS121.4 (R), CS122.2 (L)
- new net: CS63.3 (B), CS78.1 (T)
- new net: CS77.4 (R), CS78.2 (L)
- new net: CS78.3 (B), CS93.1 (T)
- new net: CS78.4 (R), CS79.2 (L)
- new net: CS16.3 (B), CS31.1 (T)
- new net: CS31.3 (B), CS46.1 (T)
- new net: CS31.4 (R), CS32.2 (L)
- new net: CS34.3 (B), CS49.1 (T)
- new net: CS48.4 (R), CS49.2 (L)
- new net: CS49.3 (B), CS64.1 (T)
- new net: CS49.4 (R), CS50.2 (L)
- new net: CS52.3 (B), CS67.1 (T)
- new net: CS66.4 (R), CS67.2 (L)
- new net: CS67.3 (B), CS82.1 (T)
- new net: CS103.3 (B), CS118.1 (T)
- new net: CS117.4 (R), CS118.2 (L)
- new net: CS118.3 (B), CS133.1 (T)
- new net: CS118.4 (R), CS119.2 (L)
- new net: CS2.4 (R), CS3.2 (L)
- new net: CS18.1 (T), CS3.3 (B)
- new net: CS3.4 (R), CS4.2 (L)
- new net: CS32.3 (B), CS47.1 (T)
- new net: CS46.4 (R), CS47.2 (L)
- new net: CS47.3 (B), CS62.1 (T)
- new net: CS47.4 (R), CS48.2 (L)
- new net: CS102.3 (B), CS117.1 (T)
- new net: CS116.4 (R), CS117.2 (L)
- new net: CS117.3 (B), CS132.1 (T)
- new net: CS5.4 (R), CS6.2 (L)
- new net: CS21.1 (T), CS6.3 (B)
- new net: CS6.4 (R), CS7.2 (L)
- new net: CS83.3 (B), CS98.1 (T)
- new net: CS97.4 (R), CS98.2 (L)
- new net: CS113.1 (T), CS98.3 (B)
- new net: CS98.4 (R), CS99.2 (L)
- new net: CS55.3 (B), CS70.1 (T)
- new net: CS69.4 (R), CS70.2 (L)
- new net: CS70.3 (B), CS85.1 (T)
- new net: CS70.4 (R), CS71.2 (L)
- new net: CS109.3 (B), CS124.1 (T)
- new net: CS123.4 (R), CS124.2 (L)
- new net: CS124.3 (B), CS139.1 (T)
- new net: CS124.4 (R), CS125.2 (L)
- new net: CS104.1 (T), CS89.3 (B)
- new net: CS103.4 (R), CS104.2 (L)
- new net: CS104.3 (B), CS119.1 (T)
- new net: CS104.4 (R), CS105.2 (L)
- new net: CS122.3 (B), CS137.1 (T)
- new net: CS136.4 (R), CS137.2 (L)
- new net: CS82.4 (R), CS83.2 (L)
- new net: CS83.4 (R), CS84.2 (L)
- new net: CS81.3 (B), CS96.1 (T)
- new net: CS95.4 (R), CS96.2 (L)
- new net: CS111.1 (T), CS96.3 (B)
- new net: CS96.4 (R), CS97.2 (L)
- new net: CS37.3 (B), CS52.1 (T)
- new net: CS51.4 (R), CS52.2 (L)
- new net: CS52.4 (R), CS53.2 (L)
- new net: CS20.3 (B), CS35.1 (T)
- new net: CS34.4 (R), CS35.2 (L)
- new net: CS35.3 (B), CS50.1 (T)
- new net: CS35.4 (R), CS36.2 (L)
- new net: CS112.4 (R), CS113.2 (L)
- new net: CS113.3 (B), CS128.1 (T)
- new net: CS113.4 (R), CS114.2 (L)
- new net: CS92.4 (R), CS93.2 (L)
- new net: CS108.1 (T), CS93.3 (B)
- new net: CS93.4 (R), CS94.2 (L)
- new net: CS23.3 (B), CS38.1 (T)
- new net: CS37.4 (R), CS38.2 (L)
- new net: CS38.3 (B), CS53.1 (T)
- new net: CS38.4 (R), CS39.2 (L)
- new net: CS132.3 (B), CS147.1 (T)
- new net: CS146.4 (R), CS147.2 (L)
- new net: CS147.4 (R), CS148.2 (L)
- new net: CS102.1 (T), CS87.3 (B)
- new net: CS101.4 (R), CS102.2 (L)
- new net: CS102.4 (R), CS103.2 (L)
- new net: CS21.3 (B), CS36.1 (T)
- new net: CS36.3 (B), CS51.1 (T)
- new net: CS36.4 (R), CS37.2 (L)
- new net: CS111.3 (B), CS126.1 (T)
- new net: CS125.4 (R), CS126.2 (L)
- new net: CS126.3 (B), CS141.1 (T)
- new net: CS126.4 (R), CS127.2 (L)
- new net: CS8.4 (R), CS9.2 (L)
- new net: CS24.1 (T), CS9.3 (B)
- new net: CS10.2 (L), CS9.4 (R)
- new net: CS127.4 (R), CS128.2 (L)
- new net: CS128.3 (B), CS143.1 (T)
- new net: CS128.4 (R), CS129.2 (L)
- new net: CS80.3 (B), CS95.1 (T)
- new net: CS94.4 (R), CS95.2 (L)
- new net: CS110.1 (T), CS95.3 (B)
- new net: CS14.4 (R), CS15.2 (L)
- new net: CS15.3 (B), CS30.1 (T)
- new net: CS120.3 (B), CS135.1 (T)
- new net: CS134.4 (R), CS135.2 (L)
- new net: CS135.3 (B), CS150.1 (T)
- new net: CS139.4 (R), CS140.2 (L)
- new net: CS73.3 (B), CS88.1 (T)
- new net: CS87.4 (R), CS88.2 (L)
- new net: CS103.1 (T), CS88.3 (B)
- new net: CS88.4 (R), CS89.2 (L)
- new net: CS125.3 (B), CS140.1 (T)
- new net: CS140.4 (R), CS141.2 (L)
- new net: CS59.3 (B), CS74.1 (T)
- new net: CS73.4 (R), CS74.2 (L)
- new net: CS74.3 (B), CS89.1 (T)
- new net: CS74.4 (R), CS75.2 (L)
- new net: CS22.3 (B), CS37.1 (T)
- new net: CS112.3 (B), CS127.1 (T)
- new net: CS127.3 (B), CS142.1 (T)
- new net: CS50.3 (B), CS65.1 (T)
- new net: CS50.4 (R), CS51.2 (L)
- new net: CS110.3 (B), CS125.1 (T)
- new net: CS26.3 (B), CS41.1 (T)
- new net: CS40.4 (R), CS41.2 (L)
- new net: CS41.3 (B), CS56.1 (T)
- new net: CS41.4 (R), CS42.2 (L)
- new net: CS10.3 (B), CS25.1 (T)
- new net: CS10.4 (R), CS11.2 (L)
- new net: CS114.1 (T), CS99.3 (B)
- new net: CS114.3 (B), CS129.1 (T)
- new net: CS114.4 (R), CS115.2 (L)
- new net: CS51.3 (B), CS66.1 (T)
- new net: CS129.3 (B), CS144.1 (T)
- new net: CS129.4 (R), CS130.2 (L)
- new net: CS64.3 (B), CS79.1 (T)
- new net: CS79.3 (B), CS94.1 (T)
- new net: CS79.4 (R), CS80.2 (L)
- new net: CS100.1 (T), CS85.3 (B)
- new net: CS100.2 (L), CS99.4 (R)
- new net: CS100.3 (B), CS115.1 (T)
- new net: CS100.4 (R), CS101.2 (L)
- new net: CS62.3 (B), CS77.1 (T)
- new net: CS76.4 (R), CS77.2 (L)
- new net: CS77.3 (B), CS92.1 (T)
- new net: CS11.3 (B), CS26.1 (T)
- new net: CS25.4 (R), CS26.2 (L)
- new net: CS26.4 (R), CS27.2 (L)
- new net: CS141.4 (R), CS142.2 (L)
- new net: CS25.3 (B), CS40.1 (T)
- new net: CS39.4 (R), CS40.2 (L)
- new net: CS40.3 (B), CS55.1 (T)
- new net: CS11.4 (R), CS12.2 (L)
- new net: CS132.4 (R), CS133.2 (L)
- new net: CS133.3 (B), CS148.1 (T)
- new net: CS133.4 (R), CS134.2 (L)
- new net: CS45.3 (B), CS60.1 (T)
- new net: CS59.4 (R), CS60.2 (L)
- new net: CS60.3 (B), CS75.1 (T)
- new net: CS116.3 (B), CS131.1 (T)
- new net: CS130.4 (R), CS131.2 (L)
- new net: CS131.3 (B), CS146.1 (T)
- new net: CS131.4 (R), CS132.2 (L)
- new net: CS81.4 (R), CS82.2 (L)
- new net: CS82.3 (B), CS97.1 (T)
- new net: CS101.3 (B), CS116.1 (T)
- new net: CS115.4 (R), CS116.2 (L)
- new net: CS13.3 (B), CS28.1 (T)
- new net: CS27.4 (R), CS28.2 (L)
- new net: CS28.3 (B), CS43.1 (T)
- new net: CS130.3 (B), CS145.1 (T)
- new net: CS144.4 (R), CS145.2 (L)
- new net: CS145.4 (R), CS146.2 (L)
- new net: CS91.4 (R), CS92.2 (L)
- new net: CS107.1 (T), CS92.3 (B)
- new net: CS42.4 (R), CS43.2 (L)
- new net: CS43.3 (B), CS58.1 (T)
- new net: CS43.4 (R), CS44.2 (L)
- new net: CS108.3 (B), CS123.1 (T)
- new net: CS122.4 (R), CS123.2 (L)
- new net: CS66.3 (B), CS81.1 (T)
- new net: CS80.4 (R), CS81.2 (L)
- new net: CS112.1 (T), CS97.3 (B)
- new net: CS111.4 (R), CS112.2 (L)
- new net: CS30.3 (B), CS45.1 (T)
- new net: CS32.4 (R), CS33.2 (L)
- new net: CS57.3 (B), CS72.1 (T)
- new net: CS71.4 (R), CS72.2 (L)
- new net: CS72.3 (B), CS87.1 (T)
- new net: CS72.4 (R), CS73.2 (L)
- new net: CS89.4 (R), CS90.2 (L)
- new net: CS19.3 (B), CS34.1 (T)
- new net: CS33.4 (R), CS34.2 (L)
- new net: CS148.4 (R), CS149.2 (L)
- new net: CS1.3 (B), CS16.1 (T)
- new net: CS55.4 (R), CS56.2 (L)
- new net: CS56.3 (B), CS71.1 (T)
- new net: CS56.4 (R), CS57.2 (L)
- new net: CS1.4 (R), CS2.2 (L)
- new net: CS42.3 (B), CS57.1 (T)
- new net: CS57.4 (R), CS58.2 (L)
- new net: CS134.3 (B), CS149.1 (T)
- new net: CS149.4 (R), CS150.2 (L)
- new net: CS105.3 (B), CS120.1 (T)
- new net: CS119.4 (R), CS120.2 (L)
- new net: CS86.4 (R), CS87.2 (L)
- new net: CS61.4 (R), CS62.2 (L)
- new net: CS62.4 (R), CS63.2 (L)
- new net: CS46.3 (B), CS61.1 (T)
- new net: CS61.3 (B), CS76.1 (T)
- new net: CS4.4 (R), CS5.2 (L)
- new net: CS20.1 (T), CS5.3 (B)
- new net: CS76.3 (B), CS91.1 (T)
- new net: CS63.4 (R), CS64.2 (L)
- new net: CS64.4 (R), CS65.2 (L)
- new net: CS23.1 (T), CS8.3 (B)
- new net: CS22.4 (R), CS23.2 (L)
- new net: CS23.4 (R), CS24.2 (L)
- new net: CS109.1 (T), CS94.3 (B)
- new net: CS58.3 (B), CS73.1 (T)
- new net: CS58.4 (R), CS59.2 (L)
- new net: CS19.1 (T), CS4.3 (B)
- new net: CS18.4 (R), CS19.2 (L)
- new net: CS19.4 (R), CS20.2 (L)
- new net: CS105.1 (T), CS90.3 (B)
- new net: CS107.3 (B), CS122.1 (T)
- new net: CS109.4 (R), CS110.2 (L)
- new net: CS110.4 (R), CS111.2 (L)
- new net: CS39.3 (B), CS54.1 (T)
- new net: CS53.4 (R), CS54.2 (L)
- new net: CS54.3 (B), CS69.1 (T)
- new net: CS54.4 (R), CS55.2 (L)
- new net: CS18.3 (B), CS33.1 (T)
- new net: CS84.3 (B), CS99.1 (T)
- new net: CS44.3 (B), CS59.1 (T)
- new net: CS101.1 (T), CS86.3 (B)
- new net: CS115.3 (B), CS130.1 (T)
- new net: CS24.3 (B), CS39.1 (T)
- new net: CS44.4 (R), CS45.2 (L)
- new net: CS65.3 (B), CS80.1 (T)
- new net: CS71.3 (B), CS86.1 (T)
- new net: CS85.4 (R), CS86.2 (L)
- new net: CS24.4 (R), CS25.2 (L)
- new net: CS142.4 (R), CS143.2 (L)
- new net: CS143.4 (R), CS144.2 (L)
- new net: CS33.3 (B), CS48.1 (T)
- new net: CS48.3 (B), CS63.1 (T)
- new net: CS65.4 (R), CS66.2 (L)
- new net: CS69.3 (B), CS84.1 (T)
- new net: CS84.4 (R), CS85.2 (L)
- new net: CS106.1 (T), CS91.3 (B)
- new net: CS106.4 (R), CS107.2 (L)
- new net: CS22.1 (T), CS7.3 (B)
- new net: CS7.4 (R), CS8.2 (L)
- new net: CS27.3 (B), CS42.1 (T)
- new net: CS21.4 (R), CS22.2 (L)
- new net: CS12.3 (B), CS27.1 (T)
- new net: CS12.4 (R), CS13.2 (L)
- new net: CS75.3 (B), CS90.1 (T)
- new net: CS13.4 (R), CS14.2 (L)
- new net: CS20.4 (R), CS21.2 (L)
- new net: CS119.3 (B), CS134.1 (T)
- new net: CS107.4 (R), CS108.2 (L)
- new net: CS108.4 (R), CS109.2 (L)
- new net RX0: CS1.2 (L)
- new net RX1: CS16.2 (L)
- new net RX2: CS31.2 (L)
- new net RX3: CS46.2 (L)
- new net RX4: CS61.2 (L)
- new net RX5: CS76.2 (L)
- new net RX6: CS91.2 (L)
- new net RX7: CS106.2 (L)
- new net RX8: CS121.2 (L)
- new net RX9: CS136.2 (L)
- new net TX0: CS1.1 (T)
- new net TX1: CS2.1 (T)
- new net TX10: CS11.1 (T)
- new net TX11: CS12.1 (T)
- new net TX12: CS13.1 (T)
- new net TX13: CS14.1 (T)
- new net TX14: CS15.1 (T)
- new net TX2: CS3.1 (T)
- new net TX3: CS4.1 (T)
- new net TX4: CS5.1 (T)
- new net TX5: CS6.1 (T)
- new net TX6: CS7.1 (T)
- new net TX7: CS8.1 (T)
- new net TX8: CS9.1 (T)
- new net TX9: CS10.1 (T)
- no-connect marks 0 -> 25
Other:
- note added: "Rotated 90 degrees clockwise than design on board"

Commit message: ic fix atept
Parts:
- removed CS100, CS101, CS102, CS103, CS104, CS105, CS106, CS107, CS108, CS109, CS110, CS111, CS112, CS113, CS114, CS115, CS116, CS117, CS118, CS119, CS120, CS121, CS122, CS123, CS124, CS125, CS126, CS127, CS128, CS129, CS130, CS131, CS132, CS133, CS134, CS135, CS136, CS137, CS138, CS139, CS140, CS141, CS142, CS143, CS144, CS145, CS146, CS147, CS148, CS149, CS150, CS91, CS92, CS93, CS94, CS95, CS96, CS97, CS98, CS99: ~, symbol captouch:Capacitive_Touch_Sensor
Connections:
- no-connect marks 25 -> 21
