File: hw_sch/autoharpie/midi.kicad_sch (KiCad schematic)
At the start: 13 parts, among them J3 DIN-5_180degree, J4 DIN-5_180degree, J5 DIN-5_180degree, U3 7404, U4 6N138

Commit message: matrix, flattening
Parts:
- renumbered J3 to J2, J4 to J3, J5 to J4, R14 to R10, R8 to R4, R9 to R5, R10 to R6, R11 to R7, R12 to R8, R13 to R9, U3 to U2, U4 to U3

Commit message: keypad
Parts:
- removed D1: 1N4148, Diode_THT:D_DO-35_SOD27_P7.62mm_Horizontal, symbol Diode:1N4148
- removed R10: 1k, symbol Device:R
- removed R4, R7: 220, symbol Device:R
- removed R9: 470, symbol Device:R
- removed U2: 7404, symbol 74xx_IEEE:7404
- removed U3: 6N138, symbol Isolator:6N138
- added D3: 1N4148, Diode_THT:D_DO-35_SOD27_P7.62mm_Horizontal, symbol Diode:1N4148
- added R12: 470, Resistor_THT:R_Axial_DIN0204_L3.6mm_D1.6mm_P7.62mm_Horizontal, symbol Device:R
- added R14: 33, Resistor_THT:R_Axial_DIN0204_L3.6mm_D1.6mm_P7.62mm_Horizontal, symbol Device:R
- added R15: 10, Resistor_THT:R_Axial_DIN0207_L6.3mm_D2.5mm_P7.62mm_Horizontal, symbol Device:R
- added U5: H11L1, Package_DIP:DIP-6_W7.62mm, symbol Isolator:H11L1
- J3: renamed from J2; footprint (none) -> Eurocad:MIDI_DIN5
- J4: renamed from J3; footprint (none) -> Eurocad:MIDI_DIN5
- J5: renamed from J4; footprint (none) -> Eurocad:MIDI_DIN5
- R13: renamed from R6; footprint (none) -> Resistor_THT:R_Axial_DIN0204_L3.6mm_D1.6mm_P7.62mm_Horizontal
- R16: renamed from R5; value 220 -> 33; footprint (none) -> Resistor_THT:R_Axial_DIN0204_L3.6mm_D1.6mm_P7.62mm_Horizontal
- R17: renamed from R8; value 220 -> 10; footprint (none) -> Resistor_THT:R_Axial_DIN0204_L3.6mm_D1.6mm_P7.62mm_Horizontal
Connections:
- net +5V: now also R14.1; no longer R16.1
- net GND: now also U5.5; no longer J3.2, J4.2, J5.2
- net MIDI_IN: now also R12.2, R15.2, U5.4
- net MIDI_OUT: now also R17.2
- net at R13.2: now also D3.1 (K), U5.1
- net at J3.5: now also D3.2 (A), U5.2
- net at J4.5: now also R15.1
- net at J4.4: now also R14.2
- new net +3V3: R12.1, R16.1, U5.6
- no-connect marks 0 -> 9

Commit message: rev 0.1 pcb
Parts:
- removed J4: DIN-5_180degree, Eurocad:MIDI_DIN5, symbol Connector:DIN-5_180degree
- removed R14: 33, Resistor_THT:R_Axial_DIN0204_L3.6mm_D1.6mm_P7.62mm_Horizontal, symbol Device:R
- removed R15: 10, Resistor_THT:R_Axial_DIN0207_L6.3mm_D2.5mm_P7.62mm_Horizontal, symbol Device:R
- U5: footprint Package_DIP:DIP-6_W7.62mm -> Package_DIP:DIP-6_W7.62mm_Socket
- renumbered D3 to D14, J3 to J2, J5 to J3, R12 to R6, R13 to R7, R16 to R8, R17 to R9
Connections:
- no-connect marks 9 -> 6
Other:
- moved on the sheet: J3, R8, R9

Commit message: ic fix atept
Parts:
- added XU6: Conn_02x03_Counter_Clockwise, Package_DIP:DIP-6_W7.62mm_Socket, symbol Connector_Generic:Conn_02x03_Counter_Clockwise
- J2, J3: footprint Eurocad:MIDI_DIN5 -> KiCad:SDS50J
- renumbered U5 to U6
Connections:
- no-connect marks 6 -> 12
Changed lines of the file:
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@@
   )
   (no_connect (at 77.47 91.44))
+  (no_connect (at 133.35 67.31))
   (no_connect (at 50.8 41.91))
   (no_connect (at 62.23 91.44))
+  (no_connect (at 146.05 64.77))
   (no_connect (at 58.42 49.53))
   (no_connect (at 66.04 41.91))
+  (no_connect (at 133.35 64.77))
   (no_connect (at 69.85 99.06))
+  (no_connect (at 146.05 69.85))
+  (no_connect (at 133.35 69.85))
+  (no_connect (at 146.05 67.31))
   (wire (pts (xy 50.8 44.45) (xy 50.8 52.07))
     (stroke (width 0) (type default))
@@
   (symbol (lib_id "power:GND") (at 113.03 57.15 0) (unit 1)
     (in_bom yes) (on_board yes) (dnp no) (fields_autoplaced)
-    (property "Reference" "#PWR039" (at 113.03 63.5 0)
+    (property "Reference" "#PWR041" (at 113.03 63.5 0)
       (effects (font (size 1.27 1.27)) hide)
     )
@@
       (project "autoharpie"
         (path "/f22a88c4-866b-40a0-9fc2-96344be0ec71/27ed800e-6367-4383-9a1e-f16e4f370da3"
-          (reference "#PWR039") (unit 1)
+          (reference "#PWR041") (unit 1)
         )
       )
@@
   (symbol (lib_id "power:+3V3") (at 50.8 74.93 0) (unit 1)
     (in_bom yes) (on_board yes) (dnp no) (fields_autoplaced)
-    (property "Reference" "#PWR040" (at 50.8 78.74 0)
+    (property "Reference" "#PWR042" (at 50.8 78.74 0)
       (effects (font (size 1.27 1.27)) hide)
     )
@@
       (project "autoharpie"
         (path "/f22a88c4-866b-40a0-9fc2-96344be0ec71/27ed800e-6367-4383-9a1e-f16e4f370da3"
-          (reference "#PWR040") (unit 1)
+          (reference "#PWR042") (unit 1)
         )
       )
@@
   (symbol (lib_id "Isolator:H11L1") (at 113.03 46.99 0) (unit 1)
     (in_bom yes) (on_board yes) (dnp no) (fields_autoplaced)
-    (property "Reference" "U5" (at 123.19 43.8151 0)
+    (property "Reference" "U6" (at 123.19 43.8151 0)
       (effects (font (size 1.27 1.27)))
     )
@@
       (project "autoharpie"
         (path "/f22a88c4-866b-40a0-9fc2-96344be0ec71/27ed800e-6367-4383-9a1e-f16e4f370da3"
-          (reference "U5") (unit 1)
+          (reference "U6") (unit 1)
         )
       )
@@
       (effects (font (size 1.27 1.27)))
     )
-    (property "Footprint" "Eurocad:MIDI_DIN5" (at 58.42 41.91 0)
-      (effects (font (size 1.27 1.27)))
+    (property "Footprint" "KiCad:SDS50J" (at 58.42 41.91 0)
+      (effects (font (size 1.27 1.27)) hide)
     )
     (property "Datasheet" "http://www.mouser.com/ds/2/18/40_c091_abd_e-75918.pdf" (at 58.42 41.91 0)
@@
   (symbol (lib_id "power:+3V3") (at 113.03 29.21 0) (unit 1)
     (in_bom yes) (on_board yes) (dnp no) (fields_autoplaced)
-    (property "Reference" "#PWR038" (at 113.03 33.02 0)
+    (property "Reference" "#PWR040" (at 113.03 33.02 0)
       (effects (font (size 1.27 1.27)) hide)
     )
@@
       (project "autoharpie"
         (path "/f22a88c4-866b-40a0-9fc2-96344be0ec71/27ed800e-6367-4383-9a1e-f16e4f370da3"
-          (reference "#PWR038") (unit 1)
+          (reference "#PWR040") (unit 1)
         )
       )
@@
   )
   (symbol (lib_id "Device:R") (at 76.2 44.45 90) (unit 1)
-    (in_bom yes) (on_board yes) (dnp no) (fields_autoplaced)
+    (in_bom yes) (on_board yes) (dnp no)
     (property "Reference" "R7" (at 76.2 39.37 90)
       (effects (font (size 1.27 1.27)))
@@
       (effects (font (size 1.27 1.27)))
     )
-    (property "Footprint" "Resistor_THT:R_Axial_DIN0204_L3.6mm_D1.6mm_P7.62mm_Horizontal" (at 76.2 46.228 90)
+    (property "Footprint" "Resistor_THT:R_Axial_DIN0204_L3.6mm_D1.6mm_P7.62mm_Horizontal" (at 76.2 40.64 90)
       (effects (font (size 1.27 1.27)))
     )
@@
       (effects (font (size 1.27 1.27)))
     )
-    (property "Footprint" "Eurocad:MIDI_DIN5" (at 69.85 91.44 0)
+    (property "Footprint" "KiCad:SDS50J" (at 69.85 91.44 0)
       (effects (font (size 1.27 1.27)) hide)
     )
@@
         )
       )
+    )
+  )
+  (symbol (lib_id "Connector_Generic:Conn_02x03_Counter_Clockwise") (at 140.97 67.31 0) (mirror y) (unit 1)
+    (in_bom yes) (on_board no) (dnp no)
+    (property "Reference" "XU6" (at 139.7 59.69 0)
+      (effects (font (size 1.27 1.27)))
+    )
+    (property "Value" "Conn_02x03_Counter_Clockwise" (at 139.7 62.23 0)
+      (effects (font (size 1.27 1.27)))
+    )
+    (property "Footprint" "Package_DIP:DIP-6_W7.62mm_Socket" (at 140.97 67.31 0)
+      (effects (font (size 1.27 1.27)) hide)
+    )
+    (property "Datasheet" "~" (at 140.97 67.31 0)
+      (effects (font (size 1.27 1.27)) hide)
+    )
+    (pin "1")
+    (pin "2")
+    (pin "3")
+    (pin "4")
+    (pin "5")
+    (pin "6")
+    (instances
+      (project "autoharpie"
+        (path "/f22a88c4-866b-40a0-9fc2-96344be0ec71/27ed800e-6367-4383-9a1e-f16e4f370da3"
+          (reference "XU6") (unit 1)
+        )
+      )

Commit message: new icc
Parts:
- renumbered XU6 to XU3
Changed lines of the file:
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@@
   (symbol (lib_id "power:GND") (at 113.03 57.15 0) (unit 1)
     (in_bom yes) (on_board yes) (dnp no) (fields_autoplaced)
-    (property "Reference" "#PWR041" (at 113.03 63.5 0)
+    (property "Reference" "#PWR042" (at 113.03 63.5 0)
       (effects (font (size 1.27 1.27)) hide)
     )
@@
       (project "autoharpie"
         (path "/f22a88c4-866b-40a0-9fc2-96344be0ec71/27ed800e-6367-4383-9a1e-f16e4f370da3"
-          (reference "#PWR041") (unit 1)
+          (reference "#PWR042") (unit 1)
         )
       )
@@
   (symbol (lib_id "power:+3V3") (at 50.8 74.93 0) (unit 1)
     (in_bom yes) (on_board yes) (dnp no) (fields_autoplaced)
-    (property "Reference" "#PWR042" (at 50.8 78.74 0)
+    (property "Reference" "#PWR043" (at 50.8 78.74 0)
       (effects (font (size 1.27 1.27)) hide)
     )
@@
       (project "autoharpie"
         (path "/f22a88c4-866b-40a0-9fc2-96344be0ec71/27ed800e-6367-4383-9a1e-f16e4f370da3"
-          (reference "#PWR042") (unit 1)
+          (reference "#PWR043") (unit 1)
         )
       )
@@
   (symbol (lib_id "power:+3V3") (at 113.03 29.21 0) (unit 1)
     (in_bom yes) (on_board yes) (dnp no) (fields_autoplaced)
-    (property "Reference" "#PWR040" (at 113.03 33.02 0)
+    (property "Reference" "#PWR041" (at 113.03 33.02 0)
       (effects (font (size 1.27 1.27)) hide)
     )
@@
       (project "autoharpie"
         (path "/f22a88c4-866b-40a0-9fc2-96344be0ec71/27ed800e-6367-4383-9a1e-f16e4f370da3"
-          (reference "#PWR040") (unit 1)
+          (reference "#PWR041") (unit 1)
         )
       )
@@
   (symbol (lib_id "Connector_Generic:Conn_02x03_Counter_Clockwise") (at 140.97 67.31 0) (mirror y) (unit 1)
     (in_bom yes) (on_board no) (dnp no)
-    (property "Reference" "XU6" (at 139.7 59.69 0)
+    (property "Reference" "XU3" (at 139.7 59.69 0)
       (effects (font (size 1.27 1.27)))
     )
@@
       (project "autoharpie"
         (path "/f22a88c4-866b-40a0-9fc2-96344be0ec71/27ed800e-6367-4383-9a1e-f16e4f370da3"
-          (reference "XU6") (unit 1)
-        )
-      )
+          (reference "XU3") (unit 1)
+        )
+      )
