File: hw_sch/autoharpie/autoharpie.kicad_pcb (KiCad board)
At the start: 2 copper layers, 333 parts, among them J1 USB_C_Receptacle_USB2.0, J10 Conn_01x02_Pin, J11 AudioJack3_SwitchTR, J2 Conn_01x02_Pin, J3 DIN-5_180degree, J4 DIN-5_180degree, J5 DIN-5_180degree, J6 Conn_01x04_Socket, J7 Conn_01x04_Pin, J8 Conn_01x25_Socket, J9 AudioJack3_SwitchTR, SW1 SW_Push, SW10 SW_Push_45deg, SW11 SW_Push_45deg, SW12 SW_Push_45deg, SW13 SW_Push_45deg, SW14 SW_Push_45deg, SW15 SW_Push_45deg, SW16 SW_Push_45deg, SW17 SW_Push_45deg, SW18 SW_Push_45deg, SW19 SW_Push_45deg, SW2 SW_Push, SW20 SW_Push_45deg, SW21 SW_Push_45deg, SW22 SW_Push_45deg, SW23 SW_Push_45deg, SW24 SW_Push_45deg, SW25 SW_Push_45deg, SW26 SW_Push_45deg, SW27 SW_Push_45deg, SW28 SW_Push_45deg, SW29 SW_Push_45deg, SW3 RotaryEncoder_Switch, SW30 SW_Push_45deg, SW31 SW_Push_45deg, SW32 SW_Push_45deg, SW33 SW_Push_45deg, SW34 SW_Push_45deg, SW35 SW_Push_45deg, SW36 SW_Push_45deg, SW37 SW_Push_45deg, SW38 SW_Push_45deg, SW39 SW_Push_45deg, SW4 SW_Push_45deg, SW40 SW_Push_45deg, SW41 SW_Push_45deg, SW42 SW_Push_45deg, SW43 SW_Push_45deg, SW44 SW_Push_45deg, SW45 SW_Push_45deg, SW46 SW_Push_45deg, SW47 SW_Push_45deg, SW48 SW_Push_45deg, SW49 SW_Push_45deg, SW5 SW_Push_45deg, SW50 SW_Push_45deg, SW51 SW_Push_45deg, SW52 SW_Push_45deg, SW53 SW_Push_45deg, SW54 SW_Push_45deg, SW55 SW_Push_45deg, SW56 SW_Push_45deg, SW57 SW_Push_45deg, SW58 SW_Push_45deg, SW59 SW_Push_45deg, SW6 SW_Push_45deg, SW60 SW_Push_45deg, SW61 SW_Push_45deg, SW62 SW_Push_45deg, SW63 SW_Push_45deg, SW64 SW_Push_45deg, SW65 SW_Push_45deg, SW66 SW_Push_45deg, SW67 SW_Push_45deg, SW68 SW_Push_45deg, SW69 SW_Push_45deg, SW7 SW_Push_45deg, SW70 SW_Push_45deg, SW71 SW_Push_45deg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

Commit message: rev 0.1 pcb
Parts:
- removed C39: 22p, Capacitor_SMD:C_0402_1005Metric
- removed C40, C41, C42, C43, C44, C45, C46, C47, C48, C57, C58, C59, C60, C61, C62, C63, C64, C65, C66, C67, C68, C69, C70, C71, C72, C73, C74, C75, C76, C77, C78, C79: 0.1u, Capacitor_SMD:C_0402_1005Metric
- removed C7: 100n, Capacitor_SMD:C_0402_1005Metric
- removed D111, D112, D113, D114, D115, D80, D81, D82, D83, D84, D85, D86: SK6812MINI, LED_SMD:LED_SK6812MINI_PLCC4_3.5x3.5mm_P1.75mm
- removed D15, D16, D17, D18, D19, D20, D21, D22, D23, D24, D25, D26, D27, D28, D29, D30, D31, D32, D33, D34, D35, D36, D37, D38, D39, D40, D41, D42, D43, D44, D45, D46, D47, D48, D49, D50, D51, D52, D53, D54, D55, D56, D57, D58, D59, D60, D61, D62, D63, D64, D65, D66, D67, D68, D69, D70, D71, D72, D73, D74, D75, D76, D77, D78: 1N4148, Diode_THT:D_DO-35_SOD27_P7.62mm_Horizontal
- removed D79: LED, LED_SMD:LED_0402_1005Metric
- removed FB1: 120R, Ferrite_THT:LairdTech_28C0236-0JW-10
- removed J10: Conn_01x02_Pin, Connector_PinSocket_2.54mm:PinSocket_1x02_P2.54mm_Vertical
- removed J11, J9: AudioJack3_SwitchTR, Connector_Audio:Jack_3.5mm_CUI_SJ1-3535NG_Horizontal_CircularHoles
- removed L1: 2u2, Inductor_SMD:L_0805_2012Metric
- removed R15: 10, Resistor_THT:R_Axial_DIN0207_L6.3mm_D2.5mm_P7.62mm_Horizontal
- removed R16: 33, Resistor_THT:R_Axial_DIN0204_L3.6mm_D1.6mm_P7.62mm_Horizontal
- removed R17: 10, Resistor_THT:R_Axial_DIN0204_L3.6mm_D1.6mm_P7.62mm_Horizontal
- removed R18, R19, R20, R21, R22, R23, R24, R25, R34: 470, Resistor_THT:R_Axial_DIN0204_L3.6mm_D1.6mm_P7.62mm_Horizontal
- removed R26, R28, R30, R31, R32: 10k, Resistor_THT:R_Axial_DIN0204_L3.6mm_D1.6mm_P7.62mm_Horizontal
- removed R27, R29, R33: 330, Resistor_THT:R_Axial_DIN0204_L3.6mm_D1.6mm_P7.62mm_Horizontal
- removed R35: 47k, Resistor_THT:R_Axial_DIN0204_L3.6mm_D1.6mm_P7.62mm_Horizontal
- removed R36, R37: 1k, Resistor_THT:R_Axial_DIN0204_L3.6mm_D1.6mm_P7.62mm_Horizontal
- removed SW62, SW63, SW64, SW65, SW66, SW67, SW68, SW69, SW70, SW71, SW72, SW73, SW75: SW_Push_45deg, Button_Switch_THT:SW_PUSH_6mm_H4.3mm
- removed SW76: SW_Push, Button_Switch_SMD:SW_Push_SPST_NO_Alps_SKRK
- removed Y1: 16MHz, Crystal:Crystal_SMD_3225-4Pin_3.2x2.5mm
- removed Y2: 32.768KHz, Crystal:Crystal_SMD_2012-2Pin_2.0x1.2mm
- added H5: M2, MountingHole:MountingHole_2.2mm_M2, F.Cu at (136.5, 15.5)
- added H6: M2, MountingHole:MountingHole_2.2mm_M2, F.Cu at (16.2, 25.1)
- added H7: M2, MountingHole:MountingHole_2.2mm_M2, F.Cu at (108.4, 51.7)
- added H8: M2, MountingHole:MountingHole_2.2mm_M2, F.Cu at (105.4, 99.2)
- added U8: NCP1117-5.0_TO252, Package_TO_SOT_SMD:TO-252-2, F.Cu at (156.7, 28.8)
- C1, C10, C12, C13, C14, C15, C8: value 100n -> 0.1u
- C11, C4, C5, C6, C9: value 100n -> 1u; footprint Capacitor_SMD:C_0402_1005Metric -> Capacitor_SMD:C_0603_1608Metric
- C16: value 4.7u -> 0.1u; footprint Capacitor_SMD:C_0603_1608Metric -> Capacitor_SMD:C_0402_1005Metric
- C17, C18: value 15p -> 0.1u
- C19: value 2.2u -> 0.1u; footprint Capacitor_SMD:C_0603_1608Metric -> Capacitor_SMD:C_0402_1005Metric
- C2, C20, C21, C22, C23, C34: value 1u -> 0.1u
- C24, C25: value 47u -> 0.1u; footprint Capacitor_SMD:C_0805_2012Metric -> Capacitor_SMD:C_0402_1005Metric
- C26, C28, C33: value 1n -> 0.1u
- C3: footprint Capacitor_SMD:C_0402_1005Metric -> Capacitor_SMD:C_0603_1608Metric
- C35: value 10u -> 0.1u; footprint Capacitor_SMD:C_0603_1608Metric -> Capacitor_SMD:C_0402_1005Metric
- C37: value 1000n -> 0.1u
- C38: value 22p -> 1u; footprint Capacitor_SMD:C_0402_1005Metric -> Capacitor_SMD:C_0603_1608Metric
- C52, C53: value 0.1u -> 220u; footprint Capacitor_SMD:C_0402_1005Metric -> Capacitor_THT:C_Disc_D7.0mm_W2.5mm_P5.00mm
- C54, C55: value 0.1u -> 1u; footprint Capacitor_SMD:C_0402_1005Metric -> Capacitor_THT:C_Disc_D7.0mm_W2.5mm_P5.00mm
- D1, D2: value PMEG2010AEH -> 1N4148; footprint Diode_SMD:D_SOD-123F -> Diode_THT:D_DO-35_SOD27_P7.62mm_Horizontal
- D100, D101, D102, D103, D104, D105, D106, D107, D108, D109, D110, D87, D88, D89, D90, D91, D92, D93, D94, D95, D96, D97, D98, D99: value SK6812MINI -> WS2812B; footprint LED_SMD:LED_SK6812MINI_PLCC4_3.5x3.5mm_P1.75mm -> LED_SMD:LED_WS2812B_PLCC4_5.0x5.0mm_P3.2mm
- D13: value 1N4148 -> PMEG2010AEH; footprint Diode_THT:D_DO-35_SOD27_P7.62mm_Horizontal -> Diode_SMD:D_SOD-123F
- D4, D5, D6: value LED -> 1N4148; footprint LED_THT:LED_D3.0mm -> Diode_THT:D_DO-35_SOD27_P7.62mm_Horizontal
- J1: value USB_C_Receptacle_USB2.0 -> Conn_01x02_Pin; footprint Connector_USB:USB_C_Receptacle_GCT_USB4135-GF-A_6P_TopMnt_Horizontal -> Connector_JST:JST_PH_S2B-PH-K_1x02_P2.00mm_Horizontal
- J2: value Conn_01x02_Pin -> DIN-5_180degree; footprint Connector_JST:JST_PH_B2B-PH-K_1x02_P2.00mm_Vertical -> Eurocad:MIDI_DIN5
- J4: value DIN-5_180degree -> Conn_01x04_Socket; footprint Eurocad:MIDI_DIN5 -> Connector_PinSocket_2.54mm:PinSocket_1x04_P2.54mm_Vertical
- J5: value DIN-5_180degree -> Conn_01x06_Pin; footprint Eurocad:MIDI_DIN5 -> Connector_PinHeader_2.54mm:PinHeader_1x06_P2.54mm_Vertical
- J6: value Conn_01x04_Socket -> AudioJack3_SwitchTR; footprint Connector_PinSocket_2.54mm:PinSocket_1x04_P2.54mm_Vertical -> Connector_Audio:Jack_3.5mm_CUI_SJ1-3535NG_Horizontal_CircularHoles
- J7: value Conn_01x04_Pin -> Conn_01x02_Pin; footprint Connector_PinHeader_2.54mm:PinHeader_1x04_P2.54mm_Vertical -> Connector_JST:JST_PH_S2B-PH-K_1x02_P2.00mm_Horizontal
- J8: value Conn_01x25_Socket -> AudioJack3_SwitchTR; footprint Connector_PinSocket_2.54mm:PinSocket_1x25_P2.54mm_Vertical -> Connector_Audio:Jack_3.5mm_CUI_SJ1-3535NG_Horizontal_CircularHoles
- R1: value 10k -> 20k
- R10, R11, R4: value 100k -> 10k
- R12: value 470 -> 10k
- R13: value 220 -> 1k
- R14: value 33 -> 1k
- R2: value 10k -> 4.7k
- R3: value 1k -> 4.7k
- R5: value 5.1k -> 4.7k
- R6: value 5.1k -> 470
- R7: value 10 -> 220
- R8: value 10 -> 33
- R9: value 100k -> 10
- SW1: value SW_Push -> RotaryEncoder_Switch; footprint Button_Switch_THT:SW_PUSH_6mm_H4.3mm -> Rotary_Encoder:RotaryEncoder_Alps_EC11E-Switch_Vertical_H20mm
- SW10, SW11, SW12, SW13, SW14, SW15, SW16, SW17, SW18, SW19, SW20, SW21, SW22, SW23, SW24, SW25, SW26, SW27, SW28, SW29, SW30, SW31, SW32, SW33, SW34, SW35, SW36, SW37, SW38, SW39, SW4, SW40, SW41, SW42, SW43, SW44, SW45, SW46, SW47, SW48, SW49, SW5, SW50, SW51, SW52, SW53, SW54, SW55, SW56, SW57, SW58, SW59, SW6, SW60, SW61, SW7, SW74, SW8, SW9: value SW_Push_45deg -> SW_Push; footprint Button_Switch_THT:SW_PUSH_6mm_H4.3mm -> Button_Switch_THT:SW_PUSH_6mm
- SW2: footprint Button_Switch_THT:SW_PUSH_6mm_H4.3mm -> Button_Switch_THT:SW_PUSH_6mm
- SW3: value RotaryEncoder_Switch -> SW_Push; footprint Rotary_Encoder:RotaryEncoder_Alps_EC11E-Switch_Vertical_H20mm -> Button_Switch_THT:SW_PUSH_6mm
- U1: value STM32F446RCTx -> 74HC595; footprint Package_QFP:LQFP-64_10x10mm_P0.5mm -> Package_DIP:DIP-16_W7.62mm_Socket
- U2: value NCV8114ASN180T1G -> YAAJ_WeAct_BlackPill_Part_Like; footprint Package_TO_SOT_SMD:TSOT-23-5 -> Footprints:YAAJ_WeAct_BlackPill_2
- U3: value AP2112K-3.3 -> 74HC595; footprint Package_TO_SOT_SMD:SOT-23-5 -> Package_DIP:DIP-16_W7.62mm_Socket
- U4: value RT6150B-33GQW -> AP2112K-1.8; footprint footprints:RT6150B-33GQW -> Package_TO_SOT_SMD:SOT-23-5
- U5: footprint Package_DIP:DIP-6_W7.62mm -> Package_DIP:DIP-6_W7.62mm_Socket
- U6: value MSP430FR2633IDAR -> IQS550-BL-QNR; footprint footprints3:MSP430FR2633IDAR -> footprints5:IQS550-BL-QNR
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Connections:
- C1 pad 1: +3.3VA -> +3V3
- C10 pad 1: +3V3 -> /Keybed/REG
- C11 pad 1: +3V3 -> /Keybed/REG
- C12 pad 1: +3V3 -> /Controller/TOUCH_RESET
- C12 pad 2: GND -> Net-(U6-NRST)
- C17 pad 1: GND -> +3V3
- C17 pad 2: /Controller/OSC_IN -> GND
- C18 pad 1: GND -> +3V3
- C18 pad 2: Net-(C18-Pad2) -> GND
- C19 pad 1: /Controller/VCAP0 -> +3V3
- C2 pad 1: +3.3VA -> +3V3
- C20 pad 1: +1V8 -> +3V3
- C21 pad 1: +BATT -> +3V3
- C22 pad 1: +BATT -> +3V3
- C23 pad 1: 3V3_AUDIO -> +3V3
- C25 pad 1: +BATT -> +3V3
- C26 pad 1: /Display/FRONT_SHIFT_LED -> +3V3
- C27 pad 1: /Display/FRONT_SHIFT_SW -> +3V3
- C28 pad 1: /Controller/PWR_LED -> +3V3
- C29 pad 1: /Controller/PWR_SW -> +3V3
- C30 pad 1: /Controller/FRONT_ROT_SW -> +3V3
- C31 pad 1: /Controller/FRONT_ROT_A -> +3V3
- C32 pad 1: /Controller/FRONT_ROT_B -> +3V3
- C33 pad 1: /Display/FRONT_UTILITY_LED -> +3V3
- C34 pad 1: /Keybed/VREG -> +3V3
- C37 pad 1: /Keybed/SPY_SWD_RST -> +3V3
- C37 pad 2: /Keybed/RESET -> GND
- C38 pad 1: /Keybed/XIN -> +3V3
- C4 pad 1: +3V3 -> +1V8
- C49 pad 1: +5V -> +1V8
- C5 pad 1: +3V3 -> Net-(D13-K)
- C50 pad 1: +5V -> +3V3
- C51 pad 1: +5V -> +3V3
- C52 pad 1: +5V -> Net-(C52-Pad1)
- C52 pad 2: GND -> /Audio Interface/HP_R
- C53 pad 1: +5V -> Net-(C53-Pad1)
- C53 pad 2: GND -> /Audio Interface/HP_L
- C54 pad 1: +5V -> Net-(C54-Pad1)
- C54 pad 2: GND -> /Audio Interface/LO_R
- C55 pad 1: +5V -> Net-(C55-Pad1)
- C55 pad 2: GND -> /Audio Interface/LO_L
- C56 pad 1: +5V -> /Audio Interface/VAG
- C6 pad 1: +3V3 -> +BATT
- D1 pad 1: +BATT -> /Chord & Sequencer/C0
- D1 pad 2: Net-(D1-A) -> /Controller/A0
- D10 pad 1: /Chord & Sequencer/R0 -> /Chord & Sequencer/C9
- D10 pad 2: Net-(D10-A) -> /Controller/A9
- D100 pad 1: Net-(D100-DOUT) -> +3V3
- D100 pad 2: GND -> Net-(D100-DOUT)
- D100 pad 3: Net-(D100-DIN) -> GND
- D100 pad 4: +5V -> Net-(D100-DIN)
- D101 pad 1: Net-(D101-DOUT) -> +3V3
- D101 pad 2: GND -> Net-(D101-DOUT)
- D101 pad 3: Net-(D100-DOUT) -> GND
- D101 pad 4: +5V -> Net-(D100-DOUT)
- D102 pad 1: Net-(D102-DOUT) -> +3V3
- D102 pad 2: GND -> Net-(D102-DOUT)
- D102 pad 3: Net-(D101-DOUT) -> GND
- D102 pad 4: +5V -> Net-(D101-DOUT)
- D103 pad 1: unconnected-(D103-DOUT-Pad1) -> +3V3
- D103 pad 2: GND -> Net-(D103-DOUT)
- D103 pad 3: Net-(D102-DOUT) -> GND
- D103 pad 4: +5V -> Net-(D102-DOUT)
- D104 pad 1: Net-(D104-DOUT) -> +3V3
- D104 pad 2: GND -> Net-(D104-DOUT)
- D104 pad 3: /Chord & Sequencer/LED_DIN_FP -> GND
- D104 pad 4: +5V -> Net-(D103-DOUT)
- D105 pad 1: Net-(D105-DOUT) -> +3V3
- D105 pad 2: GND -> Net-(D105-DOUT)
- D105 pad 3: Net-(D104-DOUT) -> GND
- D105 pad 4: +5V -> Net-(D104-DOUT)
- D106 pad 1: Net-(D106-DOUT) -> +3V3
- D106 pad 2: GND -> Net-(D106-DOUT)
- D106 pad 3: Net-(D105-DOUT) -> GND
- D106 pad 4: +5V -> Net-(D105-DOUT)
- D107 pad 1: Net-(D107-DOUT) -> +3V3
- D107 pad 2: GND -> Net-(D107-DOUT)
- D107 pad 3: Net-(D106-DOUT) -> GND
- D107 pad 4: +5V -> Net-(D106-DOUT)
- D108 pad 1: Net-(D108-DOUT) -> +3V3
- D108 pad 2: GND -> Net-(D108-DOUT)
- D108 pad 3: Net-(D107-DOUT) -> GND
- D108 pad 4: +5V -> Net-(D107-DOUT)
- D109 pad 1: /Chord & Sequencer/Chord LEDs/DOUT-R0 -> +3V3
- D109 pad 2: GND -> Net-(D109-DOUT)
- D109 pad 3: Net-(D108-DOUT) -> GND
- D109 pad 4: +5V -> Net-(D108-DOUT)
- D11 pad 1: /Chord & Sequencer/R0 -> /Chord & Sequencer/C10
- D11 pad 2: Net-(D11-A) -> /Controller/A10
- D110 pad 1: Net-(D110-DOUT) -> +3V3
- D110 pad 2: GND -> unconnected-(D110-DOUT-Pad2)
- D110 pad 3: /Chord & Sequencer/Chord LEDs/DOUT-R0 -> GND
- D110 pad 4: +5V -> Net-(D109-DOUT)
- D12 pad 1: /Chord & Sequencer/R0 -> /Chord & Sequencer/C11
- D12 pad 2: Net-(D12-A) -> /Controller/A11
- D13 pad 1: /Chord & Sequencer/R0 -> Net-(D13-K)
- D13 pad 2: Net-(D13-A) -> BATT_SENSE
- D14 pad 1: /Chord & Sequencer/R0 -> Net-(D14-K)
- D2 pad 1: +BATT -> /Chord & Sequencer/C1
- D2 pad 2: Net-(D2-A) -> /Controller/A1
- D3 pad 1: Net-(D3-K) -> /Chord & Sequencer/C2
- D3 pad 2: Net-(D3-A) -> /Controller/A2
- D4 pad 1: GND -> /Chord & Sequencer/C3
- D4 pad 2: Net-(D4-A) -> /Controller/A3
- D5 pad 1: GND -> /Chord & Sequencer/C4
- D5 pad 2: Net-(D5-A) -> /Controller/A4
- D6 pad 1: GND -> /Chord & Sequencer/C5
- D6 pad 2: Net-(D6-A) -> /Controller/A5
- D7 pad 1: /Chord & Sequencer/R0 -> /Chord & Sequencer/C6
- D7 pad 2: Net-(D7-A) -> /Controller/A6
- D8 pad 1: /Chord & Sequencer/R0 -> /Chord & Sequencer/C7
- D8 pad 2: Net-(D8-A) -> /Controller/A7
- D87 pad 1: Net-(D87-DOUT) -> +3V3
- D87 pad 2: GND -> Net-(D87-DOUT)
- D87 pad 3: Net-(D86-DOUT) -> GND
- D87 pad 4: +5V -> /Chord & Sequencer/LED_DIN
- D88 pad 1: Net-(D88-DOUT) -> +3V3
- D88 pad 2: GND -> Net-(D88-DOUT)
- D88 pad 3: Net-(D87-DOUT) -> GND
- D88 pad 4: +5V -> Net-(D87-DOUT)
- D89 pad 1: Net-(D89-DOUT) -> +3V3
- D89 pad 2: GND -> Net-(D89-DOUT)
- D89 pad 3: Net-(D88-DOUT) -> GND
- D89 pad 4: +5V -> Net-(D88-DOUT)
- D9 pad 1: /Chord & Sequencer/R0 -> /Chord & Sequencer/C8
- D9 pad 2: Net-(D9-A) -> /Controller/A8
- D90 pad 1: Net-(D90-DOUT) -> +3V3
- D90 pad 2: GND -> Net-(D90-DOUT)
- D90 pad 3: Net-(D89-DOUT) -> GND
- D90 pad 4: +5V -> Net-(D89-DOUT)
- D91 pad 1: /Chord & Sequencer/Sequencer LEDs/DOUT-R1 -> +3V3
- D91 pad 2: GND -> Net-(D91-DOUT)
- D91 pad 3: Net-(D90-DOUT) -> GND
- D91 pad 4: +5V -> Net-(D90-DOUT)
- D92 pad 1: Net-(D92-DOUT) -> +3V3
- D92 pad 2: GND -> Net-(D92-DOUT)
- D92 pad 3: /Chord & Sequencer/Sequencer LEDs/DOUT-R1 -> GND
- D92 pad 4: +5V -> Net-(D91-DOUT)
- D93 pad 1: Net-(D93-DOUT) -> +3V3
- D93 pad 2: GND -> Net-(D93-DOUT)
- D93 pad 3: Net-(D92-DOUT) -> GND
- D93 pad 4: +5V -> Net-(D92-DOUT)
- D94 pad 1: Net-(D94-DOUT) -> +3V3
- D94 pad 2: GND -> Net-(D94-DOUT)
- D94 pad 3: Net-(D93-DOUT) -> GND
- D94 pad 4: +5V -> Net-(D93-DOUT)
- D95 pad 1: Net-(D95-DOUT) -> +3V3
- D95 pad 2: GND -> Net-(D95-DOUT)
- D95 pad 3: Net-(D94-DOUT) -> GND
- D95 pad 4: +5V -> Net-(D94-DOUT)
- D96 pad 1: Net-(D96-DOUT) -> +3V3
- D96 pad 2: GND -> Net-(D96-DOUT)
- D96 pad 3: Net-(D95-DOUT) -> GND
- D96 pad 4: +5V -> Net-(D95-DOUT)
- D97 pad 1: /Chord & Sequencer/Sequencer LEDs/DOUT-R2 -> +3V3
- D97 pad 2: GND -> Net-(D97-DOUT)
- D97 pad 3: Net-(D96-DOUT) -> GND
- D97 pad 4: +5V -> Net-(D96-DOUT)
- D98 pad 1: Net-(D98-DOUT) -> +3V3
- D98 pad 2: GND -> /Chord & Sequencer/LEDs/DOUT_R0
- D98 pad 3: /Chord & Sequencer/Sequencer LEDs/DOUT-R2 -> GND
- D98 pad 4: +5V -> Net-(D97-DOUT)
- D99 pad 1: Net-(D100-DIN) -> +3V3
- D99 pad 2: GND -> Net-(D100-DIN)
- D99 pad 3: Net-(D98-DOUT) -> GND
- D99 pad 4: +5V -> /Chord & Sequencer/LEDs/DOUT_R0
- J2 pad 1: Net-(D2-A) -> unconnected-(J2-Pad1)
- J2 pad 2: -BATT -> unconnected-(J2-Pad2)
- J3 pad 5: Net-(D3-A) -> Net-(J3-Pad5)
- J4 pad 1: unconnected-(J4-Pad1) -> GND
- J4 pad 2: unconnected-(J4-Pad2) -> +3V3
- J4 pad 3: unconnected-(J4-Pad3) -> /I2C_SDA
- J4 pad 4: Net-(J4-Pad4) -> /I2C_SCL
- J5 pad 1: unconnected-(J5-Pad1) -> +3V3
- J5 pad 2: unconnected-(J5-Pad2) -> GND
- J5 pad 3: unconnected-(J5-Pad3) -> /Keybed/PGRM
- J5 pad 4: Net-(J5-Pad4) -> /Keybed/SDA
- J5 pad 5: Net-(J5-Pad5) -> /Keybed/SCL
- J7 pad 1: GND -> /Audio Interface/HP_GND
- J7 pad 2: +3V3 -> Net-(J7-Pin_2)
- R1 pad 1: +BATT -> BATT_SENSE
- R1 pad 2: /Controller/BATT_ADC -> /Controller/BAT_SENSE
- R10 pad 1: Net-(U4-EN) -> +3V3
- R10 pad 2: +BATT -> /Controller/FRONT_ROT_A
- R11 pad 1: /USB Power/PS -> +3V3
- R11 pad 2: GND -> /Controller/FRONT_ROT_B
- R12 pad 2: /Controller/MIDI_RX -> /Controller/FRONT_ROT_SW
- R13 pad 1: Net-(J3-Pad4) -> Net-(J7-Pin_2)
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Routing:
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- added copper zone on F.Cu, net +BATT
- added copper zone on F.Cu, net /Keybed/RX0
- added copper zone on F.Cu, net /Keybed/RX1
- added copper zone on F.Cu, net /Keybed/RX2
- added copper zone on F.Cu, net /Keybed/RX3
- added copper zone on F.Cu, net /Keybed/RX4
- added copper zone on F.Cu, net /Keybed/RX5
- added copper zone on F.Cu, net /Keybed/TX0
- added copper zone on F.Cu, net /Keybed/TX1
- added copper zone on F.Cu, net /Keybed/TX10
- added copper zone on F.Cu, net /Keybed/TX11
- added copper zone on F.Cu, net /Keybed/TX12
- added copper zone on F.Cu, net /Keybed/TX13
- added copper zone on F.Cu, net /Keybed/TX14
- added copper zone on F.Cu, net /Keybed/TX2
- added copper zone on F.Cu, net /Keybed/TX3
- added copper zone on F.Cu, net /Keybed/TX4
- added copper zone on F.Cu, net /Keybed/TX5
- added copper zone on F.Cu, net /Keybed/TX6
- added copper zone on F.Cu, net /Keybed/TX7
- added copper zone on F.Cu, net /Keybed/TX8
- added copper zone on F.Cu, net /Keybed/TX9
- added copper zone on B.Cu, net GND
Other:
- board outline added: 190 x 150 mm
- board text added: "1/9 PG1"
- board text added: "2/10 PG2"
- board text added: "3/11 PG3"
- board text added: "4/12 PG4"
- board text added: "5/13 LAST"
- board text added: "6/14 COPY"
- board text added: "6/m6 9/m9 Fifth"
- board text added: "7/15 PASTE"
- board text added: "7/M7"
- board text added: "8/16 CONT"
- board text added: "A"
- board text added: "A#"
- board text added: "ARP AOPT."
- board text added: "AUTOHARPIE - STRUM SYNTHESIZER - REV 0.1"
- board text added: "B"
- board text added: "C"
- board text added: "C#"
- board text added: "CP/CUT PASTE"
- board text added: "D"
- board text added: "D#"
- board text added: "DEL"
- board text added: "Dimin Augmt Add9/2"
- board text added: "E"
- board text added: "F"
- board text added: "F#"
- board text added: "G"
- board text added: "G#"
- board text added: "HOLD HOPT."
- board text added: "KEY CUSTOM"
- board text added: "LINEOUT"
- board text added: "MODE"
- board text added: "Major Minor Su4/2"
- board text added: "PAGE"
- board text added: "PARAM"
- board text added: "PHONES"
- board text added: "POWER"
- board text added: "REC MODE"
- board text added: "SHIFT"
- board text added: "VOL PANIC!"
- board text added: "▶/◼ STOP"

Commit message: ic fix atept
Parts:
- removed C49, C50, C51, C56: 0.1u, Capacitor_SMD:C_0402_1005Metric
- removed C52, C53: 220u, Capacitor_THT:C_Disc_D7.0mm_W2.5mm_P5.00mm
- removed C54, C55: 1u, Capacitor_THT:C_Disc_D7.0mm_W2.5mm_P5.00mm
- removed D100, D101, D102, D103, D104, D105, D106, D107, D108, D109, D110, D87, D88, D89, D90, D91, D92, D93, D94, D95, D96, D97, D98, D99: WS2812B, LED_SMD:LED_WS2812B_PLCC4_5.0x5.0mm_P3.2mm
- removed SW74: SW_Push, Button_Switch_THT:SW_PUSH_6mm
- added C39: 0.1u, Capacitor_SMD:C_0402_1005Metric, F.Cu at (140.0, 40.8)
- added C40: 0.1u, Capacitor_SMD:C_0402_1005Metric, F.Cu at (137.6, 45.0)
- added C41: 1u, Capacitor_THT:C_Disc_D7.0mm_W2.5mm_P5.00mm, F.Cu at (138.7, 31.6)
- added C42: 1u, Capacitor_THT:C_Disc_D7.0mm_W2.5mm_P5.00mm, F.Cu at (135.0, 31.6)
- added C43: 0.1u, Capacitor_SMD:C_0402_1005Metric, F.Cu at (138.2, 39.3)
- added C7: 0.1u, Capacitor_SMD:C_0402_1005Metric, F.Cu at (136.6, 57.1)
- added D15: WS2812B, LED_SMD:LED_WS2812B_PLCC4_5.0x5.0mm_P3.2mm, F.Cu at (18.4, 81.1)
- added D16: WS2812B, LED_SMD:LED_WS2812B_PLCC4_5.0x5.0mm_P3.2mm, F.Cu at (30.0, 81.1)
- added D17: WS2812B, LED_SMD:LED_WS2812B_PLCC4_5.0x5.0mm_P3.2mm, F.Cu at (41.7, 81.1)
- added D18: WS2812B, LED_SMD:LED_WS2812B_PLCC4_5.0x5.0mm_P3.2mm, F.Cu at (53.3, 81.1)
- added D19: WS2812B, LED_SMD:LED_WS2812B_PLCC4_5.0x5.0mm_P3.2mm, F.Cu at (65.0, 81.1)
- added D20: WS2812B, LED_SMD:LED_WS2812B_PLCC4_5.0x5.0mm_P3.2mm, F.Cu at (76.6, 81.1)
- added D21: WS2812B, LED_SMD:LED_WS2812B_PLCC4_5.0x5.0mm_P3.2mm, F.Cu at (88.3, 81.1)
- added D22: WS2812B, LED_SMD:LED_WS2812B_PLCC4_5.0x5.0mm_P3.2mm, F.Cu at (99.9, 81.1)
- added D23: WS2812B, LED_SMD:LED_WS2812B_PLCC4_5.0x5.0mm_P3.2mm, F.Cu at (111.6, 81.1)
- added D24: WS2812B, LED_SMD:LED_WS2812B_PLCC4_5.0x5.0mm_P3.2mm, F.Cu at (123.2, 81.1)
- added D25: WS2812B, LED_SMD:LED_WS2812B_PLCC4_5.0x5.0mm_P3.2mm, F.Cu at (134.9, 81.1)
- added D26: WS2812B, LED_SMD:LED_WS2812B_PLCC4_5.0x5.0mm_P3.2mm, F.Cu at (146.5, 81.1)
- added D27: WS2812B, LED_SMD:LED_WS2812B_PLCC4_5.0x5.0mm_P3.2mm, F.Cu at (146.5, 134.6)
- added D28: WS2812B, LED_SMD:LED_WS2812B_PLCC4_5.0x5.0mm_P3.2mm, F.Cu at (134.8, 134.6)
- added D29: WS2812B, LED_SMD:LED_WS2812B_PLCC4_5.0x5.0mm_P3.2mm, F.Cu at (123.2, 134.6)
- added D30: WS2812B, LED_SMD:LED_WS2812B_PLCC4_5.0x5.0mm_P3.2mm, F.Cu at (111.6, 134.6)
- added D31: WS2812B, LED_SMD:LED_WS2812B_PLCC4_5.0x5.0mm_P3.2mm, F.Cu at (100.0, 134.6)
- added D32: WS2812B, LED_SMD:LED_WS2812B_PLCC4_5.0x5.0mm_P3.2mm, F.Cu at (88.3, 134.6)
- added D33: WS2812B, LED_SMD:LED_WS2812B_PLCC4_5.0x5.0mm_P3.2mm, F.Cu at (76.7, 134.6)
- added D34: WS2812B, LED_SMD:LED_WS2812B_PLCC4_5.0x5.0mm_P3.2mm, F.Cu at (65.1, 134.6)
- added D35: WS2812B, LED_SMD:LED_WS2812B_PLCC4_5.0x5.0mm_P3.2mm, F.Cu at (53.4, 134.6)
- added D36: WS2812B, LED_SMD:LED_WS2812B_PLCC4_5.0x5.0mm_P3.2mm, F.Cu at (41.8, 134.6)
- added D37: WS2812B, LED_SMD:LED_WS2812B_PLCC4_5.0x5.0mm_P3.2mm, F.Cu at (30.2, 134.6)
- added D38: WS2812B, LED_SMD:LED_WS2812B_PLCC4_5.0x5.0mm_P3.2mm, F.Cu at (18.6, 134.6)
- added H9: M2, MountingHole:MountingHole_2.2mm_M2_DIN965_Pad, F.Cu at (22.0, 99.6)
- added Q1: 2N7000, Package_TO_SOT_THT:TO-92_Inline, F.Cu at (28.2, 45.4)
- added R13: 10k, Resistor_THT:R_Axial_DIN0204_L3.6mm_D1.6mm_P7.62mm_Horizontal, F.Cu at (30.9, 49.2)
- added R14: 10k, Resistor_THT:R_Axial_DIN0204_L3.6mm_D1.6mm_P7.62mm_Horizontal, F.Cu at (22.5, 41.9)
- added SW62: SW_Push, Button_Switch_THT:SW_PUSH_6mm, F.Cu at (143.5, 140.6)
- C10, C12, C8: value 0.1u -> 1u; footprint Capacitor_SMD:C_0402_1005Metric -> Capacitor_SMD:C_0603_1608Metric
- C11, C38, C9: value 1u -> 0.1u; footprint Capacitor_SMD:C_0603_1608Metric -> Capacitor_SMD:C_0402_1005Metric
- H1, H2, H3, H4, H5, H6, H7, H8: footprint MountingHole:MountingHole_2.2mm_M2 -> MountingHole:MountingHole_2.2mm_M2_DIN965_Pad
- J2, J3: footprint Eurocad:MIDI_DIN5 -> KiCad:SDS50J
- SW1: value RotaryEncoder_Switch -> SW_Push; footprint Rotary_Encoder:RotaryEncoder_Alps_EC11E-Switch_Vertical_H20mm -> Button_Switch_THT:SW_PUSH_6mm
- SW2: value SW_Push -> RotaryEncoder_Switch; footprint Button_Switch_THT:SW_PUSH_6mm -> Rotary_Encoder:RotaryEncoder_Bourns_Vertical_PEC12R-3xxxF-Sxxxx
- U1, U3: footprint Package_DIP:DIP-16_W7.62mm_Socket -> Package_DIP:DIP-16_W7.62mm
- U4: value AP2112K-1.8 -> NCP1117-5.0_TO252; footprint Package_TO_SOT_SMD:SOT-23-5 -> Package_TO_SOT_SMD:TO-252-2
- U5: value H11L1 -> AP2112K-1.8; footprint Package_DIP:DIP-6_W7.62mm_Socket -> Package_TO_SOT_SMD:SOT-23-5
- U6: value IQS550-BL-QNR -> H11L1; footprint footprints5:IQS550-BL-QNR -> Package_DIP:DIP-6_W7.62mm_Socket
- U7: value SGTL5000XNLA3R2 -> IQS550-BL-QNR; footprint footprints2:SGTL5000XNLA3R2 -> footprints5:IQS550-BL-QNR
- U8: value NCP1117-5.0_TO252 -> SGTL5000XNLA3R2; footprint Package_TO_SOT_SMD:TO-252-2 -> footprints2:SGTL5000XNLA3R2
- moved C37 152.6 mm to (13.5, 134.8), turned to -90 degrees
- moved C25 146.7 mm to (151.5, 84.0)
- moved SW50 129.7 mm to (143.5, 122.6)
- moved SW14 129.6 mm to (143.3, 86.9)
- moved SW38 129.0 mm to (143.5, 113.6)
- moved SW26 129.0 mm to (143.5, 104.9)
- moved C13 111.1 mm to (132.1, 55.2), turned to 0 degrees
- moved SW2 67.7 mm to (69.0, 46.4), turned to 180 degrees
- moved SW1 48.2 mm to (23.0, 60.9)
- moved U6 43.6 mm to (101.8, 50.1), turned to 180 degrees
- moved U5 34.7 mm to (136.4, 48.2)
- moved C5 32.4 mm to (140.5, 48.3), turned to 90 degrees
- moved C3 32.3 mm to (165.8, 28.1), turned to 0 degrees
- moved C4 32.2 mm to (152.8, 23.1)
- moved C6 32.2 mm to (132.6, 48.2)
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- renumbered R13 to R15, R14 to R16
Connections:
- C10 pad 1: /Keybed/REG -> +3V3
- C12 pad 1: /Controller/TOUCH_RESET -> /Keybed/REG
- C12 pad 2: Net-(U6-NRST) -> GND
- C13 pad 1: +3V3 -> /Controller/TOUCH_RESET
- C13 pad 2: GND -> Net-(U7-NRST)
- C14 pad 1: +3V3 -> +5V
- C15 pad 1: +3V3 -> +5V
- C16 pad 1: +3V3 -> +5V
- C17 pad 1: +3V3 -> +5V
- C18 pad 1: +3V3 -> +5V
- C19 pad 1: +3V3 -> +5V
- C20 pad 1: +3V3 -> +5V
- C21 pad 1: +3V3 -> +5V
- C22 pad 1: +3V3 -> +5V
- C23 pad 1: +3V3 -> +5V
- C24 pad 1: +3V3 -> +5V
- C25 pad 1: +3V3 -> +5V
- C26 pad 1: +3V3 -> +5V
- C27 pad 1: +3V3 -> +5V
- C28 pad 1: +3V3 -> +5V
- C29 pad 1: +3V3 -> +5V
- C3 pad 1: +3V3 -> Net-(D13-K)
- C30 pad 1: +3V3 -> +5V
- C31 pad 1: +3V3 -> +5V
- C32 pad 1: +3V3 -> +5V
- C33 pad 1: +3V3 -> +5V
- C34 pad 1: +3V3 -> +5V
- C35 pad 1: +3V3 -> +5V
- C36 pad 1: +3V3 -> +5V
- C37 pad 1: +3V3 -> +5V
- C38 pad 1: +3V3 -> +1V8
- C4 pad 1: +1V8 -> +5V
- C5 pad 1: Net-(D13-K) -> +3V3
- C6 pad 1: +BATT -> +1V8
- J6 pad R: Net-(C52-Pad1) -> /Audio Interface/HP_R
- J6 pad T: Net-(C53-Pad1) -> /Audio Interface/HP_L
- SW10 pad 2: /Chord & Sequencer/C8 -> /Chord & Sequencer/C7
- SW11 pad 2: /Chord & Sequencer/C9 -> /Chord & Sequencer/C8
- SW12 pad 2: /Chord & Sequencer/C10 -> /Chord & Sequencer/C9
- SW13 pad 2: /Chord & Sequencer/C11 -> /Chord & Sequencer/C10
- SW14 pad 1: /Chord & Sequencer/R1 -> /Chord & Sequencer/R0
- SW14 pad 2: /Chord & Sequencer/C0 -> /Chord & Sequencer/C11
- SW15 pad 2: /Chord & Sequencer/C1 -> /Chord & Sequencer/C0
- SW16 pad 2: /Chord & Sequencer/C2 -> /Chord & Sequencer/C1
- SW17 pad 2: /Chord & Sequencer/C3 -> /Chord & Sequencer/C2
- SW18 pad 2: /Chord & Sequencer/C4 -> /Chord & Sequencer/C3
- SW19 pad 2: /Chord & Sequencer/C5 -> /Chord & Sequencer/C4
- SW20 pad 2: /Chord & Sequencer/C6 -> /Chord & Sequencer/C5
- SW21 pad 2: /Chord & Sequencer/C7 -> /Chord & Sequencer/C6
- SW22 pad 2: /Chord & Sequencer/C8 -> /Chord & Sequencer/C7
- SW23 pad 2: /Chord & Sequencer/C9 -> /Chord & Sequencer/C8
- SW24 pad 2: /Chord & Sequencer/C10 -> /Chord & Sequencer/C9
- SW25 pad 2: /Chord & Sequencer/C11 -> /Chord & Sequencer/C10
- SW26 pad 1: /Chord & Sequencer/R2 -> /Chord & Sequencer/R1
- SW26 pad 2: /Chord & Sequencer/C0 -> /Chord & Sequencer/C11
- SW27 pad 2: /Chord & Sequencer/C1 -> /Chord & Sequencer/C0
- SW28 pad 2: /Chord & Sequencer/C2 -> /Chord & Sequencer/C1
- SW29 pad 2: /Chord & Sequencer/C3 -> /Chord & Sequencer/C2
- SW3 pad 2: /Chord & Sequencer/C1 -> /Chord & Sequencer/C0
- SW30 pad 2: /Chord & Sequencer/C4 -> /Chord & Sequencer/C3
- SW31 pad 2: /Chord & Sequencer/C5 -> /Chord & Sequencer/C4
- SW32 pad 2: /Chord & Sequencer/C6 -> /Chord & Sequencer/C5
- SW33 pad 2: /Chord & Sequencer/C7 -> /Chord & Sequencer/C6
- SW34 pad 2: /Chord & Sequencer/C8 -> /Chord & Sequencer/C7
- SW35 pad 2: /Chord & Sequencer/C9 -> /Chord & Sequencer/C8
- SW36 pad 2: /Chord & Sequencer/C10 -> /Chord & Sequencer/C9
- SW37 pad 2: /Chord & Sequencer/C11 -> /Chord & Sequencer/C10
- SW38 pad 1: /Chord & Sequencer/R3 -> /Chord & Sequencer/R2
- SW38 pad 2: /Chord & Sequencer/C0 -> /Chord & Sequencer/C11
- SW39 pad 2: /Chord & Sequencer/C1 -> /Chord & Sequencer/C0
- SW4 pad 2: /Chord & Sequencer/C2 -> /Chord & Sequencer/C1
- SW40 pad 2: /Chord & Sequencer/C2 -> /Chord & Sequencer/C1
- SW41 pad 2: /Chord & Sequencer/C3 -> /Chord & Sequencer/C2
- SW42 pad 2: /Chord & Sequencer/C4 -> /Chord & Sequencer/C3
- SW43 pad 2: /Chord & Sequencer/C5 -> /Chord & Sequencer/C4
- SW44 pad 2: /Chord & Sequencer/C6 -> /Chord & Sequencer/C5
- SW45 pad 2: /Chord & Sequencer/C7 -> /Chord & Sequencer/C6
- SW46 pad 2: /Chord & Sequencer/C8 -> /Chord & Sequencer/C7
- SW47 pad 2: /Chord & Sequencer/C9 -> /Chord & Sequencer/C8
- SW48 pad 2: /Chord & Sequencer/C10 -> /Chord & Sequencer/C9
- SW49 pad 2: /Chord & Sequencer/C11 -> /Chord & Sequencer/C10
- SW5 pad 2: /Chord & Sequencer/C3 -> /Chord & Sequencer/C2
- SW50 pad 1: /Chord & Sequencer/R4 -> /Chord & Sequencer/R3
- SW50 pad 2: /Chord & Sequencer/C0 -> /Chord & Sequencer/C11
- SW51 pad 2: /Chord & Sequencer/C1 -> /Chord & Sequencer/C0
- SW52 pad 2: /Chord & Sequencer/C2 -> /Chord & Sequencer/C1
- SW53 pad 2: /Chord & Sequencer/C3 -> /Chord & Sequencer/C2
- SW54 pad 2: /Chord & Sequencer/C4 -> /Chord & Sequencer/C3
- SW55 pad 2: /Chord & Sequencer/C5 -> /Chord & Sequencer/C4
- SW56 pad 2: /Chord & Sequencer/C6 -> /Chord & Sequencer/C5
- SW57 pad 2: /Chord & Sequencer/C7 -> /Chord & Sequencer/C6
- SW58 pad 2: /Chord & Sequencer/C8 -> /Chord & Sequencer/C7
- SW59 pad 2: /Chord & Sequencer/C9 -> /Chord & Sequencer/C8
- SW6 pad 2: /Chord & Sequencer/C4 -> /Chord & Sequencer/C3
- SW60 pad 2: /Chord & Sequencer/C10 -> /Chord & Sequencer/C9
- SW61 pad 2: /Chord & Sequencer/C11 -> /Chord & Sequencer/C10
- SW7 pad 2: /Chord & Sequencer/C5 -> /Chord & Sequencer/C4
- SW8 pad 2: /Chord & Sequencer/C6 -> /Chord & Sequencer/C5
- SW9 pad 2: /Chord & Sequencer/C7 -> /Chord & Sequencer/C6
- U2 pad 18: +BATT -> +5V
- U2 pad 26: unconnected-(U2-PA0-Pad26) -> /Controller/PWR
- U2 pad 3: /Controller/SERIAL -> /Chord & Sequencer/R3
- U2 pad 35: /Chord & Sequencer/R2 -> unconnected-(U2-PB1-Pad35)
- U2 pad 36: /Chord & Sequencer/R3 -> /Chord & Sequencer/R2
- U2 pad 4: /Controller/DATA -> /Controller/SERIAL
- U2 pad 40: +BATT -> +5V
- U2 pad 5: /Controller/PWR -> /Controller/LATCH
- U2 pad 7: /Controller/LATCH -> /Controller/DATA
- U3 pad 11: /Controller/DATA -> unconnected-(U3-SRCLK-Pad11)
- U4 pad 1: +3V3 -> GND
- U4 pad 2: GND -> +5V
- U4 pad 3: +3V3 -> Net-(D13-K)
- U5 pad 1: Net-(D14-K) -> +3V3
- U5 pad 2: Net-(D14-A) -> GND
- U5 pad 3: unconnected-(U5-Pad3) -> +3V3
- U5 pad 4: /Controller/MIDI_RX -> unconnected-(U5-NC-Pad4)
- U5 pad 5: GND -> +1V8
- U6 pad 1: /Keybed/TX14 -> Net-(D14-K)
- U6 pad 2: /Keybed/PGRM -> Net-(D14-A)
- U6 pad 3: /Controller/TOUCH_WAKE -> unconnected-(U6-Pad3)
- U6 pad 4: unconnected-(U6-N/C-Pad4) -> /Controller/MIDI_RX
- U6 pad 5: /Keybed/SDA -> GND
- U6 pad 6: /Keybed/SCL -> +3V3
- U7 pad 1: /Audio Interface/HP_R -> /Keybed/TX14
- U7 pad 10: unconnected-(U7-MIC-Pad10) -> Net-(U7-NRST)
- U7 pad 11: unconnected-(U7-CPFLT-Pad11) -> /Keybed/RDY
- U7 pad 12: +1V8 -> unconnected-(U7-N/C-Pad12)
- U7 pad 13: /Audio Interface/AUDIO_MASTER_CLK -> /Keybed/RX0
- U7 pad 14: /Audio Interface/I2S_LR_CLK -> unconnected-(U7-Rx0B-Pad14)
- U7 pad 15: /Audio Interface/I2S_SERIAL_CLK -> /Keybed/RX1
- U7 pad 16: /Audio Interface/I2S_DATA_OUT -> unconnected-(U7-Rx1B-Pad16)
- U7 pad 17: /Audio Interface/I2S_DATA_IN -> /Keybed/RX2
- U7 pad 18: /I2C_SDA -> unconnected-(U7-Rx2B-Pad18)
- U7 pad 19: /I2C_SCL -> /Keybed/RX3
- U7 pad 2: /Audio Interface/HP_GND -> /Keybed/PGRM
- U7 pad 20: +3V3 -> unconnected-(U7-Rx3B-Pad20)
- U7 pad 3: +3V3 -> /Controller/TOUCH_WAKE
- U7 pad 4: /Audio Interface/HP_L -> unconnected-(U7-N/C-Pad4)
- U7 pad 5: /Audio Interface/VAG -> /Keybed/SDA
- U7 pad 6: /Audio Interface/LO_R -> /Keybed/SCL
- U7 pad 7: /Audio Interface/LO_L -> +3V3
- U7 pad 8: unconnected-(U7-LINEIN_R-Pad8) -> GND
- U7 pad 9: unconnected-(U7-LINEIN_L-Pad9) -> /Keybed/REG
- U8 pad 1: GND -> /Audio Interface/HP_R
- U8 pad 2: +BATT -> /Audio Interface/HP_GND
- U8 pad 3: Net-(D13-K) -> +3V3
Routing:
- net +5V: track 0.00 -> 1230.0 mm, vias 0 -> 40
- net +3V3: track 1339.6 -> 376.2 mm, vias 50 -> 7
- net +BATT: track 195.0 -> 0.00 mm, vias 15 -> 0
- net /Chord & Sequencer/LEDs/DOUT_R1: track 0.00 -> 55.2 mm
- net /Chord & Sequencer/LED_DIN: track 76.0 -> 20.9 mm, vias 2 -> 0
- net /Controller/PWR: track 29.4 -> 66.1 mm
- net /Controller/DATA: track 57.7 -> 29.4 mm, vias 1 -> 0
- net /Audio Interface/HP_L: track 10.4 -> 28.1 mm, vias 0 -> 1
- net Net-(C53-Pad1): track 15.6 -> 0.00 mm
- net /Audio Interface/HP_R: track 8.72 -> 23.4 mm
- net /Chord & Sequencer/R3: track 167.1 -> 152.6 mm
- net Net-(C52-Pad1): track 13.8 -> 0.00 mm
- net GND: track 181.6 -> 193.5 mm, vias 108 -> 113
- net /Chord & Sequencer/LEDs/DOUT_R0: track 55.2 -> 44.3 mm, vias 0 -> 1
- net Net-(U7-NRST): track 0.00 -> 9.63 mm
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- added copper zone on B.Cu, net +5V
- added copper zone on F.Cu, net +5V
- removed copper zone on F.Cu, net +BATT
Other:
- board text added: "64 STEP SEQUENCER"
- board text added: "9V BATT"
- board text added: "<- AFTERTOUCH ->"
- board text added: "<- KEYS ->"
- board text added: "AUTOHARPIE"
- board text added: "CUSTOM KEY"
- board text added: "DATA ENTRY"
- board text added: "DISPLAY"
- board text added: "GPL V3"
- board text added: "MIDI IN"
- board text added: "MIDI OUT"
- board text added: "MODE MIDI"
- board text added: "MULTITOUCH STRUMPAD"
- board text added: "OCT + OCT -"
- board text added: "PARAM UTIL"
- board text added: "REV 0.1 BY L1NPENGTUL"
- board text added: "SPEAKER"
- board text added: "STM32 BLACKPILL"
- board text added: "STRUM SYNTHESIZER"
- board text added: "THIS SYNTH KILLS FASCISTS! - TRANS RIGHTS MMXXIII - RUST GANG"
- board text added: "TOUCH_PGRM"
- board text added: "VOL GLIDE"
- board text removed: "AUTOHARPIE - STRUM SYNTHESIZER - REV 0.1"
- board text removed: "KEY CUSTOM"
- board text removed: "MODE"
- board text removed: "PAGE"
- board text removed: "PARAM"
- board text removed: "VOL PANIC!"

Commit message: new icc
Parts:
- removed J8: AudioJack3_SwitchTR, Connector_Audio:Jack_3.5mm_CUI_SJ1-3535NG_Horizontal_CircularHoles
- added C44: 1u, Capacitor_SMD:C_0603_1608Metric, F.Cu at (131.0, 22.0)
- added C45: 1u, Capacitor_SMD:C_0603_1608Metric, F.Cu at (131.0, 20.0)
- added C46: 1u, Capacitor_SMD:C_0603_1608Metric, F.Cu at (133.5, 35.0)
- added C47: 2.2u, Capacitor_SMD:C_0805_2012Metric, F.Cu at (133.0, 37.0)
- added C48: 1u, Capacitor_SMD:C_0603_1608Metric, F.Cu at (133.5, 33.2)
- C38, C39, C40: value 0.1u -> 1u; footprint Capacitor_SMD:C_0402_1005Metric -> Capacitor_SMD:C_0603_1608Metric
- C41: footprint Capacitor_THT:C_Disc_D7.0mm_W2.5mm_P5.00mm -> Capacitor_SMD:C_0603_1608Metric
- C42: value 1u -> 220u; footprint Capacitor_THT:C_Disc_D7.0mm_W2.5mm_P5.00mm -> Capacitor_SMD:C_0805_2012Metric
- C43: value 0.1u -> 220u; footprint Capacitor_SMD:C_0402_1005Metric -> Capacitor_SMD:C_0805_2012Metric
- U8: value SGTL5000XNLA3R2 -> MAX9867ETJ+T; footprint footprints2:SGTL5000XNLA3R2 -> max:QFN50P500X500X80-33N
- moved C40 24.5 mm to (125.5, 23.8), turned to 180 degrees
- moved C43 23.1 mm to (135.0, 16.5), turned to 180 degrees
- moved C39 18.5 mm to (123.0, 33.5), turned to -90 degrees
- moved C41 15.2 mm to (124.0, 27.8), turned to 90 degrees
- moved C6 14.3 mm to (140.9, 36.6)
- moved U8 14.2 mm to (128.2, 30.2), turned to 90 degrees
- moved U5 13.8 mm to (143.9, 36.5)
- moved C5 13.5 mm to (147.2, 36.5)
- moved H5 10.6 mm to (142.8, 7.75)
- moved C42 7.09 mm to (134.6, 24.5), turned to 180 degrees
- moved C38 3.56 mm to (130.0, 38.0), turned to -90 degrees
Connections:
- C38 pad 2: GND -> AGND
- C39 pad 1: +3V3 -> +1V8
- C40 pad 1: +3V3 -> +1V8
- C41 pad 1: Net-(C41-Pad1) -> +3V3
- C41 pad 2: /Audio Interface/LO_R -> AGND
- C42 pad 2: /Audio Interface/LO_L -> /Audio Interface/RIGHT
- C43 pad 1: /Audio Interface/VAG -> Net-(C43-Pad1)
- C43 pad 2: GND -> /Audio Interface/LEFT
- J6 pad R: /Audio Interface/HP_R -> Net-(C42-Pad1)
- J6 pad S: /Audio Interface/HP_GND -> AGND
- J6 pad T: /Audio Interface/HP_L -> Net-(C43-Pad1)
- J7 pad 1: /Audio Interface/HP_GND -> AGND
- U2 pad 1: /Chord & Sequencer/R1 -> /Audio Interface/I2S_LR_CLK
- U2 pad 11: unconnected-(U2-PB3-Pad11) -> /Controller/SERIAL
- U2 pad 30: /Audio Interface/I2S_LR_CLK -> unconnected-(U2-PA4-Pad30)
- U2 pad 31: /Audio Interface/I2S_SERIAL_CLK -> unconnected-(U2-PA5-Pad31)
- U2 pad 33: /Audio Interface/I2S_DATA_IN -> /Audio Interface/INT
- U2 pad 34: unconnected-(U2-PB0-Pad34) -> /Chord & Sequencer/R1
- U2 pad 35: unconnected-(U2-PB1-Pad35) -> /Chord & Sequencer/R4
- U2 pad 37: /Chord & Sequencer/R4 -> /Audio Interface/I2S_SERIAL_CLK
- U2 pad 4: /Controller/SERIAL -> /Audio Interface/I2S_DATA_IN
- U8 pad 1: /Audio Interface/HP_R -> GND
- U8 pad 12: +1V8 -> unconnected-(U8-MICLP/DIGMICDATA-Pad12)
- U8 pad 13: /Audio Interface/AUDIO_MASTER_CLK -> unconnected-(U8-MICRP-Pad13)
- U8 pad 14: /Audio Interface/I2S_LR_CLK -> unconnected-(U8-MICRN-Pad14)
- U8 pad 15: /Audio Interface/I2S_SERIAL_CLK -> unconnected-(U8-LINL-Pad15)
- U8 pad 17: /Audio Interface/I2S_DATA_IN -> unconnected-(U8-JACKSNS/AUX-Pad17)
- U8 pad 18: /I2C_SDA -> AGND
- U8 pad 19: /I2C_SCL -> /Audio Interface/RIGHT
- U8 pad 2: /Audio Interface/HP_GND -> /I2C_SCL
- U8 pad 20: +3V3 -> /Audio Interface/ROUT_AGND
- U8 pad 3: +3V3 -> /I2C_SDA
- U8 pad 4: /Audio Interface/HP_L -> /Audio Interface/INT
- U8 pad 5: /Audio Interface/VAG -> +1V8
- U8 pad 6: /Audio Interface/LO_R -> /Audio Interface/REF
- U8 pad 7: /Audio Interface/LO_L -> /Audio Interface/PREG
- U8 pad 8: unconnected-(U8-LINEIN_R-Pad8) -> /Audio Interface/REG
- U8 pad 9: unconnected-(U8-LINEIN_L-Pad9) -> AGND
Routing:
- net /Audio Interface/I2S_DATA_IN: track 155.4 -> 0.00 mm, vias 1 -> 0
- net /Audio Interface/INT: track 0.00 -> 147.0 mm, vias 0 -> 1
- net /Audio Interface/I2S_SERIAL_CLK: track 144.3 -> 0.00 mm, vias 1 -> 0
- net /Audio Interface/I2S_LR_CLK: track 141.2 -> 0.00 mm, vias 1 -> 0
- net unconnected-(U2-PA5-Pad31): track 0.00 -> 139.4 mm, vias 0 -> 1
- net unconnected-(U2-PA4-Pad30): track 0.00 -> 136.5 mm, vias 0 -> 1
- net /Audio Interface/HP_GND: track 84.0 -> 0.00 mm, vias 3 -> 0
- net /Audio Interface/HP_L: track 28.1 -> 0.00 mm, vias 1 -> 0
- net /Audio Interface/HP_R: track 23.4 -> 0.00 mm
- net /Audio Interface/LEFT: track 0.00 -> 15.8 mm
- net Net-(C41-Pad1): track 15.2 -> 0.00 mm
- net Net-(J6-PadTN): track 39.6 -> 27.8 mm
- net /I2C_SCL: track 124.4 -> 114.4 mm
- net /I2C_SDA: track 148.1 -> 138.9 mm
- net /Audio Interface/LOUT_AGND: track 0.00 -> 8.72 mm
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Other:
- board text added: "AUDIO"
- board text removed: "PHONES"

Commit message: final final final 0.1 rev
Parts:
- added C49: 1u, Capacitor_SMD:C_0603_1608Metric, F.Cu at (189.4, 20.4)
- moved R3 84.2 mm to (32.2, 26.6)
- moved R2 83.2 mm to (32.2, 29.1)
- moved H5 20.1 mm to (125.4, 17.8)
- moved R11 9.11 mm to (44.4, 20.0)
- moved R12 7.92 mm to (44.4, 24.2)
- moved R10 7.10 mm to (44.4, 22.0)
- moved J5 5.39 mm to (121.9, 48.4)
- moved C43 3.26 mm to (134.0, 19.6)
- moved C2 2.70 mm to (51.6, 50.8), turned to 0 degrees
- moved C45 2.06 mm to (130.0, 21.8)
- moved C44 1.72 mm to (130.0, 23.4)
- moved H7 1.71 mm to (109.0, 52.8)
- moved C40 1.67 mm to (124.4, 25.0)
- moved C39 1.20 mm to (124.2, 33.6)
- moved C42 1.11 mm to (134.4, 25.6)
Connections:
- C38 pad 2: AGND -> GND
- C41 pad 2: AGND -> GND
- C44 pad 2: AGND -> GND
- C45 pad 2: AGND -> GND
- J4 pad 3: /I2C_SDA -> /I2C_SCL
- J4 pad 4: /I2C_SCL -> /I2C_SDA
- J5 pad 4: /Keybed/SDA -> /I2C_SCL
- J5 pad 5: /Keybed/SCL -> /I2C_SDA
- J6 pad S: AGND -> GND
- J7 pad 1: AGND -> Net-(J7-Pin_1)
- R2 pad 2: /Keybed/SCL -> /I2C_SDA
- R3 pad 2: /Keybed/SDA -> /I2C_SCL
- U2 pad 11: /Controller/SERIAL -> unconnected-(U2-PB3-Pad11)
- U2 pad 12: /Controller/TOUCH_RESET -> unconnected-(U2-PB4-Pad12)
- U2 pad 13: /Controller/TOUCH_WAKE -> unconnected-(U2-PB5-Pad13)
- U2 pad 14: /Keybed/SCL -> /I2C_SDA
- U2 pad 15: /Keybed/SDA -> /I2C_SCL
- U2 pad 16: /I2C_SCL -> /Controller/TOUCH_RESET
- U2 pad 17: unconnected-(U2-PB9-Pad17) -> /Controller/TOUCH_WAKE
- U2 pad 23: /Controller/FRONT_ROT_B -> /Controller/FRONT_ROT_A
- U2 pad 24: /Controller/FRONT_ROT_A -> /Controller/FRONT_ROT_B
- U2 pad 34: /Chord & Sequencer/R1 -> /Chord & Sequencer/R2
- U2 pad 36: /Chord & Sequencer/R2 -> /Chord & Sequencer/R1
- U2 pad 5: /Controller/LATCH -> /Controller/SERIAL
- U2 pad 6: /I2C_SDA -> /Controller/LATCH
- U7 pad 5: /Keybed/SDA -> /I2C_SDA
- U7 pad 6: /Keybed/SCL -> /I2C_SCL
- U8 pad 18: AGND -> GND
- U8 pad 33: AGND -> GND
- U8 pad 9: AGND -> GND
Routing:
- net /Audio Interface/I2S_SERIAL_CLK: track 0.00 -> 149.8 mm, vias 0 -> 3
- net /Audio Interface/I2S_LR_CLK: track 0.00 -> 145.1 mm, vias 0 -> 1
- net /Keybed/SCL: track 142.6 -> 0.00 mm
- net /Audio Interface/I2S_DATA_IN: track 0.00 -> 141.4 mm, vias 0 -> 1
- net unconnected-(U2-PA5-Pad31): track 139.4 -> 0.00 mm, vias 1 -> 0
- net unconnected-(U2-PA4-Pad30): track 136.5 -> 0.00 mm, vias 1 -> 0
- net /Keybed/SDA: track 132.1 -> 0.00 mm
- net +1V8: track 11.4 -> 64.6 mm, vias 0 -> 4
- net /Chord & Sequencer/R1: track 130.8 -> 176.5 mm
- net /I2C_SCL: track 114.4 -> 155.3 mm, vias 2 -> 1
- net +3V3: track 373.6 -> 412.9 mm, vias 5 -> 4
- net GND: track 190.2 -> 216.7 mm, vias 107 -> 128
- net /I2C_SDA: track 138.9 -> 157.5 mm, vias 2 -> 1
- net /Controller/TOUCH_RESET: track 108.9 -> 93.1 mm, vias 4 -> 0
- net Net-(C43-Pad1): track 0.00 -> 12.2 mm
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Other:
- board text removed: "LINEOUT"
- board text removed: "STM32 BLACKPILL"
