File: hw_sch/autoharpie/autoharpie.kicad_pcb (KiCad board)
At the start: 2 copper layers, 190 x 150 mm, 190 parts, among them J1 Conn_01x02_Pin, J2 DIN-5_180degree, J3 DIN-5_180degree, J4 Conn_01x04_Socket, J5 Conn_01x06_Pin, J6 AudioJack3_SwitchTR, J7 Conn_01x02_Pin, Q1 2N7000, SW1 SW_Push, SW10 SW_Push, SW11 SW_Push, SW12 SW_Push, SW13 SW_Push, SW14 SW_Push, SW15 SW_Push, SW16 SW_Push, SW17 SW_Push, SW18 SW_Push, SW19 SW_Push, SW2 RotaryEncoder_Switch, SW20 SW_Push, SW21 SW_Push, SW22 SW_Push, SW23 SW_Push, SW24 SW_Push, SW25 SW_Push, SW26 SW_Push, SW27 SW_Push, SW28 SW_Push, SW29 SW_Push, SW3 SW_Push, SW30 SW_Push, SW31 SW_Push, SW32 SW_Push, SW33 SW_Push, SW34 SW_Push, SW35 SW_Push, SW36 SW_Push, SW37 SW_Push, SW38 SW_Push, SW39 SW_Push, SW4 SW_Push, SW40 SW_Push, SW41 SW_Push, SW42 SW_Push, SW43 SW_Push, SW44 SW_Push, SW45 SW_Push, SW46 SW_Push, SW47 SW_Push, SW48 SW_Push, SW49 SW_Push, SW5 SW_Push, SW50 SW_Push, SW51 SW_Push, SW52 SW_Push, SW53 SW_Push, SW54 SW_Push, SW55 SW_Push, SW56 SW_Push, SW57 SW_Push, SW58 SW_Push, SW59 SW_Push, SW6 SW_Push, SW60 SW_Push, SW61 SW_Push, SW62 SW_Push, SW7 SW_Push, SW8 SW_Push, SW9 SW_Push, U1 74HC595, U2 YAAJ_WeAct_BlackPill_Part_Like, U3 74HC595, U4 NCP1117-5.0_TO252, U5 AP2112K-1.8, U6 H11L1, U7 IQS550-BL-QNR, U8 MAX9867ETJ+T

Commit message: erhtj
Parts:
- C42, C43: footprint Capacitor_SMD:C_0805_2012Metric -> Capacitor_SMD:C_1206_3216Metric
Routing:
- net Net-(C43-Pad1): track 12.2 -> 11.7 mm
- net Net-(C42-Pad1): track 11.7 -> 11.2 mm
- net /Audio Interface/LEFT: track 12.2 -> 11.7 mm
- net /Audio Interface/RIGHT: track 6.40 -> 5.87 mm
