File: hw_sch/autoharpie/controller.kicad_sch (KiCad schematic)
At the start: 19 parts, among them SW3 SW_Push, SW4 SW_Push, U1 STM32F446RCTx

Commit message: keypad
Parts:
- removed C46, C47: 1u, symbol Device:C
- removed C48: 100n, symbol Device:C
- removed C49, C50: 0.1u, symbol Device:C
- removed R16: 10k, symbol Device:R
- removed SW3, SW4: SW_Push, symbol Switch:SW_Push
- added C10, C11, C12, C13, C14, C15, C8: 100n, Capacitor_SMD:C_0402_1005Metric, symbol Device:C
- added C16: 4.7u, Capacitor_SMD:C_0603_1608Metric, symbol Device:C
- added C17, C18: 15p, Capacitor_SMD:C_0402_1005Metric, symbol Device:C
- added C19: 2.2u, Capacitor_SMD:C_0603_1608Metric, symbol Device:C
- added Y1: 16MHz, Crystal:Crystal_SMD_3225-4Pin_3.2x2.5mm, symbol Device:Crystal
- C1, C4, C5, C9: footprint (none) -> Capacitor_SMD:C_0402_1005Metric
- C2, C3: value 100n -> 1u; footprint (none) -> Capacitor_SMD:C_0402_1005Metric
- C6: value 4.7u -> 100n; footprint (none) -> Capacitor_SMD:C_0402_1005Metric
- C7: value 2.2u -> 100n; footprint (none) -> Capacitor_SMD:C_0402_1005Metric
- FB1: value FerriteBead_Small -> 120R; footprint (none) -> Ferrite_THT:LairdTech_28C0236-0JW-10
- R3: value 47 -> 1k; footprint (none) -> Resistor_THT:R_Axial_DIN0204_L3.6mm_D1.6mm_P7.62mm_Horizontal
Connections:
- net VREF is gone; now on net OSC_OUT: R3.2
- net +3V3: now also C7.1, C9.1, U1.1 (VBAT), U1.19 (VDD), U1.32 (VDD), U1.48 (VDD), U1.64 (VDD), C10.1, C11.1, C12.1, C13.1, C14.1, C15.1, C16.1, C8.1; no longer C1.1, C2.1
- net GND: now also C10.2, C11.2, C12.2, C13.2, C14.2, C15.2, C16.2, C17.1, C18.1, C19.2, C8.2
- net VCAP0: now also C19.1; no longer C7.1
- net R2: now reaches U1.10 (PC2)
- net I2S_SD: now reaches U1.11 (PC3)
- net +3.3VA: now reaches U1.13 (VDDA)
- net +3.3VA: now also C1.1, C2.1, FB1.2
- net FRONT_ROT_A: now reaches U1.14 (PA0)
- net FRONT_ROT_B: now reaches U1.15 (PA1)
- net FRONT_ROT_SW: now reaches U1.16 (PA2)
- net BATT_ADC: now reaches U1.17 (PA3)
- net PWR_SW: now reaches U1.2 (PC13)
- net SPI_NSS: now reaches U1.20 (PA4)
- net SPI_SCK: now reaches U1.21 (PA5)
- net SPI_MISO: now reaches U1.22 (PA6)
- net SPI_MOSI: now reaches U1.23 (PA7)
- net R3: now reaches U1.24 (PC4)
- net R4: now reaches U1.25 (PC5)
- net C4: now reaches U1.26 (PB0)
- net C5: now reaches U1.27 (PB1)
- net C6: now reaches U1.28 (PB2)
- net C7: now reaches U1.29 (PB10)
- net PWR_LED: now reaches U1.3 (PC14)
- net C8: now reaches U1.33 (PB12)
- net C9: now reaches U1.34 (PB13)
- net C10: now reaches U1.35 (PB14)
- net C11: now reaches U1.36 (PB15)
- net I2S_CK: now reaches U1.37 (PC6)
- net I2S_MCK: now reaches U1.38 (PC7)
- net LED_DOUT1: now reaches U1.39 (PC8)
- net PSU_MODE: now reaches U1.4 (PC15)
- net LED_DOUT2: now reaches U1.40 (PC9)
- net OTG_FS_ID: now reaches U1.43 (PA10)
- net OTG_FS_D-: now reaches U1.44 (PA11)
- net OTG_FS_D+: now reaches U1.45 (PA12)
- net TOUCH_RESET: now reaches U1.49 (PA14)
- net OSC_IN: now reaches U1.5 (PH0)
- net OSC_IN: now also C17.2, Y1.2
- net I2S_WS: now reaches U1.50 (PA15)
- net R5: now reaches U1.51 (PC10)
- net C0: now reaches U1.52 (PC11)
- net C1: now reaches U1.53 (PC12)
- net C2: now reaches U1.55 (PB3)
- net C3: now reaches U1.56 (PB4)
- net MIDI_TX: now reaches U1.58 (PB6)
- net MIDI_RX: now reaches U1.59 (PB7)
- net OSC_OUT: now reaches U1.6 (PH1)
- net I2C_SCL: now reaches U1.61 (PB8)
- net I2C_SDA: now reaches U1.62 (PB9)
- net R0: now reaches U1.8 (PC0)
- net R1: now reaches U1.9 (PC1)
- removed net VADD: C9.1, FB1.2, R3.1
- new net: C18.2, R3.1, Y1.1
- no-connect marks 0 -> 1

Commit message: rev 0.1 pcb
Parts:
- removed C10, C11, C12, C13, C14, C15, C4, C5, C6, C7, C8, C9: 100n, Capacitor_SMD:C_0402_1005Metric, symbol Device:C
- removed C16: 4.7u, Capacitor_SMD:C_0603_1608Metric, symbol Device:C
- removed C17, C18: 15p, Capacitor_SMD:C_0402_1005Metric, symbol Device:C
- removed C19: 2.2u, Capacitor_SMD:C_0603_1608Metric, symbol Device:C
- removed C3: 1u, Capacitor_SMD:C_0402_1005Metric, symbol Device:C
- removed FB1: 120R, Ferrite_THT:LairdTech_28C0236-0JW-10, symbol Device:FerriteBead_Small
- removed U1: STM32F446RCTx, Package_QFP:LQFP-64_10x10mm_P0.5mm, symbol MCU_ST_STM32F4:STM32F446RCTx
- removed Y1: 16MHz, Crystal:Crystal_SMD_3225-4Pin_3.2x2.5mm, symbol Device:Crystal
- added D19 (x12): 1N4148, Diode_THT:D_DO-35_SOD27_P7.62mm_Horizontal, symbol Device:D
- added R1: 20k, Resistor_THT:R_Axial_DIN0204_L3.6mm_D1.6mm_P7.62mm_Horizontal, symbol Device:R
- added R2, R5: 4.7k, Resistor_THT:R_Axial_DIN0204_L3.6mm_D1.6mm_P7.62mm_Horizontal, symbol Device:R
- added R4: 10k, Resistor_THT:R_Axial_DIN0204_L3.6mm_D1.6mm_P7.62mm_Horizontal, symbol Device:R
- added SW74: SW_Push, Button_Switch_THT:SW_PUSH_6mm, symbol Switch:SW_Push
- added U1, U3: 74HC595, Package_DIP:DIP-16_W7.62mm_Socket, symbol 74xx:74HC595
- added U2: YAAJ_WeAct_BlackPill_Part_Like, Footprints:YAAJ_WeAct_BlackPill_2, symbol YAAJ_WeAct_BlackPill_Part_Like:YAAJ_WeAct_BlackPill_Part_Like
- C1: value 100n -> 0.1u
- C2: value 1u -> 0.1u
- R3: value 1k -> 4.7k
Connections:
- net +3.3VA is gone; now on net +3V3: C1.1, C2.1
- net +3V3: now also R3.1, R2.1, R5.1, SW74.1, U1.10 (~{SRCLR}), U1.16 (VCC), U2.20 (3V3), U2.38 (3V3), U3.10 (~{SRCLR}), U3.16 (VCC)
- net C0: now also D19.1 (K)
- net C1: now also D19.1 (K)
- net C10: now also D19.1 (K)
- net C11: now also D19.1 (K)
- net C2: now also D19.1 (K)
- net C3: now also D19.1 (K)
- net C4: now also D19.1 (K)
- net C5: now also D19.1 (K)
- net C6: now also D19.1 (K)
- net C7: now also D19.1 (K)
- net C8: now also D19.1 (K)
- net C9: now also D19.1 (K)
- net FRONT_ROT_A: now also U2.24 (PC15)
- net FRONT_ROT_B: now also U2.23 (PC14)
- net FRONT_ROT_SW: now also U2.22 (PC13)
- net GND: now also R4.2, R5.2, U1.13 (~{OE}), U1.8 (GND), U2.19 (GND), U2.39 (GND), U3.13 (~{OE}), U3.8 (GND)
- net I2S_CK: now also U2.31 (PA5)
- net I2S_MCK: now also U2.32 (PA6)
- net I2S_SD: now also U2.33 (PA7)
- net I2S_WS: now also U2.30 (PA4)
- net MIDI_RX: now also U2.29 (PA3)
- net MIDI_TX: now also U2.28 (PA2)
- net R0: now also U2.2 (PB13)
- net R1: now also U2.1 (PB12)
- net R2: now also U2.35 (PB1)
- net R3: now also U2.36 (PB2)
- net R4: now also U2.37 (PB10)
- net TOUCH_RESET: now also U2.12 (PB4)
- net OSC_OUT renamed I2C1_SCL
- net I2C1_SCL: now also U2.15 (PB7)
- new net +BATT: U2.18 (5V), U2.40 (5V)
- new net A0: D19.2 (A), U1.1 (QB)
- new net A1: D19.2 (A), U1.2 (QC)
- new net A10: D19.2 (A), U3.4 (QE)
- new net A11: D19.2 (A), U3.5 (QF)
- new net A2: D19.2 (A), U1.3 (QD)
- new net A3: D19.2 (A), U1.4 (QE)
- new net A4: D19.2 (A), U1.5 (QF)
- new net A5: D19.2 (A), U1.6 (QG)
- new net A6: D19.2 (A), U1.7 (QH)
- new net A7: D19.2 (A), U3.1 (QB)
- new net A8: D19.2 (A), U3.2 (QC)
- new net A9: D19.2 (A), U3.3 (QD)
- new net BATT_SENSE: R1.1
- new net BAT_SENSE: R1.2, R4.1, U2.27 (PA1)
- new net DATA: U1.11 (SRCLK), U2.4 (PB15), U3.11 (SRCLK)
- new net DOUT0: U1.9 (QH'), U3.14 (SER)
- new net I2C1_SDA: R2.2, U2.14 (PB6)
- new net I2C3_SCL: U2.6 (PA9)
- new net I2C3_SDA: U2.16 (PB8)
- new net LATCH: U1.12 (RCLK), U2.7 (PA10), U3.12 (RCLK)
- new net LED_DOUT: U2.10 (PA15)
- new net PWR: SW74.2, U2.5 (PA8)
- new net SERIAL: U1.14 (SER), U2.3 (PB14)
- new net TOUCH_WAKE: U2.13 (PB5)
- no-connect marks 1 -> 13

Commit message: ic fix atept
Parts:
- added XU1, XU3: Conn_02x08_Counter_Clockwise, Package_DIP:DIP-16_W7.62mm_Socket, symbol Connector_Generic:Conn_02x08_Counter_Clockwise
- U1, U3: footprint Package_DIP:DIP-16_W7.62mm_Socket -> Package_DIP:DIP-16_W7.62mm
- renumbered SW74 to SW1
Connections:
- net DATA: now also U2.7 (PA10); no longer U2.4 (PB15), U3.11 (SRCLK)
- net LATCH: now also U2.5 (PA8); no longer U2.7 (PA10)
- net PWR: now also U2.26 (PA0); no longer U2.5 (PA8)
- net R2: now also U2.36 (PB2); no longer U2.35 (PB1)
- net R3: now also U2.3 (PB14); no longer U2.36 (PB2)
- net SERIAL: now also U2.4 (PB15); no longer U2.3 (PB14)
- net +BATT renamed +5V
- no-connect marks 13 -> 46

Commit message: new icc
Parts:
- renumbered XU3 to XU2
Connections:
- net I2S_CK: now also U2.37 (PB10); no longer U2.31 (PA5)
- net I2S_SD: now also U2.4 (PB15); no longer U2.33 (PA7)
- net I2S_WS: now also U2.1 (PB12); no longer U2.30 (PA4)
- net R1: now also U2.34 (PB0); no longer U2.1 (PB12)
- net R4: now also U2.35 (PB1); no longer U2.37 (PB10)
- net SERIAL: now also U2.11 (PB3); no longer U2.4 (PB15)
- new net AUDIO_IRQ: U2.33 (PA7)
- no-connect marks 46 -> 45

Commit message: final final final 0.1 rev
Connections:
- net I2C3_SCL is gone; now on net LATCH: U2.6 (PA9)
- net I2C3_SDA is gone; now on net TOUCH_RESET: U2.16 (PB8)
- net FRONT_ROT_A: now also U2.23 (PC14); no longer U2.24 (PC15)
- net FRONT_ROT_B: now also U2.24 (PC15); no longer U2.23 (PC14)
- net LATCH: no longer U2.5 (PA8)
- net R1: now also U2.36 (PB2); no longer U2.34 (PB0)
- net R2: now also U2.34 (PB0); no longer U2.36 (PB2)
- net SERIAL: now also U2.5 (PA8); no longer U2.11 (PB3)
- net TOUCH_RESET: no longer U2.12 (PB4)
- net TOUCH_WAKE: now also U2.17 (PB9); no longer U2.13 (PB5)
- no-connect marks 45 -> 47
Changed lines of the file:
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@@
   (no_connect (at 154.94 74.93))
   (no_connect (at 110.49 77.47))
+  (no_connect (at 175.26 102.87))
   (no_connect (at 142.24 82.55))
   (no_connect (at 154.94 67.31))
@@
   (no_connect (at 175.26 92.71))
   (no_connect (at 142.24 74.93))
-  (no_connect (at 175.26 115.57))
   (no_connect (at 123.19 64.77))
   (no_connect (at 154.94 77.47))
   (no_connect (at 110.49 82.55))
+  (no_connect (at 175.26 105.41))
   (no_connect (at 142.24 72.39))
   (no_connect (at 123.19 67.31))
@@
   (no_connect (at 123.19 77.47))
   (no_connect (at 154.94 80.01))
+  (no_connect (at 175.26 100.33))
   (no_connect (at 123.19 69.85))
   (no_connect (at 142.24 67.31))
@@
     (effects (font (size 1.27 1.27)) (justify left bottom))
   )
-  (label "SERIAL" (at 175.26 100.33 180) (fields_autoplaced)
-    (effects (font (size 1.27 1.27)) (justify right bottom))
-  )
   (label "BAT_SENSE" (at 215.9 107.95 0) (fields_autoplaced)
     (effects (font (size 1.27 1.27)) (justify left bottom))
   )
-  (label "LATCH" (at 175.26 85.09 180) (fields_autoplaced)
-    (effects (font (size 1.27 1.27)) (justify right bottom))
-  )
   (label "A4" (at 36.83 96.52 0) (fields_autoplaced)
     (effects (font (size 1.27 1.27)) (justify left bottom))
@@
     (effects (font (size 1.27 1.27)) (justify left bottom))
   )
+  (label "A2" (at 36.83 81.28 0) (fields_autoplaced)
+    (effects (font (size 1.27 1.27)) (justify left bottom))
+  )
+  (label "LATCH" (at 93.98 76.2 0) (fields_autoplaced)
+    (effects (font (size 1.27 1.27)) (justify left bottom))
+  )
+  (label "DOUT0" (at 54.61 86.36 180) (fields_autoplaced)
+    (effects (font (size 1.27 1.27)) (justify right bottom))
+  )
+  (label "SERIAL" (at 93.98 63.5 0) (fields_autoplaced)
+    (effects (font (size 1.27 1.27)) (justify left bottom))
+  )
+  (label "PWR" (at 135.89 146.05 0) (fields_autoplaced)
+    (effects (font (size 1.27 1.27)) (justify left bottom))
+  )
+  (label "A9" (at 66.04 142.24 180) (fields_autoplaced)
+    (effects (font (size 1.27 1.27)) (justify right bottom))
+  )
+  (label "A11" (at 66.04 147.32 180) (fields_autoplaced)
+    (effects (font (size 1.27 1.27)) (justify right bottom))
+  )
+  (label "A1" (at 66.04 68.58 180) (fields_autoplaced)
+    (effects (font (size 1.27 1.27)) (justify right bottom))
+  )
+  (label "A7" (at 36.83 120.65 0) (fields_autoplaced)
+    (effects (font (size 1.27 1.27)) (justify left bottom))
+  )
+  (label "SERIAL" (at 175.26 85.09 180) (fields_autoplaced)
+    (effects (font (size 1.27 1.27)) (justify right bottom))
+  )
+  (label "A10" (at 66.04 144.78 180) (fields_autoplaced)
+    (effects (font (size 1.27 1.27)) (justify right bottom))
+  )
   (label "DATA" (at 175.26 90.17 180) (fields_autoplaced)
     (effects (font (size 1.27 1.27)) (justify right bottom))
   )
-  (label "A2" (at 36.83 81.28 0) (fields_autoplaced)
-    (effects (font (size 1.27 1.27)) (justify left bottom))
-  )
-  (label "LATCH" (at 93.98 76.2 0) (fields_autoplaced)
-    (effects (font (size 1.27 1.27)) (justify left bottom))
-  )
-  (label "DOUT0" (at 54.61 86.36 180) (fields_autoplaced)
-    (effects (font (size 1.27 1.27)) (justify right bottom))
-  )
-  (label "SERIAL" (at 93.98 63.5 0) (fields_autoplaced)
-    (effects (font (size 1.27 1.27)) (justify left bottom))
-  )
-  (label "PWR" (at 135.89 146.05 0) (fields_autoplaced)
-    (effects (font (size 1.27 1.27)) (justify left bottom))
-  )
-  (label "A9" (at 66.04 142.24 180) (fields_autoplaced)
-    (effects (font (size 1.27 1.27)) (justify right bottom))
-  )
-  (label "A11" (at 66.04 147.32 180) (fields_autoplaced)
-    (effects (font (size 1.27 1.27)) (justify right bottom))
-  )
-  (label "A1" (at 66.04 68.58 180) (fields_autoplaced)
-    (effects (font (size 1.27 1.27)) (justify right bottom))
-  )
-  (label "A7" (at 36.83 120.65 0) (fields_autoplaced)
-    (effects (font (size 1.27 1.27)) (justify left bottom))
-  )
-  (label "A10" (at 66.04 144.78 180) (fields_autoplaced)
-    (effects (font (size 1.27 1.27)) (justify right bottom))
-  )
   (label "A4" (at 66.04 76.2 180) (fields_autoplaced)
     (effects (font (size 1.27 1.27)) (justify right bottom))
@@
   (label "BAT_SENSE" (at 246.38 106.68 0) (fields_autoplaced)
     (effects (font (size 1.27 1.27)) (justify left bottom))
+  )
+  (label "LATCH" (at 175.26 87.63 180) (fields_autoplaced)
+    (effects (font (size 1.27 1.27)) (justify right bottom))
   )
   (label "A10" (at 36.83 143.51 0) (fields_autoplaced)
@@
     (effects (font (size 1.27 1.27)) (justify right))
   )
-  (hierarchical_label "FRONT_ROT_A" (shape input) (at 215.9 115.57 0) (fields_autoplaced)
+  (hierarchical_label "FRONT_ROT_A" (shape input) (at 215.9 118.11 0) (fields_autoplaced)
     (effects (font (size 1.27 1.27)) (justify left))
   )
@@
     (effects (font (size 1.27 1.27)) (justify right))
   )
-  (hierarchical_label "I2C3_SCL" (shape output) (at 175.26 87.63 180) (fields_autoplaced)
-    (effects (font (size 1.27 1.27)) (justify right))
-  )
   (hierarchical_label "R0" (shape input) (at 175.26 77.47 180) (fields_autoplaced)
     (effects (font (size 1.27 1.27)) (justify right))
@@
     (effects (font (size 1.27 1.27)) (justify right))
   )
-  (hierarchical_label "I2C3_SDA" (shape bidirectional) (at 175.26 113.03 180) (fields_autoplaced)
-    (effects (font (size 1.27 1.27)) (justify right))
-  )
   (hierarchical_label "MIDI_RX" (shape input) (at 215.9 102.87 0) (fields_autoplaced)
     (effects (font (size 1.27 1.27)) (justify left))
@@
     (effects (font (size 1.27 1.27)) (justify right))
   )
-  (hierarchical_label "TOUCH_RESET" (shape input) (at 175.26 102.87 180) (fields_autoplaced)
-    (effects (font (size 1.27 1.27)) (justify right))
-  )
   (hierarchical_label "C10" (shape output) (at 29.21 143.51 180) (fields_autoplaced)
     (effects (font (size 1.27 1.27)) (justify right))
@@
     (effects (font (size 1.27 1.27)) (justify right))
   )
-  (hierarchical_label "FRONT_ROT_B" (shape input) (at 215.9 118.11 0) (fields_autoplaced)
-    (effects (font (size 1.27 1.27)) (justify left))
+  (hierarchical_label "TOUCH_RESET" (shape input) (at 175.26 113.03 180) (fields_autoplaced)
+    (effects (font (size 1.27 1.27)) (justify right))
+  )
+  (hierarchical_label "FRONT_ROT_B" (shape input) (at 215.9 115.57 0) (fields_autoplaced)
+    (effects (font (size 1.27 1.27)) (justify left))
+  )
+  (hierarchical_label "TOUCH_WAKE" (shape input) (at 175.26 115.57 180) (fields_autoplaced)
+    (effects (font (size 1.27 1.27)) (justify right))
   )
   (hierarchical_label "I2S_CK" (shape output) (at 215.9 82.55 0) (fields_autoplaced)
@@
     (effects (font (size 1.27 1.27)) (justify right))
   )
-  (hierarchical_label "R1" (shape input) (at 215.9 90.17 0) (fields_autoplaced)
+  (hierarchical_label "R1" (shape input) (at 215.9 85.09 0) (fields_autoplaced)
     (effects (font (size 1.27 1.27)) (justify left))
   )
@@
     (effects (font (size 1.27 1.27)) (justify right))
   )
-  (hierarchical_label "R2" (shape input) (at 215.9 85.09 0) (fields_autoplaced)
+  (hierarchical_label "R2" (shape input) (at 215.9 90.17 0) (fields_autoplaced)
     (effects (font (size 1.27 1.27)) (justify left))
   )
@@
     (effects (font (size 1.27 1.27)) (justify right))
   )
-  (hierarchical_label "TOUCH_WAKE" (shape input) (at 175.26 105.41 180) (fields_autoplaced)
-    (effects (font (size 1.27 1.27)) (justify right))
-  )
