File: hw_sch/autoharpie/keys.kicad_sch (KiCad schematic)
At the start: 13 parts, among them J1 Conn_01x04_Pin, SW1 SW_Push, U1 MSP430FR2633IDAR, Y1 32.768KHz

Commit message: keypad
Parts:
- added J8: Conn_01x25_Socket, Connector_PinSocket_2.54mm:PinSocket_1x25_P2.54mm_Vertical, symbol Connector:Conn_01x25_Socket
- C2: footprint Capacitor_SMD:C_1206_3216Metric -> Capacitor_SMD:C_0603_1608Metric
- C4: footprint Capacitor_SMD:C_0201_0603Metric -> Capacitor_SMD:C_0402_1005Metric
- R1, R2: footprint Resistor_SMD:R_0603_1608Metric -> Resistor_THT:R_Axial_DIN0204_L3.6mm_D1.6mm_P7.62mm_Horizontal
- U1: footprint footprints:MSP430FR2633IDAR -> footprints3:MSP430FR2633IDAR
- Y1: footprint Crystal:Crystal_SMD_MicroCrystal_CM9V-T1A-2Pin_1.6x1.0mm -> Crystal:Crystal_SMD_2012-2Pin_2.0x1.2mm
Connections:
- net +3V3: now also J8.10 (Pin_10), J8.22 (Pin_22)
- net CAP0: now also J8.19 (Pin_19)
- net CAP1: now also J8.18 (Pin_18)
- net CAP2: now also J8.17 (Pin_17)
- net CAP3: now also J8.16 (Pin_16)
- net CAP4: now also J8.15 (Pin_15)
- net CAP5: now also J8.14 (Pin_14)
- net CAP6: now also J8.13 (Pin_13)
- net CAP7: now also J8.12 (Pin_12)
- net CAP_SW: now also J8.25 (Pin_25)
- net FRX0: now also J8.8 (Pin_8)
- net FRX1: now also J8.7 (Pin_7)
- net FRX2: now also J8.6 (Pin_6)
- net FRX3: now also J8.5 (Pin_5)
- net FRX4: now also J8.4 (Pin_4)
- net FRX5: now also J8.3 (Pin_3)
- net FRX6: now also J8.2 (Pin_2)
- net FRX7: now also J8.1 (Pin_1)
- net GND: now also J8.11 (Pin_11), J8.20 (Pin_20), J8.21 (Pin_21), J8.23 (Pin_23), J8.24 (Pin_24), J8.9 (Pin_9)

Commit message: rev 0.1 pcb
Parts:
- removed C1: 1u, Capacitor_SMD:C_0402_1005Metric, symbol Device:C
- removed C2: 10u, Capacitor_SMD:C_0603_1608Metric, symbol Device:C
- removed C3: 0.1u, Capacitor_SMD:C_0402_1005Metric, symbol Device:C
- removed C4: 1000n, Capacitor_SMD:C_0402_1005Metric, symbol Device:C
- removed C5, C6: 22p, Capacitor_SMD:C_0402_1005Metric, symbol Device:C
- removed D1: LED, LED_SMD:LED_0402_1005Metric, symbol Device:LED
- removed J1: Conn_01x04_Pin, Connector_PinHeader_2.54mm:PinHeader_1x04_P2.54mm_Vertical, symbol Connector:Conn_01x04_Pin
- removed J8: Conn_01x25_Socket, Connector_PinSocket_2.54mm:PinSocket_1x25_P2.54mm_Vertical, symbol Connector:Conn_01x25_Socket
- removed R1: 470, Resistor_THT:R_Axial_DIN0204_L3.6mm_D1.6mm_P7.62mm_Horizontal, symbol Device:R
- removed R2: 47k, Resistor_THT:R_Axial_DIN0204_L3.6mm_D1.6mm_P7.62mm_Horizontal, symbol Device:R
- removed SW1: SW_Push, Button_Switch_SMD:SW_Push_SPST_NO_Alps_SKRK, symbol Switch:SW_Push
- removed U1: MSP430FR2633IDAR, footprints3:MSP430FR2633IDAR, symbol 2023-03-09_01-52-04:MSP430FR2633IDAR
- removed Y1: 32.768KHz, Crystal:Crystal_SMD_2012-2Pin_2.0x1.2mm, symbol Device:Crystal
- added C10, C12, C37, C8: 0.1u, Capacitor_SMD:C_0402_1005Metric, symbol Device:C
- added C11, C38, C9: 1u, Capacitor_SMD:C_0603_1608Metric, symbol Device:C
- added J5: Conn_01x06_Pin, Connector_PinHeader_2.54mm:PinHeader_1x06_P2.54mm_Vertical, symbol Connector:Conn_01x06_Pin
- added U6: IQS550-BL-QNR, footprints5:IQS550-BL-QNR, symbol 2023-04-03_23-40-49:IQS550-BL-QNR
Connections:
- net +3V3: now also C37.1, C38.1, C8.1, C9.1, J5.1 (Pin_1), U6.38 (VDDIO), U6.7 (VDDHI)
- net GND: now also C10.2, C11.2, C37.2, C38.2, C8.2, C9.2, J5.2 (Pin_2), U6.37 (VSSIO), U6.49, U6.8 (VSS)
- net RESET: now also C12.1
- net RX0: now also U6.13 (Rx0A)
- net RX1: now also U6.15 (Rx1A)
- net RX2: now also U6.17 (Rx2A)
- net RX3: now also U6.19 (Rx3A)
- net RX4: now also U6.21 (Rx4A)
- net RX5: now also U6.23 (Rx5A)
- net RX6: now also U6.25 (Rx6A)
- net RX7: now also U6.27 (Rx7A)
- new net: C12.2, U6.10 (NRST)
- new net PGRM: J5.3 (Pin_3), U6.2 (PGM)
- new net RDY: J5.6 (Pin_6), U6.11 (RDY)
- new net REG: C10.1, C11.1, U6.9 (VREG)
- new net RX8: U6.29 (Rx8A)
- new net RX9: U6.31 (Rx9A)
- new net TOUCH_SCL: J5.5 (Pin_5), U6.6 (SCL)
- new net TOUCH_SDA: J5.4 (Pin_4), U6.5 (SDA)
- new net TX0: U6.33 (Tx0)
- new net TX1: U6.34 (Tx1)
- new net TX10: U6.45 (Tx10)
- new net TX11: U6.46 (Tx11)
- new net TX12: U6.47 (Tx12)
- new net TX13: U6.48 (Tx13)
- new net TX14: U6.1 (Tx14)
- new net TX2: U6.35 (Tx2)
- new net TX3: U6.36 (Tx3)
- new net TX4: U6.39 (Tx4)
- new net TX5: U6.40 (Tx5)
- new net TX6: U6.41 (Tx6)
- new net TX7: U6.42 (Tx7)
- new net TX8: U6.43 (Tx8)
- new net TX9: U6.44 (Tx9)
- new net WAKE: U6.3 (SW_IN)
- no-connect marks 3 -> 10
Other:
- removed sheet RX Pin Filter
- added sheet Touchpad (touchpad.kicad_sch)

Commit message: ic fix atept
Parts:
- renumbered C38 to C10, C10 to C11, C11 to C12, C12 to C13, C8 to C7, C9 to C8, C37 to C9, U6 to U7
Connections:
- net RX6: no longer names the net of U7.25 (Rx6A)
- net RX7: no longer names the net of U7.27 (Rx7A)
- net RX8: no longer names the net of U7.29 (Rx8A)
- net RX9: no longer names the net of U7.31 (Rx9A)
- no-connect marks 10 -> 18

Commit message: final final final 0.1 rev
Connections:
- net TOUCH_SCL: now also J5.4 (Pin_4); no longer J5.5 (Pin_5)
- net TOUCH_SDA: now also J5.5 (Pin_5); no longer J5.4 (Pin_4)
Changed lines of the file:
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@@
     (effects (font (size 1.27 1.27)) (justify left bottom))
   )
-  (label "SDA" (at 38.1 134.62 0) (fields_autoplaced)
+  (label "SDA" (at 38.1 137.16 0) (fields_autoplaced)
     (effects (font (size 1.27 1.27)) (justify left bottom))
   )
@@
     (effects (font (size 1.27 1.27)) (justify right bottom))
   )
-  (label "SCL" (at 38.1 137.16 0) (fields_autoplaced)
+  (label "SCL" (at 38.1 134.62 0) (fields_autoplaced)
     (effects (font (size 1.27 1.27)) (justify left bottom))
   )
