File: hw_sch/keypad16/capsense_bus_switch.kicad_sch (KiCad schematic)
At the start: 9 parts, among them U2 TS5A23159RSE, U3 TS5A23159RSE, U4 TS5A23159RSE, U5 TS5A23159RSE

Commit message: routing and new footprint
Parts:
- added C10, C8, C9: 1u, Capacitor_SMD:C_0201_0603Metric, symbol Device:C
- C11: renamed from C8; footprint Capacitor_SMD:C_0402_1005Metric -> Capacitor_SMD:C_0201_0603Metric
- C12: renamed from C9; footprint Capacitor_SMD:C_0402_1005Metric -> Capacitor_SMD:C_0201_0603Metric
- C13: renamed from C10; footprint Capacitor_SMD:C_0402_1005Metric -> Capacitor_SMD:C_0201_0603Metric
- C14: renamed from C11; footprint Capacitor_SMD:C_0402_1005Metric -> Capacitor_SMD:C_0201_0603Metric
- C7: value 10u -> 1u; footprint Capacitor_SMD:C_1206_3216Metric -> Capacitor_SMD:C_0201_0603Metric
Connections:
- net +3V3: now also C10.1, C8.1, C9.1
- net GND: now also C10.2, C8.2, C9.2
Other:
- moved on the sheet: C11, C12, C13, C14

Commit message: finish keypad
Parts:
- removed C10, C8, C9: 1u, Capacitor_SMD:C_0201_0603Metric, symbol Device:C
- removed C11, C12, C13, C14: 0.1u, Capacitor_SMD:C_0201_0603Metric, symbol Device:C
- removed U2, U3, U4, U5: TS5A23159RSE, Package_DFN_QFN:Texas_R-PUQFN-N10, symbol Analog_Switch:TS5A23159RSE
- added C2: 0.1u, Capacitor_SMD:C_0402_1005Metric, symbol Device:C
- added U1: TS3L501ERUA, Package_DFN_QFN:WQFN-42-1EP_3.5x9mm_P0.5mm_EP2.05x7.55mm, symbol Analog_Switch:TS3L501ERUA
- C1: renamed from C7; footprint Capacitor_SMD:C_0201_0603Metric -> Capacitor_SMD:C_0603_1608Metric
Connections:
- net +3V3: now also C2.1, U1.39 (VDD)
- net A0: now also U1.25 (B6)
- net A1: now also U1.24 (B7)
- net A2: now also U1.29 (B4)
- net A3: now also U1.28 (B5)
- net A4: now also U1.34 (B2)
- net A5: now also U1.33 (B3)
- net A6: now also U1.38 (B0)
- net A7: now also U1.37 (B1)
- net B0: now also U1.23 (C6)
- net B1: now also U1.22 (C7)
- net B2: now also U1.27 (C4)
- net B3: now also U1.26 (C5)
- net B4: now also U1.32 (C2)
- net B5: now also U1.31 (C3)
- net B6: now also U1.36 (C0)
- net B7: now also U1.35 (C1)
- net GND: now also C2.2, U1.43 (GND)
- net I0: now also U1.12 (A7)
- net I1: now also U1.11 (A6)
- net I2: now also U1.10 (A5)
- net I3: now also U1.9 (A4)
- net I4: now also U1.7 (A3)
- net I5: now also U1.6 (A2)
- net I6: now also U1.3 (A1)
- net I7: now also U1.2 (A0)
- net SWITCH: now also U1.13 (SEL)
- no-connect marks 0 -> 16
Other:
- moved on the sheet: C1
