File: hw_sch/keypad16/key_sensor.kicad_sch (KiCad schematic)
At the start: 0 parts

Commit message: routing and new footprint
Parts:
- added TP1, TP100, TP101, TP102, TP103, TP104, TP11, TP113, TP114, TP115, TP116, TP117, TP118, TP119, TP120, TP13, TP15, TP17, TP18, TP19, TP20, TP21, TP22, TP23, TP24, TP3, TP33, TP34, TP35, TP36, TP37, TP38, TP39, TP40, TP49, TP5, TP50, TP51, TP52, TP53, TP54, TP55, TP56, TP65, TP66, TP67, TP68, TP69, TP7, TP70, TP71, TP72, TP81, TP82, TP83, TP84, TP85, TP86, TP87, TP88, TP9, TP97, TP98, TP99: ~, keypad:Mutual Capicitance Pad, symbol keypad:Mutual_Touch_Pad
Connections:
- net C0: now also TP1.1 (T), TP11.1 (T), TP13.1 (T), TP15.1 (T), TP3.1 (T), TP5.1 (T), TP7.1 (T), TP9.1 (T)
- net C1: now also TP17.1 (T), TP18.1 (T), TP19.1 (T), TP20.1 (T), TP21.1 (T), TP22.1 (T), TP23.1 (T), TP24.1 (T)
- net C2: now also TP33.1 (T), TP34.1 (T), TP35.1 (T), TP36.1 (T), TP37.1 (T), TP38.1 (T), TP39.1 (T), TP40.1 (T)
- net C3: now also TP49.1 (T), TP50.1 (T), TP51.1 (T), TP52.1 (T), TP53.1 (T), TP54.1 (T), TP55.1 (T), TP56.1 (T)
- net C4: now also TP65.1 (T), TP66.1 (T), TP67.1 (T), TP68.1 (T), TP69.1 (T), TP70.1 (T), TP71.1 (T), TP72.1 (T)
- net C5: now also TP81.1 (T), TP82.1 (T), TP83.1 (T), TP84.1 (T), TP85.1 (T), TP86.1 (T), TP87.1 (T), TP88.1 (T)
- net C6: now also TP100.1 (T), TP101.1 (T), TP102.1 (T), TP103.1 (T), TP104.1 (T), TP97.1 (T), TP98.1 (T), TP99.1 (T)
- net C7: now also TP113.1 (T), TP114.1 (T), TP115.1 (T), TP116.1 (T), TP117.1 (T), TP118.1 (T), TP119.1 (T), TP120.1 (T)
- net RX0: now also TP1.2 (R), TP113.2 (R), TP17.2 (R), TP33.2 (R), TP49.2 (R), TP65.2 (R), TP81.2 (R), TP97.2 (R)
- net RX1: now also TP114.2 (R), TP18.2 (R), TP3.2 (R), TP34.2 (R), TP50.2 (R), TP66.2 (R), TP82.2 (R), TP98.2 (R)
- net RX2: now also TP115.2 (R), TP19.2 (R), TP35.2 (R), TP5.2 (R), TP51.2 (R), TP67.2 (R), TP83.2 (R), TP99.2 (R)
- net RX3: now also TP100.2 (R), TP116.2 (R), TP20.2 (R), TP36.2 (R), TP52.2 (R), TP68.2 (R), TP7.2 (R), TP84.2 (R)
- net RX4: now also TP101.2 (R), TP117.2 (R), TP21.2 (R), TP37.2 (R), TP53.2 (R), TP69.2 (R), TP85.2 (R), TP9.2 (R)
- net RX5: now also TP102.2 (R), TP11.2 (R), TP118.2 (R), TP22.2 (R), TP38.2 (R), TP54.2 (R), TP70.2 (R), TP86.2 (R)
- net RX6: now also TP103.2 (R), TP119.2 (R), TP13.2 (R), TP23.2 (R), TP39.2 (R), TP55.2 (R), TP71.2 (R), TP87.2 (R)
- net RX7: now also TP104.2 (R), TP120.2 (R), TP15.2 (R), TP24.2 (R), TP40.2 (R), TP56.2 (R), TP72.2 (R), TP88.2 (R)
Other:
- removed sheet Key 1
- removed sheet Key 2
- removed sheet Key 3
- removed sheet Key 4
- removed sheet Key 5
- removed sheet Key 6
- removed sheet Key 7
- removed sheet Key 8

Commit message: finish keypad
Parts:
- renumbered TP53 to TP100, TP69 to TP101, TP85 to TP102, TP101 to TP103, TP117 to TP104, TP11 to TP105, TP22 to TP106, TP38 to TP107, TP54 to TP108, TP70 to TP109, TP86 to TP110, TP102 to TP111, TP118 to TP112, TP13 to TP113, TP23 to TP114, TP39 to TP115, TP55 to TP116, TP71 to TP117, TP87 to TP118, TP103 to TP119, TP119 to TP120, TP15 to TP121, TP24 to TP122, TP40 to TP123, TP56 to TP124, TP72 to TP125, TP88 to TP126, TP104 to TP127, TP120 to TP128, TP1 to TP65, TP17 to TP66, TP33 to TP67, TP49 to TP68, TP65 to TP69, TP81 to TP70, TP97 to TP71, TP113 to TP72, TP3 to TP73, TP18 to TP74, TP34 to TP75, TP50 to TP76, TP66 to TP77, TP82 to TP78, TP98 to TP79, TP114 to TP80, TP5 to TP81, TP19 to TP82, TP35 to TP83, TP51 to TP84, TP67 to TP85, TP83 to TP86, TP99 to TP87, TP115 to TP88, TP7 to TP89, TP20 to TP90, TP36 to TP91, TP52 to TP92, TP68 to TP93, TP84 to TP94, TP100 to TP95, TP116 to TP96, TP9 to TP97, TP21 to TP98, TP37 to TP99
Connections:
- net RX0: now also TP121.2 (R), TP122.2 (R), TP123.2 (R), TP124.2 (R), TP125.2 (R), TP126.2 (R), TP127.2 (R), TP128.2 (R); no longer TP65.2 (R), TP66.2 (R), TP67.2 (R), TP68.2 (R), TP69.2 (R), TP70.2 (R), TP71.2 (R), TP72.2 (R)
- net RX1: now also TP113.2 (R), TP114.2 (R), TP115.2 (R), TP116.2 (R), TP117.2 (R), TP118.2 (R), TP119.2 (R), TP120.2 (R); no longer TP73.2 (R), TP74.2 (R), TP75.2 (R), TP76.2 (R), TP77.2 (R), TP78.2 (R), TP79.2 (R), TP80.2 (R)
- net RX2: now also TP105.2 (R), TP106.2 (R), TP107.2 (R), TP108.2 (R), TP109.2 (R), TP110.2 (R), TP111.2 (R), TP112.2 (R); no longer TP81.2 (R), TP82.2 (R), TP83.2 (R), TP84.2 (R), TP85.2 (R), TP86.2 (R), TP87.2 (R), TP88.2 (R)
- net RX3: now also TP100.2 (R), TP101.2 (R), TP102.2 (R), TP103.2 (R), TP104.2 (R), TP97.2 (R), TP98.2 (R), TP99.2 (R); no longer TP89.2 (R), TP90.2 (R), TP91.2 (R), TP92.2 (R), TP93.2 (R), TP94.2 (R), TP95.2 (R), TP96.2 (R)
- net RX4: now also TP89.2 (R), TP90.2 (R), TP91.2 (R), TP92.2 (R), TP93.2 (R), TP94.2 (R), TP95.2 (R), TP96.2 (R); no longer TP100.2 (R), TP101.2 (R), TP102.2 (R), TP103.2 (R), TP104.2 (R), TP97.2 (R), TP98.2 (R), TP99.2 (R)
- net RX5: now also TP81.2 (R), TP82.2 (R), TP83.2 (R), TP84.2 (R), TP85.2 (R), TP86.2 (R), TP87.2 (R), TP88.2 (R); no longer TP105.2 (R), TP106.2 (R), TP107.2 (R), TP108.2 (R), TP109.2 (R), TP110.2 (R), TP111.2 (R), TP112.2 (R)
- net RX6: now also TP73.2 (R), TP74.2 (R), TP75.2 (R), TP76.2 (R), TP77.2 (R), TP78.2 (R), TP79.2 (R), TP80.2 (R); no longer TP113.2 (R), TP114.2 (R), TP115.2 (R), TP116.2 (R), TP117.2 (R), TP118.2 (R), TP119.2 (R), TP120.2 (R)
- net RX7: now also TP65.2 (R), TP66.2 (R), TP67.2 (R), TP68.2 (R), TP69.2 (R), TP70.2 (R), TP71.2 (R), TP72.2 (R); no longer TP121.2 (R), TP122.2 (R), TP123.2 (R), TP124.2 (R), TP125.2 (R), TP126.2 (R), TP127.2 (R), TP128.2 (R)
