File: hw_sch/keypad16/rxpin_filter.kicad_sch (KiCad schematic)
At the start: 16 parts

Commit message: routing and new footprint
Parts:
- renumbered C12 to C15, C13 to C16, C14 to C17, C15 to C18, C16 to C19, C17 to C20, C18 to C21, C19 to C22

Commit message: finish keypad
Parts:
- removed R10, R3, R4, R5, R6, R7, R8, R9: 470, Resistor_SMD:R_0201_0603Metric, symbol Device:R
- C10: renamed from C22; footprint Capacitor_SMD:C_0201_0603Metric -> Capacitor_SMD:C_0402_1005Metric
- C3: renamed from C15; footprint Capacitor_SMD:C_0201_0603Metric -> Capacitor_SMD:C_0402_1005Metric
- C4: renamed from C16; footprint Capacitor_SMD:C_0201_0603Metric -> Capacitor_SMD:C_0402_1005Metric
- C5: renamed from C17; footprint Capacitor_SMD:C_0201_0603Metric -> Capacitor_SMD:C_0402_1005Metric
- C6: renamed from C18; footprint Capacitor_SMD:C_0201_0603Metric -> Capacitor_SMD:C_0402_1005Metric
- C7: renamed from C19; footprint Capacitor_SMD:C_0201_0603Metric -> Capacitor_SMD:C_0402_1005Metric
- C8: renamed from C20; footprint Capacitor_SMD:C_0201_0603Metric -> Capacitor_SMD:C_0402_1005Metric
- C9: renamed from C21; footprint Capacitor_SMD:C_0201_0603Metric -> Capacitor_SMD:C_0402_1005Metric
Other:
- note added: "NOTE: Series 470Ohm Resistor on Main PCB"
