File: hw_sch/keypad16/keypad16.kicad_sch (KiCad schematic)
At the start: 18 parts, among them J1 Conn_01x04_Pin, J2 Conn_01x10_Pin, SW1 SW_Push, U1 MSP430FR2633IDAR, Y1 32.768KHz

Commit message: routing and new footprint
Parts:
- removed H1, H2, H3, H4: MountingHole, MountingHole:MountingHole_2.2mm_M2, symbol Mechanical:MountingHole
- added H1, H2, H3, H4: MountingHole_Pad, MountingHole:MountingHole_2.2mm_M2_DIN965_Pad, symbol Mechanical:MountingHole_Pad
- R1: footprint Resistor_SMD:R_0805_2012Metric -> Resistor_SMD:R_0603_1608Metric
Connections:
- net GND_ISO is gone; now on net GND: J1.1 (Pin_1), U1.3 (DVSS)
- net GND: now also H1.1, H2.1, H3.1, H4.1
- no-connect marks 0 -> 3
Other:
- sheet Bus Switch ports: added none; removed 3V3_ISO, ISO_GND
- sheet Key Sensor 1 ports: added C[0..7]; removed I[0..7]
- sheet Key Sensor 2 ports: added C[0..7]; removed I[0..7]

Commit message: finish keypad
Parts:
- removed C1: 1u, Capacitor_SMD:C_0402_1005Metric, symbol Device:C
- removed C2: 10u, Capacitor_SMD:C_1206_3216Metric, symbol Device:C
- removed C3: 0.1u, Capacitor_SMD:C_0402_1005Metric, symbol Device:C
- removed C4: 1000n, Capacitor_SMD:C_0201_0603Metric, symbol Device:C
- removed C5, C6: 22p, Capacitor_SMD:C_0402_1005Metric, symbol Device:C
- removed D1: LED, LED_SMD:LED_0402_1005Metric, symbol Device:LED
- removed J1: Conn_01x04_Pin, Connector_PinHeader_2.54mm:PinHeader_1x04_P2.54mm_Horizontal, symbol Connector:Conn_01x04_Pin
- removed J2: Conn_01x10_Pin, Connector_PinHeader_2.54mm:PinHeader_1x10_P2.54mm_Vertical, symbol Connector:Conn_01x10_Pin
- removed R1: 470, Resistor_SMD:R_0603_1608Metric, symbol Device:R
- removed R2: 47k, Resistor_SMD:R_0603_1608Metric, symbol Device:R
- removed SW1: SW_Push, Button_Switch_SMD:SW_Push_SPST_NO_Alps_SKRK, symbol Switch:SW_Push
- removed U1: MSP430FR2633IDAR, footprints:MSP430FR2633IDAR, symbol 2023-03-09_01-52-04:MSP430FR2633IDAR
- removed Y1: 32.768KHz, Crystal:Crystal_SMD_MicroCrystal_CM9V-T1A-2Pin_1.6x1.0mm, symbol Device:Crystal
- added J1: 09231486921, 09321:09231486921, symbol 09231486921:09231486921
- added J2, J3: Conn_01x08_Pin, Connector_PinHeader_2.54mm:PinHeader_1x08_P2.54mm_Vertical, symbol Connector:Conn_01x08_Pin
- added J4: Conn_01x04_Pin, Connector_PinHeader_2.54mm:PinHeader_1x04_P2.54mm_Vertical, symbol Connector:Conn_01x04_Pin
Connections:
- net +3V3: now also J1.A2, J4.1 (Pin_1)
- net CAP0: now also J1.C1, J2.1 (Pin_1)
- net CAP1: now also J1.C2, J2.2 (Pin_2)
- net CAP2: now also J1.C3, J2.3 (Pin_3)
- net CAP3: now also J1.C4, J2.4 (Pin_4)
- net CAP4: now also J1.C5, J2.5 (Pin_5)
- net CAP5: now also J1.C6, J2.6 (Pin_6)
- net CAP6: now also J1.C7, J2.7 (Pin_7)
- net CAP7: now also J1.C8, J2.8 (Pin_8)
- net CAP_SW: now also J4.4 (Pin_4)
- net GND: now also J1.A1, J1.A10, J1.A11, J1.A16, J1.A7, J1.A8, J1.A9, J1.B1, J1.B10, J1.B11, J1.B12, J1.B13, J1.B14, J1.B15, J1.B16, J1.B2, J1.B3, J1.B4, J1.B5, J1.B6, J1.B7, J1.B8, J1.B9, J4.2 (Pin_2), J4.3 (Pin_3)
- net RX0: now also J1.C9, J3.1 (Pin_1)
- net RX1: now also J1.C10, J3.2 (Pin_2)
- net RX2: now also J1.C11, J3.3 (Pin_3)
- net RX3: now also J1.C12, J3.4 (Pin_4)
- net RX4: now also J1.C13, J3.5 (Pin_5)
- net RX5: now also J1.C14, J3.6 (Pin_6)
- net RX6: now also J1.C15, J3.7 (Pin_7)
- net RX7: now also J1.C16, J3.8 (Pin_8)
- no-connect marks 3 -> 8
Other:
- removed sheet Key Sensor 1
- removed sheet Key Sensor 2
- added sheet Keys (keys.kicad_sch)

Commit message: keypad
Parts:
- removed J2, J3: Conn_01x08_Pin, Connector_PinHeader_2.54mm:PinHeader_1x08_P2.54mm_Vertical, symbol Connector:Conn_01x08_Pin
- removed J4: Conn_01x04_Pin, Connector_PinHeader_2.54mm:PinHeader_1x04_P2.54mm_Vertical, symbol Connector:Conn_01x04_Pin
- added J2: Conn_01x25_Pin, Connector_PinHeader_2.54mm:PinHeader_1x25_P2.54mm_Vertical, symbol Connector:Conn_01x25_Pin
Connections:
- net +3V3: now also J2.10 (Pin_10), J2.22 (Pin_22)
- net CAP0: now also J2.19 (Pin_19)
- net CAP1: now also J2.18 (Pin_18)
- net CAP2: now also J2.17 (Pin_17)
- net CAP3: now also J2.16 (Pin_16)
- net CAP4: now also J2.15 (Pin_15)
- net CAP5: now also J2.14 (Pin_14)
- net CAP6: now also J2.13 (Pin_13)
- net CAP7: now also J2.12 (Pin_12)
- net CAP_SW: now also J2.25 (Pin_25)
- net GND: now also J2.11 (Pin_11), J2.20 (Pin_20), J2.21 (Pin_21), J2.23 (Pin_23), J2.24 (Pin_24), J2.9 (Pin_9)
- net RX0: now also J2.8 (Pin_8)
- net RX1: now also J2.7 (Pin_7)
- net RX2: now also J2.6 (Pin_6)
- net RX3: now also J2.5 (Pin_5)
- net RX4: now also J2.4 (Pin_4)
- net RX5: now also J2.3 (Pin_3)
- net RX6: now also J2.2 (Pin_2)
- net RX7: now also J2.1 (Pin_1)
